File: RAM+LEFT_BOTTOM_BANKs.sch (KiCad schematic (older format))
At the start: 15 parts, among them J501 CONN_01X35, U301 iCE40-HX4K-TQ144, U501 AS4C1M16S

Commit message: The schematic is now free of any ERC error. Not connected and power flags added. No more global power pins, hierarchical labels used for power connections. TODO list: -Check if all footpritns are already assigned. -Export a BOM list, and check if all part numbers are assigned. -Add leds and testpoints. -Make another branch, with the RAM connections to the left and right banks, so the ram could be located in the bottom layer and the FPGA in the top layer. -Reorder the connections of the current branch if necessary, do the placement of components and ground planes.
Connections:
- net labels removed: IOL_10A, IOL_10B, IOL_12A, IOL_12B, IOL_13A, IOL_2A, IOL_2B, IOL_3A, IOL_3B, IOL_4A, IOL_4B, IOL_5A, IOL_5B, IOL_8A, IOL_8B
- wire segments 75 -> 74
- no-connect marks 0 -> 2

Commit message: First netlist export
Parts:
- J501: footprint (none) -> Pin_Headers:Pin_Header_Straight_1x35_Pitch1.27mm
- U301: footprint (none) -> Housings_QFP:LQFP-144_20x20mm_Pitch0.5mm
- U501: footprint MODULE -> TSOP50-II:TSOP50-II
Changed lines of the file:
@@
 F 0 "U301" H 7450 4950 60  0000 L CNN
 F 1 "iCE40-HX4K-TQ144" H 7450 4850 60  0000 L CNN
-F 2 "" H 7250 4700 60  0001 C CNN
+F 2 "Housings_QFP:LQFP-144_20x20mm_Pitch0.5mm" H 7250 4700 60  0001 C CNN
 F 3 "" H 7250 4700 60  0001 C CNN
 	4    7250 4700
@@
 F 0 "U301" H 2500 2400 60  0000 L CNN
 F 1 "iCE40-HX4K-TQ144" H 2500 2300 60  0000 L CNN
-F 2 "" H 2300 2150 60  0001 C CNN
+F 2 "Housings_QFP:LQFP-144_20x20mm_Pitch0.5mm" H 2300 2150 60  0001 C CNN
 F 3 "" H 2300 2150 60  0001 C CNN
 	5    2300 2150
@@
 F 0 "J501" H 8850 5300 50  0000 C CNN
 F 1 "CONN_01X35" V 8950 3500 50  0000 C CNN
-F 2 "" H 8850 3500 50  0001 C CNN
+F 2 "Pin_Headers:Pin_Header_Straight_1x35_Pitch1.27mm" H 8850 3500 50  0001 C CNN
 F 3 "" H 8850 3500 50  0001 C CNN
 	1    8850 3500
@@
 F 0 "U501" H 4750 3350 50  0000 C CNN
 F 1 "AS4C1M16S" H 4750 3550 50  0000 C CNN
-F 2 "MODULE" H 4750 3450 50  0001 C CNN
+F 2 "TSOP50-II:TSOP50-II" H 4750 3450 50  0001 C CNN
 F 3 "DOCUMENTATION" H 4750 3450 50  0001 C CNN
 	1    4750 3450

Commit message: Se conecta la tensión 5V a los conectores (right y left) y se cambia de nombre de un componente MIC2005A-2 -> MIC2005A-2YM5
Connections:
- net labels added: +5V
- wire segments 74 -> 73
Other:
- moved on the sheet: C512
Changed lines of the file:
@@
 LIBS:MIC2005A-2
 LIBS:AS4C1M16S
-LIBS:iCE40hxk4_dev_board-cache
 EELAYER 25 0
 EELAYER END
@@
 L C C512
 U 1 1 58E817F5
-P 10300 1950
-F 0 "C512" H 10400 1950 50  0000 L CNN
-F 1 "100nF" H 10350 1850 50  0000 L CNN
-F 2 "Capacitors_SMD:C_0603_HandSoldering" H 10338 1800 50  0001 C CNN
-F 3 "http://www.mouser.com/ds/2/212/KEM_C1002_X7R_SMD-357932.pdf" H 10300 1950 50  0001 C CNN
-F 4 "C0603C104K3RACTU" H 10300 1950 60  0001 C CNN "Manufacturer Part"
-F 5 "X7R" H 10300 1950 60  0001 C CNN "Dielectric"
-F 6 "25V (min. 10V)" H 10300 1950 60  0001 C CNN "VDC"
-	1    10300 1950
+P 10000 1950
+F 0 "C512" H 10100 1950 50  0000 L CNN
+F 1 "100nF" H 10050 1850 50  0000 L CNN
+F 2 "Capacitors_SMD:C_0603_HandSoldering" H 10038 1800 50  0001 C CNN
+F 3 "http://www.mouser.com/ds/2/212/KEM_C1002_X7R_SMD-357932.pdf" H 10000 1950 50  0001 C CNN
+F 4 "C0603C104K3RACTU" H 10000 1950 60  0001 C CNN "Manufacturer Part"
+F 5 "X7R" H 10000 1950 60  0001 C CNN "Dielectric"
+F 6 "25V (min. 10V)" H 10000 1950 60  0001 C CNN "VDC"
+	1    10000 1950
 	1    0    0    -1
 $EndComp
@@
 Connection ~ 4900 5100
 Wire Wire Line
-	10050 5050 10050 5200
+	10050 5200 10050 5050
 Wire Wire Line
 	9050 5200 10350 5200
@@
 	1800 5700 2550 5700
 Wire Wire Line
-	10300 2200 10300 2100
-Wire Wire Line
 	9050 1800 10300 1800
-Wire Wire Line
-	9550 1650 9550 1800
-Connection ~ 9550 1800
 Wire Wire Line
 	9050 1900 9300 1900
@@
 Connection ~ 9300 1900
 Wire Wire Line
-	9050 2100 9700 2100
+	9050 2100 10300 2100
 Wire Wire Line
 	9050 2200 9250 2200
@@
 NoConn ~ 5800 4400
 NoConn ~ 5800 4500
-Wire Wire Line
-	9050 3100 9050 4600
 Connection ~ 9050 3200
 Connection ~ 9050 3300
@@
 Text HLabel 7750 1900 2    60   Input Italic 12
 +3.3V
-Text HLabel 9550 1650 2    60   Input Italic 12
+Text HLabel 10300 1800 2    60   Input Italic 12
 +3.3V
 Text HLabel 10350 5200 2    60   Input Italic 12
 GNDD
-Text HLabel 10300 2200 2    60   Input Italic 12
-GNDD
-Text HLabel 9700 2100 2    60   Input Italic 12
+Text HLabel 10300 2100 2    60   Input Italic 12
 GNDD
 Text HLabel 9650 3400 2    60   Input Italic 12
@@
 	2300 4950 2300 5400
 Connection ~ 2300 5400
+Text HLabel 10350 4600 2    60   Input ~ 12
++5V
+Wire Wire Line
+	9050 4600 10350 4600
+Wire Wire Line
+	9050 3100 9050 4500
+Connection ~ 10000 1800
+Connection ~ 10000 2100
 $EndSCHEMATC

Commit message: Routing
Changed lines of the file:
@@
 Text Label 3700 2700 2    60   ~ 0
 A3
-Text Label 3700 2800 2    60   ~ 0
-A4
-Text Label 3700 2900 2    60   ~ 0
-A5
 Text Label 3700 3000 2    60   ~ 0
 A6
@@
 	9050 5000 9200 5000
 Connection ~ 9200 5100
-Text Label 2300 3550 0    60   ~ 0
-A4
-Text Label 2300 3450 0    60   ~ 0
-A5
-Text Label 2300 3350 0    60   ~ 0
+Text Label 2300 2150 0    60   ~ 0
 A6
-Text Label 2300 3250 0    60   ~ 0
+Text Label 2300 2250 0    60   ~ 0
 A7
-Text Label 2300 3150 0    60   ~ 0
+Text Label 2300 2350 0    60   ~ 0
 A8
-Text Label 2300 3050 0    60   ~ 0
+Text Label 2300 2450 0    60   ~ 0
 A9
-Text Label 2300 2950 0    60   ~ 0
+Text Label 2300 2550 0    60   ~ 0
 CKE
-Text Label 2300 2850 0    60   ~ 0
+Text Label 2300 2650 0    60   ~ 0
 CLK
 Text Label 2300 2750 0    60   ~ 0
 UDQM
-Text Label 2300 2550 0    60   ~ 0
+Text Label 2300 2950 0    60   ~ 0
 DQ9
-Text Label 2300 2450 0    60   ~ 0
+Text Label 2300 3050 0    60   ~ 0
 DQ10
-Text Label 2300 2350 0    60   ~ 0
+Text Label 2300 3150 0    60   ~ 0
 DQ11
-Text Label 2300 2250 0    60   ~ 0
+Text Label 2300 3250 0    60   ~ 0
 DQ12
-Text Label 2300 2150 0    60   ~ 0
+Text Label 2300 3350 0    60   ~ 0
 DQ13
-Text HLabel 5800 3900 2    60   BiDi ~ 12
-DQ15
-Text Label 2300 2650 0    60   ~ 0
+Text Label 2300 2850 0    60   ~ 0
 DQ8
-Text HLabel 5800 3800 2    60   BiDi ~ 12
-DQ14
 Wire Wire Line
 	9050 3400 9650 3400
@@
 Connection ~ 10000 1800
 Connection ~ 10000 2100
+Text Label 5800 3800 0    60   ~ 0
+DQ14
+Text Label 5800 3900 0    60   ~ 0
+DQ15
+Text HLabel 3700 2800 0    60   Input ~ 0
+A4
+Text HLabel 3700 2900 0    60   Input ~ 0
+A5
+Text Label 2300 3450 0    60   ~ 0
+DQ14
+Text Label 2300 3550 0    60   ~ 0
+DQ15
 $EndSCHEMATC

Commit message: Assignement of FPGA pins for analog stage control
Parts:
- removed C511, C512: 100nF, Capacitors_SMD:C_0603_HandSoldering, symbol C
- removed J501: CONN_01X35, Pin_Headers:Pin_Header_Straight_1x35_Pitch1.27mm, symbol CONN_01X35
Connections:
- net labels removed: +5V, IOT_168, IOT_169, IOT_170, IOT_171, IOT_172, IOT_173, IOT_174
- wire segments 73 -> 52
Other:
- note removed: "LEFT HEADER"
Changed lines of the file:
@@
 $Descr A4 11693 8268
 encoding utf-8
-Sheet 5 11
+Sheet 4 11
 Title ""
 Date ""
@@
 Comment4 ""
 $EndDescr
-Text Notes 8800 1550 0    60   ~ 12
-LEFT HEADER
 Text HLabel 6900 2900 0    60   BiDi Italic 12
 D0
@@
 	5    2300 2150
 	-1   0    0    -1
-$EndComp
-$Comp
-L C C511
-U 1 1 58E81763
-P 10050 4900
-F 0 "C511" H 10150 4900 50  0000 L CNN
-F 1 "100nF" H 10100 4800 50  0000 L CNN
-F 2 "Capacitors_SMD:C_0603_HandSoldering" H 10088 4750 50  0001 C CNN
-F 3 "http://www.mouser.com/ds/2/212/KEM_C1002_X7R_SMD-357932.pdf" H 10050 4900 50  0001 C CNN
-F 4 "C0603C104K3RACTU" H 10050 4900 60  0001 C CNN "Manufacturer Part"
-F 5 "X7R" H 10050 4900 60  0001 C CNN "Dielectric"
-F 6 "25V (min. 10V)" H 10050 4900 60  0001 C CNN "VDC"
-	1    10050 4900
-	1    0    0    -1
-$EndComp
-$Comp
-L C C512
-U 1 1 58E817F5
-P 10000 1950
-F 0 "C512" H 10100 1950 50  0000 L CNN
-F 1 "100nF" H 10050 1850 50  0000 L CNN
-F 2 "Capacitors_SMD:C_0603_HandSoldering" H 10038 1800 50  0001 C CNN
-F 3 "http://www.mouser.com/ds/2/212/KEM_C1002_X7R_SMD-357932.pdf" H 10000 1950 50  0001 C CNN
-F 4 "C0603C104K3RACTU" H 10000 1950 60  0001 C CNN "Manufacturer Part"
-F 5 "X7R" H 10000 1950 60  0001 C CNN "Dielectric"
-F 6 "25V (min. 10V)" H 10000 1950 60  0001 C CNN "VDC"
-	1    10000 1950
-	1    0    0    -1
 $EndComp
 Text Label 5800 2400 0    60   ~ 0
@@
 Text Notes 7600 1500 2    60   ~ 12
 FPGA BANK 2\n(BOTTOM BANK)
-$Comp
-L CONN_01X35 J501
-U 1 1 58E92216
-P 8850 3500
-F 0 "J501" H 8850 5300 50  0000 C CNN
-F 1 "CONN_01X35" V 8950 3500 50  0000 C CNN
-F 2 "Pin_Headers:Pin_Header_Straight_1x35_Pitch1.27mm" H 8850 3500 50  0001 C CNN
-F 3 "" H 8850 3500 50  0001 C CNN
-	1    8850 3500
-	-1   0    0    -1
-$EndComp
-Text HLabel 9050 2400 2    60   BiDi ~ 12
-IOT_168
-Text HLabel 9050 2500 2    60   BiDi ~ 12
-IOT_169
-Text HLabel 9050 2600 2    60   BiDi ~ 12
-IOT_170
-Text HLabel 9050 2700 2    60   BiDi ~ 12
-IOT_171
-Text HLabel 9050 2800 2    60   BiDi ~ 12
-IOT_172
-Text HLabel 9050 2900 2    60   BiDi ~ 12
-IOT_173
-Text HLabel 9050 3000 2    60   BiDi ~ 12
-IOT_174
 Wire Wire Line
 	1800 5400 2550 5400
@@
 Connection ~ 4900 5100
 Wire Wire Line
-	10050 5200 10050 5050
-Wire Wire Line
-	9050 5200 10350 5200
-Wire Wire Line
 	1800 5700 2550 5700
-Wire Wire Line
-	9050 1800 10300 1800
-Wire Wire Line
-	9050 1900 9300 1900
-Wire Wire Line
-	9300 1800 9300 2000
-Connection ~ 9300 1800
-Wire Wire Line
-	9300 2000 9050 2000
-Connection ~ 9300 1900
-Wire Wire Line
-	9050 2100 10300 2100
-Wire Wire Line
-	9050 2200 9250 2200
-Wire Wire Line
-	9250 2100 9250 2300
-Connection ~ 9250 2100
-Wire Wire Line
-	9250 2300 9050 2300
-Connection ~ 9250 2200
-Wire Wire Line
-	9050 4700 10350 4700
-Wire Wire Line
-	10050 4700 10050 4750
-Connection ~ 10050 4700
-Wire Wire Line
-	9050 4800 9200 4800
-Wire Wire Line
-	9200 4700 9200 4900
-Connection ~ 9200 4700
-Wire Wire Line
-	9200 4900 9050 4900
-Connection ~ 9200 4800
-Connection ~ 10050 5200
-Wire Wire Line
-	9050 5100 9200 5100
-Wire Wire Line
-	9200 5000 9200 5200
-Connection ~ 9200 5200
-Wire Wire Line
-	9050 5000 9200 5000
-Connection ~ 9200 5100
 Text Label 2300 2150 0    60   ~ 0
 A6
@@
 Text Label 2300 2850 0    60   ~ 0
 DQ8
-Wire Wire Line
-	9050 3400 9650 3400
 NoConn ~ 5800 4400
 NoConn ~ 5800 4500
-Connection ~ 9050 3200
-Connection ~ 9050 3300
-Connection ~ 9050 3400
-Connection ~ 9050 3500
-Connection ~ 9050 3600
-Connection ~ 9050 3700
-Connection ~ 9050 3800
-Connection ~ 9050 3900
-Connection ~ 9050 4000
-Connection ~ 9050 4100
-Connection ~ 9050 4200
-Connection ~ 9050 4300
-Connection ~ 9050 4400
-Connection ~ 9050 4500
 Text HLabel 2550 5400 2    60   Input Italic 12
 +3.3V
@@
 Text HLabel 7750 1900 2    60   Input Italic 12
 +3.3V
-Text HLabel 10300 1800 2    60   Input Italic 12
-+3.3V
-Text HLabel 10350 5200 2    60   Input Italic 12
-GNDD
-Text HLabel 10300 2100 2    60   Input Italic 12
-GNDD
-Text HLabel 9650 3400 2    60   Input Italic 12
-GNDD
 Text HLabel 7750 2300 2    60   Input Italic 12
 GNDD
@@
 GNDD
 Connection ~ 3250 1850
-Text HLabel 10350 4700 2    60   Input Italic 12
-+3.3V
 Wire Wire Line
 	3700 1800 3700 1850
@@
 	2300 4950 2300 5400
 Connection ~ 2300 5400
-Text HLabel 10350 4600 2    60   Input ~ 12
-+5V
-Wire Wire Line
-	9050 4600 10350 4600
-Wire Wire Line
-	9050 3100 9050 4500
-Connection ~ 10000 1800
-Connection ~ 10000 2100
 Text Label 5800 3800 0    60   ~ 0
 DQ14
 Text Label 5800 3900 0    60   ~ 0
 DQ15
-Text HLabel 3700 2800 0    60   Input ~ 0
+Text HLabel 3700 2800 0    60   BiDi ~ 0
 A4
-Text HLabel 3700 2900 0    60   Input ~ 0
+Text HLabel 3700 2900 0    60   BiDi ~ 0
 A5
 Text Label 2300 3450 0    60   ~ 0
