File: RAM+LEFT_BOTTOM_BANKs.sch (KiCad schematic (older format))
At the start: 12 parts, among them U301 iCE40-HX4K-TQ144, U501 AS4C1M16S

Commit message: Modified a lot of fields in components parts. BOM generated. Added BOM plugin script.
Parts:
- C501, C502, C503, C504, C505, C506, C507, C508, C509, C510: MPN (none) -> C0603C104K3RACTU; Manufacturer Part C0603C104K3RACTU -> (none); Type (none) -> Ceramic; VDC 25V (min. 10V) -> 25V
- U301: MPN (none) -> iCE40-HX4K-TQ144
- U501: MPN (none) -> AS4C1M16S
