File: ADC.sch (KiCad schematic (older format))
At the start: 47 parts, among them U501 ADC1175, U502 ADC1175

Commit message: Completed part selection of analog board. Merged analog and digital boards.
Parts:
- renumbered C501 to C1001, C502 to C1002, C503 to C1003, C504 to C1004, C505 to C1005, C506 to C1006, C507 to C1007, C508 to C1008, C509 to C1009, C510 to C1010, C511 to C1011, C512 to C1012, C513 to C1013, C514 to C1014, C515 to C1015, C516 to C1016, C517 to C1017, C518 to C1018, D501 to D1001, D502 to D1002, D503 to D1003, D504 to D1004, D505 to D1005, D506 to D1006, D507 to D1007, L501 to L1001, L502 to L1002, L503 to L1003, L504 to L1004, L505 to L1005, L506 to L1006, L507 to L1007, R501 to R1001, R502 to R1002, R503 to R1003, R504 to R1004, R505 to R1005, R506 to R1006, R507 to R1007, R508 to R1008, R509 to R1009, R510 to R1010, R511 to R1011, R512 to R1012, R513 to R1013, U501 to U1001, U502 to U1002

Commit message: Continued with routing...
Parts:
- R1002: footprint Resistors_SMD:R_0603 -> Resistors_SMD:R_0603_HandSoldering
Changed lines of the file:
@@
 F 0 "R1002" V 3725 5200 50  0000 L CNN
 F 1 "0" V 3900 5175 50  0000 L CNN
-F 2 "Resistors_SMD:R_0603" H 3825 5250 50  0001 C CNN
+F 2 "Resistors_SMD:R_0603_HandSoldering" H 3825 5250 50  0001 C CNN
 F 3 "http://www.mouser.com/ds/2/447/PYu-RC1206_51_RoHS_L-4-349080.pdf" H 3825 5250 50  0001 C CNN
 F 4 "RC1206JR-070RL" V 3825 5250 60  0001 C CNN "Manufacturer Part"

Commit message: Ended placing (?)
Parts:
- R1005: footprint Resistors_SMD:R_0603 -> Resistors_SMD:R_0603_HandSoldering
Changed lines of the file:
@@
 F 0 "R1005" V 3825 2650 50  0000 L CNN
 F 1 "0" V 4000 2625 50  0000 L CNN
-F 2 "Resistors_SMD:R_0603" H 3925 2700 50  0001 C CNN
+F 2 "Resistors_SMD:R_0603_HandSoldering" H 3925 2700 50  0001 C CNN
 F 3 "http://www.mouser.com/ds/2/447/PYu-RC1206_51_RoHS_L-4-349080.pdf" H 3925 2700 50  0001 C CNN
 F 4 "RC1206JR-070RL" V 3925 2700 60  0001 C CNN "Manufacturer Part"
