File: ADC.sch (KiCad schematic (older format))
At the start: 47 parts, among them U1001 ADC1175, U1002 ADC1175

Commit message: Added testpoints to schematic.
Parts:
- added J? (x6): Testpoint, library:Via-0.8mm, symbol CONN_01X01
Connections:
- wire segments 151 -> 159
Changed lines of the file:
@@
 $Descr A4 11693 8268
 encoding utf-8
-Sheet 9 11
+Sheet 7 11
 Title ""
 Date ""
@@
 Text Notes 7250 1225 0    60   ~ 0
 ADC Input Protection
-Text Notes 6975 4075 0    60   ~ 0
+Text Notes 7100 3950 0    60   ~ 0
 ADC Input Protection
 Text Notes 3725 3900 0    60   ~ 0
@@
 Text Label 9725 5925 3    60   ~ 0
 GND_D
+NoConn ~ 8800 2175
+NoConn ~ 8800 2675
+NoConn ~ 8825 5000
+NoConn ~ 8825 5500
+$Comp
+L CONN_01X01 J?
+U 1 1 599E7444
+P 8475 1500
+F 0 "J?" H 8475 1600 50  0000 C CNN
+F 1 "Testpoint" V 8575 1500 50  0000 C CNN
+F 2 "library:Via-0.8mm" H 8475 1500 50  0001 C CNN
+F 3 "" H 8475 1500 50  0001 C CNN
+	1    8475 1500
+	1    0    0    -1
+$EndComp
+$Comp
+L CONN_01X01 J?
+U 1 1 599E7723
+P 8425 4300
+F 0 "J?" H 8425 4400 50  0000 C CNN
+F 1 "Testpoint" V 8525 4300 50  0000 C CNN
+F 2 "library:Via-0.8mm" H 8425 4300 50  0001 C CNN
+F 3 "" H 8425 4300 50  0001 C CNN
+	1    8425 4300
+	1    0    0    -1
+$EndComp
+$Comp
+L CONN_01X01 J?
+U 1 1 599E7936
+P 6950 4175
+F 0 "J?" H 6950 4275 50  0000 C CNN
+F 1 "Testpoint" V 7050 4175 50  0000 C CNN
+F 2 "library:Via-0.8mm" H 6950 4175 50  0001 C CNN
+F 3 "" H 6950 4175 50  0001 C CNN
+	1    6950 4175
+	1    0    0    -1
+$EndComp
+$Comp
+L CONN_01X01 J?
+U 1 1 599E7A18
+P 7100 1475
+F 0 "J?" H 7100 1575 50  0000 C CNN
+F 1 "Testpoint" V 7200 1475 50  0000 C CNN
+F 2 "library:Via-0.8mm" H 7100 1475 50  0001 C CNN
+F 3 "" H 7100 1475 50  0001 C CNN
+	1    7100 1475
+	1    0    0    -1
+$EndComp
+$Comp
+L CONN_01X01 J?
+U 1 1 599E8E3F
+P 5175 4200
+F 0 "J?" H 5175 4300 50  0000 C CNN
+F 1 "Testpoint" V 5275 4200 50  0000 C CNN
+F 2 "library:Via-0.8mm" H 5175 4200 50  0001 C CNN
+F 3 "" H 5175 4200 50  0001 C CNN
+	1    5175 4200
+	1    0    0    -1
+$EndComp
+$Comp
+L CONN_01X01 J?
+U 1 1 599E904A
+P 5275 1625
+F 0 "J?" H 5275 1725 50  0000 C CNN
+F 1 "Testpoint" V 5375 1625 50  0000 C CNN
+F 2 "library:Via-0.8mm" H 5275 1625 50  0001 C CNN
+F 3 "" H 5275 1625 50  0001 C CNN
+	1    5275 1625
+	1    0    0    -1
+$EndComp
 Wire Wire Line
 	7100 1775 7375 1775
@@
 Connection ~ 7175 2475
 Connection ~ 9300 1375
-NoConn ~ 8800 2175
-NoConn ~ 8800 2675
-NoConn ~ 8825 5000
-NoConn ~ 8825 5500
+Wire Wire Line
+	8275 1500 8275 1775
+Connection ~ 8275 1775
+Wire Wire Line
+	8225 4300 8225 4600
+Connection ~ 8225 4600
+Wire Wire Line
+	6900 1775 6900 1475
+Wire Wire Line
+	6750 4175 6675 4175
+Wire Wire Line
+	6675 4175 6675 4600
+Connection ~ 6675 4600
+Wire Wire Line
+	4975 4200 4975 4475
+Connection ~ 4975 4475
+Wire Wire Line
+	5075 1625 5075 1925
+Wire Wire Line
+	5075 1925 5100 1925
+Connection ~ 5100 1925
 $EndSCHEMATC

Commit message: Updated BOM and netlist
Parts:
- gave numbers to parts that had none: 6
Changed lines of the file:
@@
 $EndComp
 $Comp
-L PWR_FLAG #FLG036
+L PWR_FLAG #FLG701
 U 1 1 5969EEDC
 P 1875 4000
-F 0 "#FLG036" H 1875 4075 50  0001 C CNN
+F 0 "#FLG701" H 1875 4075 50  0001 C CNN
 F 1 "PWR_FLAG" H 1875 4150 50  0000 C CNN
 F 2 "" H 1875 4000 50  0001 C CNN
@@
 $EndComp
 $Comp
-L PWR_FLAG #FLG037
+L PWR_FLAG #FLG702
 U 1 1 5969F012
 P 1875 4950
-F 0 "#FLG037" H 1875 5025 50  0001 C CNN
+F 0 "#FLG702" H 1875 5025 50  0001 C CNN
 F 1 "PWR_FLAG" H 1875 5100 50  0000 C CNN
 F 2 "" H 1875 4950 50  0001 C CNN
@@
 NoConn ~ 8825 5500
 $Comp
-L CONN_01X01 J?
+L CONN_01X01 J706
 U 1 1 599E7444
 P 8475 1500
-F 0 "J?" H 8475 1600 50  0000 C CNN
+F 0 "J706" H 8475 1600 50  0000 C CNN
 F 1 "Testpoint" V 8575 1500 50  0000 C CNN
 F 2 "library:Via-0.8mm" H 8475 1500 50  0001 C CNN
@@
 $EndComp
 $Comp
-L CONN_01X01 J?
+L CONN_01X01 J705
 U 1 1 599E7723
 P 8425 4300
-F 0 "J?" H 8425 4400 50  0000 C CNN
+F 0 "J705" H 8425 4400 50  0000 C CNN
 F 1 "Testpoint" V 8525 4300 50  0000 C CNN
 F 2 "library:Via-0.8mm" H 8425 4300 50  0001 C CNN
@@
 $EndComp
 $Comp
-L CONN_01X01 J?
+L CONN_01X01 J703
 U 1 1 599E7936
 P 6950 4175
-F 0 "J?" H 6950 4275 50  0000 C CNN
+F 0 "J703" H 6950 4275 50  0000 C CNN
 F 1 "Testpoint" V 7050 4175 50  0000 C CNN
 F 2 "library:Via-0.8mm" H 6950 4175 50  0001 C CNN
@@
 $EndComp
 $Comp
-L CONN_01X01 J?
+L CONN_01X01 J704
 U 1 1 599E7A18
 P 7100 1475
-F 0 "J?" H 7100 1575 50  0000 C CNN
+F 0 "J704" H 7100 1575 50  0000 C CNN
 F 1 "Testpoint" V 7200 1475 50  0000 C CNN
 F 2 "library:Via-0.8mm" H 7100 1475 50  0001 C CNN
@@
 $EndComp
 $Comp
-L CONN_01X01 J?
+L CONN_01X01 J701
 U 1 1 599E8E3F
 P 5175 4200
-F 0 "J?" H 5175 4300 50  0000 C CNN
+F 0 "J701" H 5175 4300 50  0000 C CNN
 F 1 "Testpoint" V 5275 4200 50  0000 C CNN
 F 2 "library:Via-0.8mm" H 5175 4200 50  0001 C CNN
@@
 $EndComp
 $Comp
-L CONN_01X01 J?
+L CONN_01X01 J702
 U 1 1 599E904A
 P 5275 1625
-F 0 "J?" H 5275 1725 50  0000 C CNN
+F 0 "J702" H 5275 1725 50  0000 C CNN
 F 1 "Testpoint" V 5375 1625 50  0000 C CNN
 F 2 "library:Via-0.8mm" H 5275 1625 50  0001 C CNN

Commit message: DRC
Parts:
- J701, J702, J703, J704, J705, J706: footprint library:Via-0.8mm -> library:TestPoint
Changed lines of the file:
@@
 F 0 "J706" H 8475 1600 50  0000 C CNN
 F 1 "Testpoint" V 8575 1500 50  0000 C CNN
-F 2 "library:Via-0.8mm" H 8475 1500 50  0001 C CNN
+F 2 "library:TestPoint" H 8475 1500 50  0001 C CNN
 F 3 "" H 8475 1500 50  0001 C CNN
 	1    8475 1500
@@
 F 0 "J705" H 8425 4400 50  0000 C CNN
 F 1 "Testpoint" V 8525 4300 50  0000 C CNN
-F 2 "library:Via-0.8mm" H 8425 4300 50  0001 C CNN
+F 2 "library:TestPoint" H 8425 4300 50  0001 C CNN
 F 3 "" H 8425 4300 50  0001 C CNN
 	1    8425 4300
@@
 F 0 "J703" H 6950 4275 50  0000 C CNN
 F 1 "Testpoint" V 7050 4175 50  0000 C CNN
-F 2 "library:Via-0.8mm" H 6950 4175 50  0001 C CNN
+F 2 "library:TestPoint" H 6950 4175 50  0001 C CNN
 F 3 "" H 6950 4175 50  0001 C CNN
 	1    6950 4175
@@
 F 0 "J704" H 7100 1575 50  0000 C CNN
 F 1 "Testpoint" V 7200 1475 50  0000 C CNN
-F 2 "library:Via-0.8mm" H 7100 1475 50  0001 C CNN
+F 2 "library:TestPoint" H 7100 1475 50  0001 C CNN
 F 3 "" H 7100 1475 50  0001 C CNN
 	1    7100 1475
@@
 F 0 "J701" H 5175 4300 50  0000 C CNN
 F 1 "Testpoint" V 5275 4200 50  0000 C CNN
-F 2 "library:Via-0.8mm" H 5175 4200 50  0001 C CNN
+F 2 "library:TestPoint" H 5175 4200 50  0001 C CNN
 F 3 "" H 5175 4200 50  0001 C CNN
 	1    5175 4200
@@
 F 0 "J702" H 5275 1725 50  0000 C CNN
 F 1 "Testpoint" V 5375 1625 50  0000 C CNN
-F 2 "library:Via-0.8mm" H 5275 1625 50  0001 C CNN
+F 2 "library:TestPoint" H 5275 1625 50  0001 C CNN
 F 3 "" H 5275 1625 50  0001 C CNN
 	1    5275 1625
