File: ADC.sch (KiCad schematic (older format))
At the start: 51 parts, among them J701 Testpoint, J702 Testpoint, J705 Testpoint, J706 Testpoint, U1001 ADC1175, U1002 ADC1175

Commit message: New BOM generated with kicost
Parts:
- J701, J702, J705, J706: DNP (none) -> 1

Commit message: changed ref of adc (2.5V-->2V), and Rf of last amp stage (62K-->51K)
Parts:
- D1001: value LM4040DYM3-2.5-TR -> LM4040D; MPN LM4040DYM3-2.5-TR -> LM4040D20IDBZR; Vref 2.5V -> 2V
- D1003: value LM4040DYM3-2.5-TR -> LM4040; MPN LM4040DYM3-2.5-TR -> LM4040D20IDBZR; Vref 2.5V -> 2V
- L1003, L1004, L1006, L1007: value L_BLM18AG121SN1D -> Choke
- R1003: value 220R -> 220
Changed lines of the file:
@@
 U 1 1 58FEC865
 P 7700 4800
-F 0 "D1006" V 7700 4625 50  0000 L CNN
-F 1 "D_Schottky_BAT54S-7-F" H 7300 4975 50  0000 L CNN
+F 0 "D1006" H 7650 4675 50  0000 L CNN
+F 1 "D_Schottky_BAT54S-7-F" H 7425 4950 50  0000 L CNN
 F 2 "TO_SOT_Packages_SMD:SOT-23" H 4450 3400 50  0001 C CNN
 F 3 "http://ar.mouser.com/ProductDetail/ON-Semiconductor-Fairchild/BAT54S/?qs=sGAEpiMZZMtQ8nqTKtFS%2fIwmNNVNDRcYUrXGPe5oOTQ%3d" H 4450 4100 50  0001 C CNN
@@
 U 1 1 5913A0F9
 P 3875 6900
-F 0 "D1002" H 3875 7000 50  0000 C CNN
+F 0 "D1002" H 3950 7025 50  0000 C CNN
 F 1 "LM4041EIM3-1.2/NOPB" H 3875 6700 50  0000 C CNN
 F 2 "TO_SOT_Packages_SMD:SOT-23" H 3825 6400 50  0001 C CNN
@@
 U 1 1 5917F07E
 P 3825 4650
-F 0 "D1001" H 3825 4550 50  0000 L CNN
-F 1 "LM4040DYM3-2.5-TR" H 3475 4450 50  0000 L CNN
+F 0 "D1001" H 3775 4775 50  0000 L CNN
+F 1 "LM4040D" H 3725 4525 50  0000 L CNN
 F 2 "TO_SOT_Packages_SMD:SOT-23" H -625 -1135 50  0001 C CNN
-F 3 "http://www.microchip.com/mymicrochip/filehandler.aspx?ddocname=en579040" H -475 -1525 50  0001 C CNN
+F 3 "http://www.ti.com/lit/ds/slos456k/slos456k.pdf" H -475 -1525 50  0001 C CNN
 F 4 "65uA < I < 15mA" H 3400 4475 60  0001 L CNN "Irange"
-F 5 "LM4040DYM3-2.5-TR" H 3825 4650 50  0001 C CNN "MPN"
-F 6 "2.5V" H 3725 4375 60  0001 L CNN "Vref"
+F 5 "LM4040D20IDBZR" H 3825 4650 50  0001 C CNN "MPN"
+F 6 "2V" H 3725 4375 60  0001 L CNN "Vref"
 	1    3825 4650
 	0    1    1    0
@@
 U 1 1 591802E2
 P 3925 2100
-F 0 "D1003" H 3950 2000 50  0000 L CNN
-F 1 "LM4040DYM3-2.5-TR" H 3575 1900 50  0000 L CNN
+F 0 "D1003" H 3875 2200 50  0000 L CNN
+F 1 "LM4040" H 3850 1975 50  0000 L CNN
 F 2 "TO_SOT_Packages_SMD:SOT-23" H -525 -3685 50  0001 C CNN
-F 3 "http://www.microchip.com/mymicrochip/filehandler.aspx?ddocname=en579040" H -375 -4075 50  0001 C CNN
+F 3 "http://www.ti.com/lit/ds/slos456k/slos456k.pdf" H -375 -4075 50  0001 C CNN
 F 4 "65uA < I < 15mA" H 3500 1925 60  0001 L CNN "Irange"
-F 5 "LM4040DYM3-2.5-TR" H 3950 2100 50  0001 C CNN "MPN"
-F 6 "2.5V" H 3825 1825 60  0001 L CNN "Vref"
+F 5 "LM4040D20IDBZR" H 3950 2100 50  0001 C CNN "MPN"
+F 6 "2V" H 3825 1825 60  0001 L CNN "Vref"
 	1    3925 2100
 	0    1    1    0
@@
 P 4050 4475
 F 0 "L1003" V 4000 4425 50  0000 C CNN
-F 1 "L_BLM18AG121SN1D" V 4175 4225 50  0000 C CNN
+F 1 "Choke" V 4150 4400 50  0000 C CNN
 F 2 "Inductors_SMD:L_0603_HandSoldering" H -850 3775 50  0001 C CNN
 F 3 "http://www.mouser.com/ds/2/281/c31e-794748.pdf" H -850 3775 50  0001 C CNN
@@
 U 1 1 595E0CF6
 P 4050 5000
-F 0 "L1004" V 4250 5150 50  0000 C CNN
-F 1 "L_BLM18AG121SN1D" V 4150 5025 50  0000 C CNN
+F 0 "L1004" V 4150 4925 50  0000 C CNN
+F 1 "Choke" V 3975 5025 50  0000 C CNN
 F 2 "Inductors_SMD:L_0603_HandSoldering" H -850 4300 50  0001 C CNN
 F 3 "http://www.mouser.com/ds/2/281/c31e-794748.pdf" H -850 4300 50  0001 C CNN
@@
 U 1 1 595E1E1C
 P 4100 6675
-F 0 "L1005" V 4325 6700 50  0000 C CNN
-F 1 "L_BLM18AG121SN1D" V 4225 6400 50  0000 C CNN
+F 0 "L1005" V 4025 6625 50  0000 C CNN
+F 1 "L_BLM18AG121SN1D" V 4200 6400 50  0000 C CNN
 F 2 "Inductors_SMD:L_0603_HandSoldering" H -800 5975 50  0001 C CNN
 F 3 "http://www.mouser.com/ds/2/281/c31e-794748.pdf" H -800 5975 50  0001 C CNN
@@
 P 4475 6900
 F 0 "C1015" V 4550 7000 50  0000 C CNN
-F 1 "10uF" V 4525 6775 50  0000 C CNN
+F 1 "10uF" V 4425 6750 50  0000 C CNN
 F 2 "Capacitors_SMD:C_1206_HandSoldering" H -175 5950 50  0001 C CNN
 F 3 "http://www.mouser.com/ds/2/40/TAJ_AUTO-783622.pdf" H -175 5950 50  0001 C CNN
@@
 U 1 1 595E201B
 P 4750 6875
-F 0 "C1018" V 4625 6775 50  0000 C CNN
-F 1 "100nF" V 4575 7025 50  0000 C CNN
+F 0 "C1018" V 4650 6800 50  0000 C CNN
+F 1 "100nF" V 4800 7025 50  0000 C CNN
 F 2 "Capacitors_SMD:C_0603_HandSoldering" H 550 5900 50  0001 C CNN
 F 3 "http://www.mouser.com/ds/2/212/KEM_C1002_X7R_SMD-357932.pdf" H 550 5900 50  0001 C CNN
@@
 U 1 1 595E2F88
 P 4150 2450
-F 0 "L1007" V 4100 2350 50  0000 C CNN
-F 1 "L_BLM18AG121SN1D" V 4250 2300 50  0000 C CNN
+F 0 "L1007" V 4075 2450 50  0000 C CNN
+F 1 "Choke" V 4250 2425 50  0000 C CNN
 F 2 "Inductors_SMD:L_0603_HandSoldering" H -750 1750 50  0001 C CNN
 F 3 "http://www.mouser.com/ds/2/281/c31e-794748.pdf" H -750 1750 50  0001 C CNN
@@
 P 4150 1925
 F 0 "L1006" V 4100 1875 50  0000 C CNN
-F 1 "L_BLM18AG121SN1D" V 4250 1725 50  0000 C CNN
+F 1 "Choke" V 4250 1875 50  0000 C CNN
 F 2 "Inductors_SMD:L_0603_HandSoldering" H -750 1225 50  0001 C CNN
 F 3 "http://www.mouser.com/ds/2/281/c31e-794748.pdf" H -750 1225 50  0001 C CNN
@@
 U 1 1 595F9240
 P 3875 6500
-F 0 "R1003" V 3775 6450 50  0000 L CNN
-F 1 "220R" V 3975 6325 50  0000 L CNN
+F 0 "R1003" V 3800 6275 50  0000 L CNN
+F 1 "220" V 3950 6400 50  0000 L CNN
 F 2 "Resistors_SMD:R_0603_HandSoldering" H 3875 6500 50  0001 C CNN
 F 3 "http://www.mouser.com/ds/2/447/RC0603-272842.pdf" H 3875 6500 50  0001 C CNN
