File: Attenuation.sch (KiCad schematic (older format))
At the start: 26 parts, among them U201 CPC1017N, U202 CPC1017N, U203 CD4051BM96, U204 CD4051BM96

Commit message: Completed part selection of analog board. Merged analog and digital boards.
Parts:
- removed C201, C202: 100p, Capacitors_SMD:C_0603_HandSoldering, symbol C
- removed C203, C206: 22p, Capacitors_SMD:C_0603_HandSoldering, symbol C
- removed C204, C207: 0.56-3.58p, Capacitors_SMD:C_0603_HandSoldering, symbol C_Variable
- removed C205, C208: 5-20pF, Capacitors_SMD:C_0603_HandSoldering, symbol C_Variable
- removed C209, C211: 180p, Capacitors_SMD:C_0603_HandSoldering, symbol C
- removed C210, C212: 1800p, Capacitors_SMD:C_0603_HandSoldering, symbol C
- removed D201, D202: D_Schottky_BAT54S-7-F, TO_SOT_Packages_SMD:SOT-23, symbol D_Schottky_BAT54S-7-F
- removed R201, R205: 13k, Resistors_SMD:R_0603_HandSoldering, symbol R
- removed R202, R206: 887k, Resistors_SMD:R_0603_HandSoldering, symbol R
- removed R203, R207: 89.8k, Resistors_SMD:R_0603_HandSoldering, symbol R
- removed R204, R208: 10k, Resistors_SMD:R_0603_HandSoldering, symbol R
- removed U201, U202: CPC1017N, library:2.54SOP4, symbol CPC1017N
- removed U203, U204: CD4051BM96, Housings_SOIC:SOIC-16_3.9x9.9mm_Pitch1.27mm, symbol CD4051BM96
- added C701, C702: 100p, Capacitors_SMD:C_0603_HandSoldering, symbol C
- added C703, C706: 22p, Capacitors_SMD:C_0603_HandSoldering, symbol C
- added C704, C707: 0.56-3.58p, Capacitors_SMD:C_0603_HandSoldering, symbol C_Variable
- added C705, C708: 5-20pF, Capacitors_SMD:C_0603_HandSoldering, symbol C_Variable
- added C709, C711: 180p, Capacitors_SMD:C_0603_HandSoldering, symbol C
- added C710, C712: 1800p, Capacitors_SMD:C_0603_HandSoldering, symbol C
- added D701, D702: D_Schottky_BAT54S-7-F, TO_SOT_Packages_SMD:SOT-23, symbol D_Schottky_BAT54S-7-F
- added R701, R705: 13k, Resistors_SMD:R_0603_HandSoldering, symbol R
- added R702, R706: 887k, Resistors_SMD:R_0603_HandSoldering, symbol R
- added R703, R707: 89.8k, Resistors_SMD:R_0603_HandSoldering, symbol R
- added R704, R708: 10k, Resistors_SMD:R_0603_HandSoldering, symbol R
- added U701, U702: CPC1017N, library:2.54SOP4, symbol CPC1017N
- added U703, U704: CD4051BM96, Housings_SOIC:SOIC-16_3.9x9.9mm_Pitch1.27mm, symbol CD4051BM96

Commit message: No more DRC errors :)
Changed lines of the file:
@@
 VDD_A
 $Comp
-L GNDA #PWR025
+L GNDA #PWR029
 U 1 1 5965C32C
 P 8700 1550
-F 0 "#PWR025" H 8700 1300 50  0001 C CNN
+F 0 "#PWR029" H 8700 1300 50  0001 C CNN
 F 1 "GNDA" V 8700 1300 50  0000 C CNN
 F 2 "" H 8700 1550 50  0001 C CNN
@@
 CHB_OFFSET
 $Comp
-L GNDA #PWR026
+L GNDA #PWR030
 U 1 1 5965C32D
 P 8700 1450
-F 0 "#PWR026" H 8700 1200 50  0001 C CNN
+F 0 "#PWR030" H 8700 1200 50  0001 C CNN
 F 1 "GNDA" V 8700 1200 50  0000 C CNN
 F 2 "" H 8700 1450 50  0001 C CNN
@@
 $EndComp
 $Comp
-L GNDA #PWR027
+L GNDA #PWR031
 U 1 1 5965C32E
 P 8700 1650
-F 0 "#PWR027" H 8700 1400 50  0001 C CNN
+F 0 "#PWR031" H 8700 1400 50  0001 C CNN
 F 1 "GNDA" V 8700 1400 50  0000 C CNN
 F 2 "" H 8700 1650 50  0001 C CNN
@@
 $EndComp
 $Comp
-L GNDA #PWR028
+L GNDA #PWR032
 U 1 1 5965C32F
 P 8700 1750
-F 0 "#PWR028" H 8700 1500 50  0001 C CNN
+F 0 "#PWR032" H 8700 1500 50  0001 C CNN
 F 1 "GNDA" V 8700 1500 50  0000 C CNN
 F 2 "" H 8700 1750 50  0001 C CNN
@@
 $EndComp
 $Comp
-L GNDA #PWR029
+L GNDA #PWR033
 U 1 1 5965C330
 P 8700 1850
-F 0 "#PWR029" H 8700 1600 50  0001 C CNN
+F 0 "#PWR033" H 8700 1600 50  0001 C CNN
 F 1 "GNDA" V 8700 1600 50  0000 C CNN
 F 2 "" H 8700 1850 50  0001 C CNN
@@
 $EndComp
 $Comp
-L GNDA #PWR030
+L GNDA #PWR034
 U 1 1 5965C332
 P 8725 4275
-F 0 "#PWR030" H 8725 4025 50  0001 C CNN
+F 0 "#PWR034" H 8725 4025 50  0001 C CNN
 F 1 "GNDA" V 8725 4025 50  0000 C CNN
 F 2 "" H 8725 4275 50  0001 C CNN
@@
 CHA_OFFSET
 $Comp
-L GNDA #PWR031
+L GNDA #PWR035
 U 1 1 5965C333
 P 8725 4175
-F 0 "#PWR031" H 8725 3925 50  0001 C CNN
+F 0 "#PWR035" H 8725 3925 50  0001 C CNN
 F 1 "GNDA" V 8725 3925 50  0000 C CNN
 F 2 "" H 8725 4175 50  0001 C CNN
@@
 $EndComp
 $Comp
-L GNDA #PWR032
+L GNDA #PWR036
 U 1 1 5965C334
 P 8725 4375
-F 0 "#PWR032" H 8725 4125 50  0001 C CNN
+F 0 "#PWR036" H 8725 4125 50  0001 C CNN
 F 1 "GNDA" V 8725 4125 50  0000 C CNN
 F 2 "" H 8725 4375 50  0001 C CNN
@@
 $EndComp
 $Comp
-L GNDA #PWR033
+L GNDA #PWR037
 U 1 1 5965C335
 P 8725 4475
-F 0 "#PWR033" H 8725 4225 50  0001 C CNN
+F 0 "#PWR037" H 8725 4225 50  0001 C CNN
 F 1 "GNDA" V 8725 4225 50  0000 C CNN
 F 2 "" H 8725 4475 50  0001 C CNN
@@
 $EndComp
 $Comp
-L GNDA #PWR034
+L GNDA #PWR038
 U 1 1 5965C336
 P 8725 4575
-F 0 "#PWR034" H 8725 4325 50  0001 C CNN
+F 0 "#PWR038" H 8725 4325 50  0001 C CNN
 F 1 "GNDA" V 8725 4325 50  0000 C CNN
 F 2 "" H 8725 4575 50  0001 C CNN
@@
 Text Label 9425 5375 3    60   ~ 0
 VSS_A
-Text Label 6775 4775 0    60   ~ 0
+Text Label 6800 4800 0    60   ~ 0
 VSS_A
 Text Label 6775 3850 0    60   ~ 0
@@
 	6700 3850 6700 4050
 Wire Wire Line
-	6675 4700 6750 4700
-Wire Wire Line
 	6225 4300 6925 4300
 Connection ~ 6600 4300
-Wire Wire Line
-	6700 4775 6700 4650
 Wire Wire Line
 	3950 4650 4150 4650
@@
 	0    1    1    0
 $EndComp
+Wire Wire Line
+	6700 4800 6800 4800
+Wire Wire Line
+	6700 4650 6700 4800
 $EndSCHEMATC

Commit message: Continued with routing...
Parts:
- added C713, C714: Optional, Capacitors_SMD:C_0603_HandSoldering, symbol C_Variable
- added R709, R710: 0, Resistors_SMD:R_0603_HandSoldering, symbol R_Small
Connections:
- wire segments 56 -> 61
Other:
- moved on the sheet: C701, C702, C703, C706, C709, C710, C711, C712, R701, R702, R703, R704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

Commit message: Ended placing (?)
Parts:
- added J701, J702: CONN_01X01, Pin_Headers:Pin_Header_Straight_1x01_Pitch1.27mm, symbol CONN_01X01
Connections:
- net labels removed: CHA_OFFSET, CHB_OFFSET
- wire segments 61 -> 63
Other:
- note added: "Test Point. \nConnect to channel offset A."
- note added: "Test Point. \nConnect to channel offset B."
Changed lines of the file:
@@
 	0    1    1    0
 $EndComp
-Text HLabel 8700 1350 0    60   Input ~ 0
-CHB_OFFSET
 $Comp
 L GNDA #PWR030
@@
 	0    1    1    0
 $EndComp
-Text HLabel 8725 4075 0    60   Input ~ 0
-CHA_OFFSET
 $Comp
 L GNDA #PWR035
@@
 Wire Wire Line
 	5100 4400 5100 4600
+$Comp
+L CONN_01X01 J701
+U 1 1 596A5B58
+P 7800 1350
+F 0 "J701" H 7800 1450 50  0000 C CNN
+F 1 "CONN_01X01" V 7900 1350 50  0000 C CNN
+F 2 "Pin_Headers:Pin_Header_Straight_1x01_Pitch1.27mm" H 7800 1350 50  0001 C CNN
+F 3 "" H 7800 1350 50  0001 C CNN
+	1    7800 1350
+	-1   0    0    1
+$EndComp
+Wire Wire Line
+	8000 1350 8700 1350
+$Comp
+L CONN_01X01 J702
+U 1 1 596A6054
+P 7925 4075
+F 0 "J702" H 7925 4175 50  0000 C CNN
+F 1 "CONN_01X01" V 8025 4075 50  0000 C CNN
+F 2 "Pin_Headers:Pin_Header_Straight_1x01_Pitch1.27mm" H 7925 4075 50  0001 C CNN
+F 3 "" H 7925 4075 50  0001 C CNN
+	1    7925 4075
+	-1   0    0    1
+$EndComp
+Wire Wire Line
+	8125 4075 8725 4075
+Text Notes 7000 1700 0    60   ~ 0
+Test Point. \nConnect to channel offset B.
+Text Notes 7050 4400 0    60   ~ 0
+Test Point. \nConnect to channel offset A.
 $EndSCHEMATC
