File: Attenuation.sch (KiCad schematic (older format))
At the start: 32 parts, among them J701 CONN_01X01, J702 CONN_01X01, U701 CPC1017N, U702 CPC1017N, U703 CD4051BM96, U704 CD4051BM96

Commit message: Modified a lot of fields in components parts. BOM generated. Added BOM plugin script.
Parts:
- removed J701, J702: CONN_01X01, Pin_Headers:Pin_Header_Straight_1x01_Pitch1.27mm, symbol CONN_01X01
- added J601, J602: CONN_01X02, Pin_Headers:Pin_Header_Angled_1x02_Pitch1.27mm, symbol CONN_01X02
- C701, C702: value 100p -> 100pF; Dielectric (none) -> C0G; MPN (none) -> VJ0603A101JXACW1BC; Manufacturer Part VJ0603A101JXACW1BC -> (none); Type (none) -> Ceramic; VDC (none) -> 50V
- C703, C706: value 22p -> 22pF; Dielectric (none) -> C0G; MPN (none) -> 06031U220FAT2A; Manufacturer Part 06031U220FAT2A -> (none); Type (none) -> Ceramic; VDC (none) -> 100V
- C704, C707: MPN (none) -> STPTIC-27L2C5; Manufacturer Part STPTIC-27L2C5 -> (none)
- C705, C708: MPN (none) -> GKG20015; Manufacturer Part GKG20015 -> (none)
- C709, C711: Dielectric (none) -> C0G; MPN (none) -> VJ0603A181FXXPW1BC; Manufacturer Part VJ0603A181FXXPW1BC -> (none); Type (none) -> Ceramic; VDC (none) -> 25V
- C710, C712: Dielectric (none) -> C0G; MPN (none) -> GCM1885C1H182FA16D; Manufacturer Part GCM1885C1H182FA16D -> (none); Type (none) -> Ceramic; VDC (none) -> 50V
- C713, C714: value Optional -> Not used
- D701, D702: Link Digikey https://www.digikey.com/product-detail/en/diodes-incorporat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 -> (none); MPN (none) -> BAT54S-7-F; Manuf. Part Number BAT54S-7-F -> (none); Price $0.21 -> (none)
- R701, R705: MPN (none) -> RC0603FR-0713KL; Manufacturer Part RC0603FR-0713KL -> (none)
- R702, R706: value 887k -> 887K; MPN (none) -> RC0603FR-07887KL; Manufacturer Part RC0603FR-07887KL -> (none)
- R703, R707: value 89.8k -> 89K8; MPN (none) -> RT0603DRE0789K8L; Manufacturer Part RT0603DRE0789K8L -> (none)
- R704, R708: value 10k -> 10K; MPN (none) -> RT0603DRE0710KL; Manufacturer Part RT0603DRE0710KL -> (none)
- R709, R710: value 0 -> 0R; MPN (none) -> RC1206JR-070RL; Manufacturer Part RC1206JR-070RL -> (none)
- U701, U702: Link Mouser http://www.mouser.com/ProductDetail/IXYS-Integrated-Circuit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 -> (none); MPN (none) -> CPC1017N; Manuf. Part Number CPC1017NTR -> (none); Price $1.05 -> (none)
- U703, U704: MPN (none) -> CD4051BM96; Manuf. Part Number CD4051BM96 -> (none)
Connections:
- wire segments 63 -> 65

Commit message: Changed some MPN and footprints. BOM updated.
Parts:
- R701, R705: value 13k -> 13K

Commit message: Changed trimmer caps MPN and footprints
Parts:
- C704, C707: value 0.56-3.58p -> 1-3pF; footprint Capacitors_SMD:C_0603_HandSoldering -> Capacitors_THT:CP_Radial_Tantal_D6.0mm_P5.00mm; MPN STPTIC-27L2C5 -> GKG3R015
- C705, C708, C713, C714: footprint Capacitors_SMD:C_0603_HandSoldering -> Capacitors_THT:CP_Radial_Tantal_D6.0mm_P5.00mm
Changed lines of the file:
@@
 $Descr A4 11693 8268
 encoding utf-8
-Sheet 6 11
+Sheet 4 11
 Title ""
 Date ""
@@
 F 0 "C705" H 4725 3250 50  0000 L CNN
 F 1 "5-20pF" H 4725 3175 50  0000 L CNN
-F 2 "Capacitors_SMD:C_0603_HandSoldering" H 4700 3325 50  0001 C CNN
+F 2 "Capacitors_THT:CP_Radial_Tantal_D6.0mm_P5.00mm" H 4700 3325 50  0001 C CNN
 F 3 "http://www.mouser.com/ds/2/384/659305J-204462.pdf" H 4700 3325 50  0001 C CNN
 F 4 "GKG20015" H 4725 3350 50  0001 C CNN "MPN"
@@
 P 4700 2500
 F 0 "C704" H 4725 2425 50  0000 L CNN
-F 1 "0.56-3.58p" H 4725 2350 50  0000 L CNN
-F 2 "Capacitors_SMD:C_0603_HandSoldering" H 4700 2500 50  0001 C CNN
-F 3 "http://www.mouser.com/ds/2/389/stptic-27l2-956732.pdf" H 4700 2500 50  0001 C CNN
-F 4 "STPTIC-27L2C5" H 4725 2525 50  0001 C CNN "MPN"
+F 1 "1-3pF" H 4725 2350 50  0000 L CNN
+F 2 "Capacitors_THT:CP_Radial_Tantal_D6.0mm_P5.00mm" H 4700 2500 50  0001 C CNN
+F 3 "http://www.mouser.com/ds/2/384/659305J-204462.pdf" H 4700 2500 50  0001 C CNN
+F 4 "GKG3R015" H 4725 2525 50  0001 C CNN "MPN"
 	1    4700 2500
 	1    0    0    -1
@@
 F 0 "C708" H 4600 6150 50  0000 L CNN
 F 1 "5-20pF" H 4600 6075 50  0000 L CNN
-F 2 "Capacitors_SMD:C_0603_HandSoldering" H 4575 6225 50  0001 C CNN
+F 2 "Capacitors_THT:CP_Radial_Tantal_D6.0mm_P5.00mm" H 4575 6225 50  0001 C CNN
 F 3 "http://www.mouser.com/ds/2/384/659305J-204462.pdf" H 4575 6225 50  0001 C CNN
 F 4 "GKG20015" H 4600 6250 50  0001 C CNN "MPN"
@@
 P 4575 5350
 F 0 "C707" H 4600 5275 50  0000 L CNN
-F 1 "0.56-3.58p" H 4600 5200 50  0000 L CNN
-F 2 "Capacitors_SMD:C_0603_HandSoldering" H 4575 5350 50  0001 C CNN
-F 3 "http://www.mouser.com/ds/2/389/stptic-27l2-956732.pdf" H 4575 5350 50  0001 C CNN
-F 4 "STPTIC-27L2C5" H 4600 5375 50  0001 C CNN "MPN"
+F 1 "1-3pF" H 4600 5200 50  0000 L CNN
+F 2 "Capacitors_THT:CP_Radial_Tantal_D6.0mm_P5.00mm" H 4575 5350 50  0001 C CNN
+F 3 "http://www.mouser.com/ds/2/384/659305J-204462.pdf" H 4575 5350 50  0001 C CNN
+F 4 "GKG3R015" H 4600 5375 50  0001 C CNN "MPN"
 	1    4575 5350
 	1    0    0    -1
@@
 F 0 "C714" H 4725 1775 50  0000 L CNN
 F 1 "Not used" H 4725 1700 50  0000 L CNN
-F 2 "Capacitors_SMD:C_0603_HandSoldering" H 4700 1850 50  0001 C CNN
+F 2 "Capacitors_THT:CP_Radial_Tantal_D6.0mm_P5.00mm" H 4700 1850 50  0001 C CNN
 F 3 "" H 4700 1850 50  0001 C CNN
 	1    4700 1850
@@
 F 0 "C713" H 4600 4650 50  0000 L CNN
 F 1 "Not used" H 4600 4575 50  0000 L CNN
-F 2 "Capacitors_SMD:C_0603_HandSoldering" H 4575 4725 50  0001 C CNN
+F 2 "Capacitors_THT:CP_Radial_Tantal_D6.0mm_P5.00mm" H 4575 4725 50  0001 C CNN
 F 3 "" H 4575 4725 50  0001 C CNN
 	1    4575 4725

Commit message: Added testpoints to schematic.
Parts:
- added J? (x6): Testpoint, library:Via-0.8mm, symbol CONN_01X01
Connections:
- wire segments 65 -> 75
Changed lines of the file:
@@
 Text HLabel 2825 4275 0    60   Input ~ 0
 CHB_IN
-Text HLabel 9800 1300 2    60   Input ~ 0
+Text HLabel 9925 1300 2    60   Input ~ 0
 CHA_OUT
-Text HLabel 9825 4025 2    60   Input ~ 0
+Text HLabel 10025 4025 2    60   Input ~ 0
 CHB_OUT
 Text HLabel 2950 2275 0    60   Input ~ 0
@@
 Text Label 8200 4175 3    60   ~ 0
 GND_A
+$Comp
+L CONN_01X01 J?
+U 1 1 599EC0AF
+P 10025 1600
+F 0 "J?" H 10025 1700 50  0000 C CNN
+F 1 "Testpoint" V 10125 1600 50  0000 C CNN
+F 2 "library:Via-0.8mm" H 10025 1600 50  0001 C CNN
+F 3 "" H 10025 1600 50  0001 C CNN
+	1    10025 1600
+	1    0    0    -1
+$EndComp
+$Comp
+L CONN_01X01 J?
+U 1 1 599EC0FA
+P 10150 3725
+F 0 "J?" H 10150 3825 50  0000 C CNN
+F 1 "Testpoint" V 10250 3725 50  0000 C CNN
+F 2 "library:Via-0.8mm" H 10150 3725 50  0001 C CNN
+F 3 "" H 10150 3725 50  0001 C CNN
+	1    10150 3725
+	1    0    0    -1
+$EndComp
+$Comp
+L CONN_01X01 J?
+U 1 1 599EC1CA
+P 5825 4325
+F 0 "J?" H 5825 4425 50  0000 C CNN
+F 1 "Testpoint" V 5925 4325 50  0000 C CNN
+F 2 "library:Via-0.8mm" H 5825 4325 50  0001 C CNN
+F 3 "" H 5825 4325 50  0001 C CNN
+	1    5825 4325
+	1    0    0    -1
+$EndComp
+$Comp
+L CONN_01X01 J?
+U 1 1 599EC2EF
+P 5675 6200
+F 0 "J?" H 5675 6300 50  0000 C CNN
+F 1 "Testpoint" V 5775 6200 50  0000 C CNN
+F 2 "library:Via-0.8mm" H 5675 6200 50  0001 C CNN
+F 3 "" H 5675 6200 50  0001 C CNN
+	1    5675 6200
+	1    0    0    -1
+$EndComp
+$Comp
+L CONN_01X01 J?
+U 1 1 599EC39F
+P 5950 3200
+F 0 "J?" H 5950 3300 50  0000 C CNN
+F 1 "Testpoint" V 6050 3200 50  0000 C CNN
+F 2 "library:Via-0.8mm" H 5950 3200 50  0001 C CNN
+F 3 "" H 5950 3200 50  0001 C CNN
+	1    5950 3200
+	1    0    0    -1
+$EndComp
+$Comp
+L CONN_01X01 J?
+U 1 1 599EC468
+P 5850 1975
+F 0 "J?" H 5850 2075 50  0000 C CNN
+F 1 "Testpoint" V 5950 1975 50  0000 C CNN
+F 2 "library:Via-0.8mm" H 5850 1975 50  0001 C CNN
+F 3 "" H 5850 1975 50  0001 C CNN
+	1    5850 1975
+	1    0    0    -1
+$EndComp
 Wire Wire Line
 	4500 1550 5225 1550
@@
 	5100 5500 5100 6075
 Wire Wire Line
-	4375 5950 5350 5950
+	4375 5950 5475 5950
 Wire Wire Line
 	5100 4900 5100 5200
@@
 Connection ~ 4700 1550
 Connection ~ 4575 4400
+Wire Wire Line
+	5650 1975 5650 2275
+Wire Wire Line
+	5650 2275 5675 2275
+Connection ~ 5675 2275
+Wire Wire Line
+	5475 5950 5475 6200
+Wire Wire Line
+	5625 4325 5625 5125
+Connection ~ 5625 5125
+Wire Wire Line
+	5750 3200 5475 3200
+Wire Wire Line
+	5475 3200 5475 3050
+Wire Wire Line
+	9800 1300 9925 1300
+Wire Wire Line
+	9825 1600 9825 1300
+Connection ~ 9825 1300
+Wire Wire Line
+	9825 4025 10025 4025
+Wire Wire Line
+	9950 3725 9950 4025
+Connection ~ 9950 4025
 $EndSCHEMATC

Commit message: Updated BOM and netlist
Parts:
- gave numbers to parts that had none: 6
Changed lines of the file:
@@
 $EndComp
 $Comp
-L GNDA #PWR026
+L GNDA #PWR402
 U 1 1 5965C32C
 P 8700 1550
-F 0 "#PWR026" H 8700 1300 50  0001 C CNN
+F 0 "#PWR402" H 8700 1300 50  0001 C CNN
 F 1 "GNDA" V 8700 1300 50  0000 C CNN
 F 2 "" H 8700 1550 50  0001 C CNN
@@
 $EndComp
 $Comp
-L GNDA #PWR027
+L GNDA #PWR401
 U 1 1 5965C32D
 P 8700 1450
-F 0 "#PWR027" H 8700 1200 50  0001 C CNN
+F 0 "#PWR401" H 8700 1200 50  0001 C CNN
 F 1 "GNDA" V 8700 1200 50  0000 C CNN
 F 2 "" H 8700 1450 50  0001 C CNN
@@
 $EndComp
 $Comp
-L GNDA #PWR028
+L GNDA #PWR403
 U 1 1 5965C32E
 P 8700 1650
-F 0 "#PWR028" H 8700 1400 50  0001 C CNN
+F 0 "#PWR403" H 8700 1400 50  0001 C CNN
 F 1 "GNDA" V 8700 1400 50  0000 C CNN
 F 2 "" H 8700 1650 50  0001 C CNN
@@
 $EndComp
 $Comp
-L GNDA #PWR029
+L GNDA #PWR404
 U 1 1 5965C32F
 P 8700 1750
-F 0 "#PWR029" H 8700 1500 50  0001 C CNN
+F 0 "#PWR404" H 8700 1500 50  0001 C CNN
 F 1 "GNDA" V 8700 1500 50  0000 C CNN
 F 2 "" H 8700 1750 50  0001 C CNN
@@
 $EndComp
 $Comp
-L GNDA #PWR030
+L GNDA #PWR405
 U 1 1 5965C330
 P 8700 1850
-F 0 "#PWR030" H 8700 1600 50  0001 C CNN
+F 0 "#PWR405" H 8700 1600 50  0001 C CNN
 F 1 "GNDA" V 8700 1600 50  0000 C CNN
 F 2 "" H 8700 1850 50  0001 C CNN
@@
 $EndComp
 $Comp
-L GNDA #PWR031
+L GNDA #PWR407
 U 1 1 5965C332
 P 8725 4275
-F 0 "#PWR031" H 8725 4025 50  0001 C CNN
+F 0 "#PWR407" H 8725 4025 50  0001 C CNN
 F 1 "GNDA" V 8725 4025 50  0000 C CNN
 F 2 "" H 8725 4275 50  0001 C CNN
@@
 $EndComp
 $Comp
-L GNDA #PWR032
+L GNDA #PWR406
 U 1 1 5965C333
 P 8725 4175
-F 0 "#PWR032" H 8725 3925 50  0001 C CNN
+F 0 "#PWR406" H 8725 3925 50  0001 C CNN
 F 1 "GNDA" V 8725 3925 50  0000 C CNN
 F 2 "" H 8725 4175 50  0001 C CNN
@@
 $EndComp
 $Comp
-L GNDA #PWR033
+L GNDA #PWR408
 U 1 1 5965C334
 P 8725 4375
-F 0 "#PWR033" H 8725 4125 50  0001 C CNN
+F 0 "#PWR408" H 8725 4125 50  0001 C CNN
 F 1 "GNDA" V 8725 4125 50  0000 C CNN
 F 2 "" H 8725 4375 50  0001 C CNN
@@
 $EndComp
 $Comp
-L GNDA #PWR034
+L GNDA #PWR409
 U 1 1 5965C335
 P 8725 4475
-F 0 "#PWR034" H 8725 4225 50  0001 C CNN
+F 0 "#PWR409" H 8725 4225 50  0001 C CNN
 F 1 "GNDA" V 8725 4225 50  0000 C CNN
 F 2 "" H 8725 4475 50  0001 C CNN
@@
 $EndComp
 $Comp
-L GNDA #PWR035
+L GNDA #PWR410
 U 1 1 5965C336
 P 8725 4575
-F 0 "#PWR035" H 8725 4325 50  0001 C CNN
+F 0 "#PWR410" H 8725 4325 50  0001 C CNN
 F 1 "GNDA" V 8725 4325 50  0000 C CNN
 F 2 "" H 8725 4575 50  0001 C CNN
@@
 GND_A
 $Comp
-L CONN_01X01 J?
+L CONN_01X01 J405
 U 1 1 599EC0AF
 P 10025 1600
-F 0 "J?" H 10025 1700 50  0000 C CNN
+F 0 "J405" H 10025 1700 50  0000 C CNN
 F 1 "Testpoint" V 10125 1600 50  0000 C CNN
 F 2 "library:Via-0.8mm" H 10025 1600 50  0001 C CNN
@@
 $EndComp
 $Comp
-L CONN_01X01 J?
+L CONN_01X01 J406
 U 1 1 599EC0FA
 P 10150 3725
-F 0 "J?" H 10150 3825 50  0000 C CNN
+F 0 "J406" H 10150 3825 50  0000 C CNN
 F 1 "Testpoint" V 10250 3725 50  0000 C CNN
 F 2 "library:Via-0.8mm" H 10150 3725 50  0001 C CNN
@@
 $EndComp
 $Comp
-L CONN_01X01 J?
+L CONN_01X01 J402
 U 1 1 599EC1CA
 P 5825 4325
-F 0 "J?" H 5825 4425 50  0000 C CNN
+F 0 "J402" H 5825 4425 50  0000 C CNN
 F 1 "Testpoint" V 5925 4325 50  0000 C CNN
 F 2 "library:Via-0.8mm" H 5825 4325 50  0001 C CNN
@@
 $EndComp
 $Comp
-L CONN_01X01 J?
+L CONN_01X01 J401
 U 1 1 599EC2EF
 P 5675 6200
-F 0 "J?" H 5675 6300 50  0000 C CNN
+F 0 "J401" H 5675 6300 50  0000 C CNN
 F 1 "Testpoint" V 5775 6200 50  0000 C CNN
 F 2 "library:Via-0.8mm" H 5675 6200 50  0001 C CNN
@@
 $EndComp
 $Comp
-L CONN_01X01 J?
+L CONN_01X01 J404
 U 1 1 599EC39F
 P 5950 3200
-F 0 "J?" H 5950 3300 50  0000 C CNN
+F 0 "J404" H 5950 3300 50  0000 C CNN
 F 1 "Testpoint" V 6050 3200 50  0000 C CNN
 F 2 "library:Via-0.8mm" H 5950 3200 50  0001 C CNN
@@
 $EndComp
 $Comp
-L CONN_01X01 J?
+L CONN_01X01 J403
 U 1 1 599EC468
 P 5850 1975
-F 0 "J?" H 5850 2075 50  0000 C CNN
+F 0 "J403" H 5850 2075 50  0000 C CNN
 F 1 "Testpoint" V 5950 1975 50  0000 C CNN
 F 2 "library:Via-0.8mm" H 5850 1975 50  0001 C CNN
