File: Attenuation.sch (KiCad schematic (older format))
At the start: 38 parts, among them J401 Testpoint, J402 Testpoint, J403 Testpoint, J404 Testpoint, J405 Testpoint, J406 Testpoint, J601 CONN_01X02, J602 CONN_01X02, U701 CPC1017N, U702 CPC1017N, U703 CD4051BM96, U704 CD4051BM96

Commit message: Doing re-routing
Parts:
- J601, J602: footprint Pin_Headers:Pin_Header_Angled_1x02_Pitch1.27mm -> Pin_Headers:Pin_Header_Straight_1x02_Pitch1.27mm
Changed lines of the file:
@@
 $EndComp
 $Comp
-L GNDA #PWR402
+L GNDA #PWR026
 U 1 1 5965C32C
 P 8700 1550
-F 0 "#PWR402" H 8700 1300 50  0001 C CNN
+F 0 "#PWR026" H 8700 1300 50  0001 C CNN
 F 1 "GNDA" V 8700 1300 50  0000 C CNN
 F 2 "" H 8700 1550 50  0001 C CNN
@@
 $EndComp
 $Comp
-L GNDA #PWR401
+L GNDA #PWR027
 U 1 1 5965C32D
 P 8700 1450
-F 0 "#PWR401" H 8700 1200 50  0001 C CNN
+F 0 "#PWR027" H 8700 1200 50  0001 C CNN
 F 1 "GNDA" V 8700 1200 50  0000 C CNN
 F 2 "" H 8700 1450 50  0001 C CNN
@@
 $EndComp
 $Comp
-L GNDA #PWR403
+L GNDA #PWR028
 U 1 1 5965C32E
 P 8700 1650
-F 0 "#PWR403" H 8700 1400 50  0001 C CNN
+F 0 "#PWR028" H 8700 1400 50  0001 C CNN
 F 1 "GNDA" V 8700 1400 50  0000 C CNN
 F 2 "" H 8700 1650 50  0001 C CNN
@@
 $EndComp
 $Comp
-L GNDA #PWR404
+L GNDA #PWR029
 U 1 1 5965C32F
 P 8700 1750
-F 0 "#PWR404" H 8700 1500 50  0001 C CNN
+F 0 "#PWR029" H 8700 1500 50  0001 C CNN
 F 1 "GNDA" V 8700 1500 50  0000 C CNN
 F 2 "" H 8700 1750 50  0001 C CNN
@@
 $EndComp
 $Comp
-L GNDA #PWR405
+L GNDA #PWR030
 U 1 1 5965C330
 P 8700 1850
-F 0 "#PWR405" H 8700 1600 50  0001 C CNN
+F 0 "#PWR030" H 8700 1600 50  0001 C CNN
 F 1 "GNDA" V 8700 1600 50  0000 C CNN
 F 2 "" H 8700 1850 50  0001 C CNN
@@
 $EndComp
 $Comp
-L GNDA #PWR407
+L GNDA #PWR031
 U 1 1 5965C332
 P 8725 4275
-F 0 "#PWR407" H 8725 4025 50  0001 C CNN
+F 0 "#PWR031" H 8725 4025 50  0001 C CNN
 F 1 "GNDA" V 8725 4025 50  0000 C CNN
 F 2 "" H 8725 4275 50  0001 C CNN
@@
 $EndComp
 $Comp
-L GNDA #PWR406
+L GNDA #PWR032
 U 1 1 5965C333
 P 8725 4175
-F 0 "#PWR406" H 8725 3925 50  0001 C CNN
+F 0 "#PWR032" H 8725 3925 50  0001 C CNN
 F 1 "GNDA" V 8725 3925 50  0000 C CNN
 F 2 "" H 8725 4175 50  0001 C CNN
@@
 $EndComp
 $Comp
-L GNDA #PWR408
+L GNDA #PWR033
 U 1 1 5965C334
 P 8725 4375
-F 0 "#PWR408" H 8725 4125 50  0001 C CNN
+F 0 "#PWR033" H 8725 4125 50  0001 C CNN
 F 1 "GNDA" V 8725 4125 50  0000 C CNN
 F 2 "" H 8725 4375 50  0001 C CNN
@@
 $EndComp
 $Comp
-L GNDA #PWR409
+L GNDA #PWR034
 U 1 1 5965C335
 P 8725 4475
-F 0 "#PWR409" H 8725 4225 50  0001 C CNN
+F 0 "#PWR034" H 8725 4225 50  0001 C CNN
 F 1 "GNDA" V 8725 4225 50  0000 C CNN
 F 2 "" H 8725 4475 50  0001 C CNN
@@
 $EndComp
 $Comp
-L GNDA #PWR410
+L GNDA #PWR035
 U 1 1 5965C336
 P 8725 4575
-F 0 "#PWR410" H 8725 4325 50  0001 C CNN
+F 0 "#PWR035" H 8725 4325 50  0001 C CNN
 F 1 "GNDA" V 8725 4325 50  0000 C CNN
 F 2 "" H 8725 4575 50  0001 C CNN
@@
 F 0 "J601" H 7800 1550 50  0000 C CNN
 F 1 "CONN_01X02" V 7900 1400 50  0000 C CNN
-F 2 "Pin_Headers:Pin_Header_Angled_1x02_Pitch1.27mm" H 7800 1400 50  0001 C CNN
+F 2 "Pin_Headers:Pin_Header_Straight_1x02_Pitch1.27mm" H 7800 1400 50  0001 C CNN
 F 3 "" H 7800 1400 50  0001 C CNN
 	1    7800 1400
@@
 F 0 "J602" H 7800 4275 50  0000 C CNN
 F 1 "CONN_01X02" V 7900 4125 50  0000 C CNN
-F 2 "Pin_Headers:Pin_Header_Angled_1x02_Pitch1.27mm" H 7800 4125 50  0001 C CNN
+F 2 "Pin_Headers:Pin_Header_Straight_1x02_Pitch1.27mm" H 7800 4125 50  0001 C CNN
 F 3 "" H 7800 4125 50  0001 C CNN
 	1    7800 4125

Commit message: DRC
Parts:
- J401, J402, J403, J404, J405, J406: footprint library:Via-0.8mm -> library:TestPoint
Changed lines of the file:
@@
 F 0 "J405" H 10025 1700 50  0000 C CNN
 F 1 "Testpoint" V 10125 1600 50  0000 C CNN
-F 2 "library:Via-0.8mm" H 10025 1600 50  0001 C CNN
+F 2 "library:TestPoint" H 10025 1600 50  0001 C CNN
 F 3 "" H 10025 1600 50  0001 C CNN
 	1    10025 1600
@@
 F 0 "J406" H 10150 3825 50  0000 C CNN
 F 1 "Testpoint" V 10250 3725 50  0000 C CNN
-F 2 "library:Via-0.8mm" H 10150 3725 50  0001 C CNN
+F 2 "library:TestPoint" H 10150 3725 50  0001 C CNN
 F 3 "" H 10150 3725 50  0001 C CNN
 	1    10150 3725
@@
 F 0 "J402" H 5825 4425 50  0000 C CNN
 F 1 "Testpoint" V 5925 4325 50  0000 C CNN
-F 2 "library:Via-0.8mm" H 5825 4325 50  0001 C CNN
+F 2 "library:TestPoint" H 5825 4325 50  0001 C CNN
 F 3 "" H 5825 4325 50  0001 C CNN
 	1    5825 4325
@@
 F 0 "J401" H 5675 6300 50  0000 C CNN
 F 1 "Testpoint" V 5775 6200 50  0000 C CNN
-F 2 "library:Via-0.8mm" H 5675 6200 50  0001 C CNN
+F 2 "library:TestPoint" H 5675 6200 50  0001 C CNN
 F 3 "" H 5675 6200 50  0001 C CNN
 	1    5675 6200
@@
 F 0 "J404" H 5950 3300 50  0000 C CNN
 F 1 "Testpoint" V 6050 3200 50  0000 C CNN
-F 2 "library:Via-0.8mm" H 5950 3200 50  0001 C CNN
+F 2 "library:TestPoint" H 5950 3200 50  0001 C CNN
 F 3 "" H 5950 3200 50  0001 C CNN
 	1    5950 3200
@@
 F 0 "J403" H 5850 2075 50  0000 C CNN
 F 1 "Testpoint" V 5950 1975 50  0000 C CNN
-F 2 "library:Via-0.8mm" H 5850 1975 50  0001 C CNN
+F 2 "library:TestPoint" H 5850 1975 50  0001 C CNN
 F 3 "" H 5850 1975 50  0001 C CNN
 	1    5850 1975

Commit message: Updated some MPN
Parts:
- C713, C714: DNP (none) -> 1
Changed lines of the file:
@@
 $EndComp
 $Comp
-L GNDA #PWR402
+L GNDA #PWR026
 U 1 1 5965C32C
 P 8700 1550
-F 0 "#PWR402" H 8700 1300 50  0001 C CNN
+F 0 "#PWR026" H 8700 1300 50  0001 C CNN
 F 1 "GNDA" V 8700 1300 50  0000 C CNN
 F 2 "" H 8700 1550 50  0001 C CNN
@@
 $EndComp
 $Comp
-L GNDA #PWR401
+L GNDA #PWR027
 U 1 1 5965C32D
 P 8700 1450
-F 0 "#PWR401" H 8700 1200 50  0001 C CNN
+F 0 "#PWR027" H 8700 1200 50  0001 C CNN
 F 1 "GNDA" V 8700 1200 50  0000 C CNN
 F 2 "" H 8700 1450 50  0001 C CNN
@@
 $EndComp
 $Comp
-L GNDA #PWR403
+L GNDA #PWR028
 U 1 1 5965C32E
 P 8700 1650
-F 0 "#PWR403" H 8700 1400 50  0001 C CNN
+F 0 "#PWR028" H 8700 1400 50  0001 C CNN
 F 1 "GNDA" V 8700 1400 50  0000 C CNN
 F 2 "" H 8700 1650 50  0001 C CNN
@@
 $EndComp
 $Comp
-L GNDA #PWR404
+L GNDA #PWR029
 U 1 1 5965C32F
 P 8700 1750
-F 0 "#PWR404" H 8700 1500 50  0001 C CNN
+F 0 "#PWR029" H 8700 1500 50  0001 C CNN
 F 1 "GNDA" V 8700 1500 50  0000 C CNN
 F 2 "" H 8700 1750 50  0001 C CNN
@@
 $EndComp
 $Comp
-L GNDA #PWR405
+L GNDA #PWR030
 U 1 1 5965C330
 P 8700 1850
-F 0 "#PWR405" H 8700 1600 50  0001 C CNN
+F 0 "#PWR030" H 8700 1600 50  0001 C CNN
 F 1 "GNDA" V 8700 1600 50  0000 C CNN
 F 2 "" H 8700 1850 50  0001 C CNN
@@
 $EndComp
 $Comp
-L GNDA #PWR407
+L GNDA #PWR031
 U 1 1 5965C332
 P 8725 4275
-F 0 "#PWR407" H 8725 4025 50  0001 C CNN
+F 0 "#PWR031" H 8725 4025 50  0001 C CNN
 F 1 "GNDA" V 8725 4025 50  0000 C CNN
 F 2 "" H 8725 4275 50  0001 C CNN
@@
 $EndComp
 $Comp
-L GNDA #PWR406
+L GNDA #PWR032
 U 1 1 5965C333
 P 8725 4175
-F 0 "#PWR406" H 8725 3925 50  0001 C CNN
+F 0 "#PWR032" H 8725 3925 50  0001 C CNN
 F 1 "GNDA" V 8725 3925 50  0000 C CNN
 F 2 "" H 8725 4175 50  0001 C CNN
@@
 $EndComp
 $Comp
-L GNDA #PWR408
+L GNDA #PWR033
 U 1 1 5965C334
 P 8725 4375
-F 0 "#PWR408" H 8725 4125 50  0001 C CNN
+F 0 "#PWR033" H 8725 4125 50  0001 C CNN
 F 1 "GNDA" V 8725 4125 50  0000 C CNN
 F 2 "" H 8725 4375 50  0001 C CNN
@@
 $EndComp
 $Comp
-L GNDA #PWR409
+L GNDA #PWR034
 U 1 1 5965C335
 P 8725 4475
-F 0 "#PWR409" H 8725 4225 50  0001 C CNN
+F 0 "#PWR034" H 8725 4225 50  0001 C CNN
 F 1 "GNDA" V 8725 4225 50  0000 C CNN
 F 2 "" H 8725 4475 50  0001 C CNN
@@
 $EndComp
 $Comp
-L GNDA #PWR410
+L GNDA #PWR035
 U 1 1 5965C336
 P 8725 4575
-F 0 "#PWR410" H 8725 4325 50  0001 C CNN
+F 0 "#PWR035" H 8725 4325 50  0001 C CNN
 F 1 "GNDA" V 8725 4325 50  0000 C CNN
 F 2 "" H 8725 4575 50  0001 C CNN
@@
 F 2 "Capacitors_THT:CP_Radial_Tantal_D6.0mm_P5.00mm" H 4700 1850 50  0001 C CNN
 F 3 "" H 4700 1850 50  0001 C CNN
+F 4 "1" H 4700 1850 60  0001 C CNN "DNP"
 	1    4700 1850
 	1    0    0    -1
@@
 F 2 "Capacitors_THT:CP_Radial_Tantal_D6.0mm_P5.00mm" H 4575 4725 50  0001 C CNN
 F 3 "" H 4575 4725 50  0001 C CNN
+F 4 "1" H 4575 4725 60  0001 C CNN "DNP"
 	1    4575 4725
 	1    0    0    -1

Commit message: Updated MPN to components avalaible in mouser. Updating footprints now ...
Parts:
- C701, C702: MPN VJ0603A101JXACW1BC -> GRM1885C1H101GA01J
- C709, C711: value 180p -> 180pF
- C710, C712: value 1800p -> 1800pF; MPN GCM1885C1H182FA16D -> GRM1885C1H182FA01D
- C713, C714: VDC (none) -> 1
- D701, D702: MPN BAT54S-7-F -> BAT54S
- J601, J602: MPN (none) -> M50-3030242
- R703, R707: value 89K8 -> 90K9; MPN RT0603DRE0789K8L -> RR0816P-9092-D-93C
