File: etapa_analogica.sch (KiCad schematic (older format))
At the start: 36 parts

Commit message: Completed part selection of analog board. Merged analog and digital boards.
Parts:
- renumbered C101 to C601, C102 to C602, C103 to C603, C104 to C604, C105 to C605, C106 to C606, C107 to C607, C108 to C608, C109 to C609, C110 to C610, C111 to C611, C112 to C612, C113 to C613, C114 to C614, C115 to C615, C116 to C616, C117 to C617, C118 to C618, C119 to C619, C120 to C620, C121 to C621, C122 to C622, C123 to C623, C124 to C624, C125 to C625, C126 to C626, C127 to C627, C128 to C628, C129 to C629, C130 to C630, C131 to C631, C132 to C632, C133 to C633, C134 to C634, C135 to C635, C136 to C636

Commit message: ....
Connections:
- net labels added: SCL_OFF, SDA_OFF
- net labels removed: SCL, SDA
Changed lines of the file:
@@
 CHB_DAC
 Text HLabel 5325 4400 0    60   Input ~ 0
-SDA
+SDA_OFF
 Text HLabel 5325 4525 0    60   Input ~ 0
-SCL
+SCL_OFF
 $Sheet
 S 5550 3725 1350 1750

Commit message: No more DRC errors :)
Connections:
- net labels added: +3V3_A
- net labels removed: +3V3
Changed lines of the file:
@@
 +5V
 Text Label 2150 700  2    60   ~ 0
-+3V3
++3V3_A
 Text Label 2150 850  2    60   ~ 0
 -3V0
@@
 F1 "Analog_Power_Supply.sch" 60
 F2 "+5V" I L 1900 1825 60
-F3 "+3V3" O R 2725 1825 60
-F4 "-3V0" O R 2725 1975 60
-F5 "GND_A" I L 1900 2125 60
-F6 "-5V" O R 2725 2125 60
+F3 "-3V0" O R 2725 1975 60
+F4 "GND_A" I L 1900 2125 60
+F5 "-5V" O R 2725 2125 60
+F6 "+3V3_A" O R 2725 1825 60
 $EndSheet
 Text Label 1900 1825 2    60   ~ 0
 +5V
 Text Label 2725 1825 0    60   ~ 0
-+3V3
++3V3_A
 Text Label 2725 1975 0    60   ~ 0
 -3V0

Commit message: Assignement of FPGA pins for analog stage control
Connections:
- wire segments 140 -> 138
Changed lines of the file:
@@
 $Descr A4 11693 8268
 encoding utf-8
-Sheet 6 11
+Sheet 5 11
 Title ""
 Date ""
@@
 F5 "CHA_ATT_EN" I L 5525 1500 60
 F6 "VDD_A" I L 5525 2675 60
-F7 "CHB_OFFSET" I L 5525 1600 60
 F8 "CHB_ATT_SEL_0" I L 5525 1750 60
 F9 "CHB_ATT_SEL_1" I L 5525 1850 60
 F10 "CHB_ATT_SEL_2" I L 5525 1950 60
 F11 "CHB_ATT_EN" I L 5525 2050 60
-F12 "CHA_OFFSET" I L 5525 2150 60
 F13 "CHA_DC_COUPLING" I L 5525 2300 60
 F14 "CHB_DC_COUPLING" I L 5525 2400 60
@@
 Text Label 6900 4950 0    60   ~ 0
 CHB_OFFSET
-Text Label 4400 2150 2    60   ~ 0
-CHA_OFFSET
-Text Label 4400 1600 2    60   ~ 0
-CHB_OFFSET
 Text Label 7025 4275 0    60   ~ 0
 CHB_VREF_CENT
@@
 	5525 2400 5225 2400
 Wire Wire Line
-	5525 2150 4400 2150
-Wire Wire Line
-	5525 1600 4400 1600
-Wire Wire Line
 	8925 1525 8625 1525

Commit message: Modified a lot of fields in components parts. BOM generated. Added BOM plugin script.
Parts:
- C601, C603, C605, C606, C608, C612, C614, C616, C618, C619, C621, C623, C625, C627, C629, C631, C633, C635: Dielectric (none) -> X7R; MPN (none) -> C0603C104K3RACTU; Manufacturer Part C0603C104K3RACTU -> (none); Tipo Ceramic -> (none); Type (none) -> Ceramic; VDC (none) -> 25V
- C602, C604, C607, C609, C611, C613, C615, C617, C622, C624, C626, C628, C630, C632, C634, C636: Dielectric (none) -> X5R; MPN (none) -> GRM188R61C105KA93D; Manufacturer Part C0603C105K8PACTU -> (none); Tipo Ceramic -> (none); Type (none) -> Ceramic; VDC (none) -> 16V
- C610, C620: Dielectric (none) -> X5R; Tipo Ceramic -> (none); Type (none) -> Ceramic; VDC (none) -> 6,3V
