File: etapa_analogica.sch (KiCad schematic (older format))
At the start: 36 parts

Commit message: Changed some MPN and footprints. BOM updated.
Parts:
- C610, C620: VDC 6,3V -> 6V3

Commit message: Added resistance to control lines to prevent overshoot
Parts:
- added R309, R310, R311, R312, R313, R314, R315, R316, R317, R318, R319, R320, R321, R322: 1K, Resistors_SMD:R_0603_HandSoldering, symbol R
Connections:
- wire segments 138 -> 152

Commit message: Updated MPN to components avalaible in mouser. Updating footprints now ...
Parts:
- C602, C604, C607, C609, C611, C613, C615, C617, C622, C624, C626, C628, C630, C632, C634, C636: MPN GRM188R61C105KA93D -> C0603C105K8PACTU; VDC 16V -> 10V
