File: iCE40hxk4_dev_board.sch (KiCad schematic (older format))
At the start: 0 parts

Commit message: Added square wave output.
Parts:
- added J101: CONN_01X01, Pin_Headers:Pin_Header_Angled_1x01_Pitch1.27mm, symbol CONN_01X01
- added R101: 10k, Resistors_SMD:R_0603_HandSoldering, symbol R
Connections:
- wire segments 84 -> 86
Other:
- note added: "Rectangular \npulsed signal\n"
Changed lines of the file:
@@
 $EndSheet
 $Comp
-L GNDD #PWR01
+L GNDD #PWR110
 U 1 1 58DE77E1
 P 6075 3325
-F 0 "#PWR01" H 6075 3075 50  0001 C CNN
+F 0 "#PWR110" H 6075 3075 50  0001 C CNN
 F 1 "GNDD" H 6075 3175 50  0000 C CNN
 F 2 "" H 6075 3325 50  0001 C CNN
@@
 $EndComp
 $Comp
-L +3.3V #PWR02
+L +3.3V #PWR104
 U 1 1 58DDF070
 P 2775 1875
-F 0 "#PWR02" H 2775 1725 50  0001 C CNN
+F 0 "#PWR104" H 2775 1725 50  0001 C CNN
 F 1 "+3.3V" H 2775 2015 50  0000 C CNN
 F 2 "" H 2775 1875 50  0001 C CNN
@@
 $EndComp
 $Comp
-L +3.3V #PWR03
+L +3.3V #PWR105
 U 1 1 58DDF24C
 P 3675 4325
-F 0 "#PWR03" H 3675 4175 50  0001 C CNN
+F 0 "#PWR105" H 3675 4175 50  0001 C CNN
 F 1 "+3.3V" H 3675 4465 50  0000 C CNN
 F 2 "" H 3675 4325 50  0001 C CNN
@@
 $EndComp
 $Comp
-L GND #PWR04
+L GND #PWR102
 U 1 1 58DDFD7B
 P 775 2675
-F 0 "#PWR04" H 775 2425 50  0001 C CNN
+F 0 "#PWR102" H 775 2425 50  0001 C CNN
 F 1 "GND" H 775 2525 50  0000 C CNN
 F 2 "" H 775 2675 50  0001 C CNN
@@
 $EndComp
 $Comp
-L GNDD #PWR05
+L GNDD #PWR101
 U 1 1 58DDFDF5
 P 625 2525
-F 0 "#PWR05" H 625 2275 50  0001 C CNN
+F 0 "#PWR101" H 625 2275 50  0001 C CNN
 F 1 "GNDD" H 625 2375 50  0000 C CNN
 F 2 "" H 625 2525 50  0001 C CNN
@@
 $EndComp
 $Comp
-L GNDD #PWR06
+L GNDD #PWR108
 U 1 1 58DDFE6D
 P 5875 6275
-F 0 "#PWR06" H 5875 6025 50  0001 C CNN
+F 0 "#PWR108" H 5875 6025 50  0001 C CNN
 F 1 "GNDD" H 5875 6125 50  0000 C CNN
 F 2 "" H 5875 6275 50  0001 C CNN
@@
 $EndComp
 $Comp
-L GNDD #PWR07
+L GNDD #PWR107
 U 1 1 58DE33A2
 P 5775 6975
-F 0 "#PWR07" H 5775 6725 50  0001 C CNN
+F 0 "#PWR107" H 5775 6725 50  0001 C CNN
 F 1 "GNDD" H 5775 6825 50  0000 C CNN
 F 2 "" H 5775 6975 50  0001 C CNN
@@
 $EndComp
 $Comp
-L GND #PWR08
+L GND #PWR109
 U 1 1 58DE341F
 P 5975 6975
-F 0 "#PWR08" H 5975 6725 50  0001 C CNN
+F 0 "#PWR109" H 5975 6725 50  0001 C CNN
 F 1 "GND" H 5975 6825 50  0000 C CNN
 F 2 "" H 5975 6975 50  0001 C CNN
@@
 $EndComp
 $Comp
-L +5V #PWR09
+L +5V #PWR103
 U 1 1 592DDA96
 P 2675 3975
-F 0 "#PWR09" H 2675 3825 50  0001 C CNN
+F 0 "#PWR103" H 2675 3825 50  0001 C CNN
 F 1 "+5V" H 2675 4115 50  0000 C CNN
 F 2 "" H 2675 3975 50  0001 C CNN
@@
 $EndSheet
 $Comp
-L +3.3V #PWR010
+L +3.3V #PWR118
 U 1 1 59674AAB
 P 8425 1575
-F 0 "#PWR010" H 8425 1425 50  0001 C CNN
+F 0 "#PWR118" H 8425 1425 50  0001 C CNN
 F 1 "+3.3V" H 8425 1715 50  0000 C CNN
 F 2 "" H 8425 1575 50  0001 C CNN
@@
 	10450 6200 10575 6200
 $Comp
-L GNDA #PWR011
+L GNDA #PWR106
 U 1 1 596A4A64
 P 5575 6975
-F 0 "#PWR011" H 5575 6725 50  0001 C CNN
+F 0 "#PWR106" H 5575 6725 50  0001 C CNN
 F 1 "GNDA" H 5575 6825 50  0000 C CNN
 F 2 "" H 5575 6975 50  0001 C CNN
@@
 F30 "IOT_177" B R 8100 3725 60
 F31 "IOT_178" B R 8100 3825 60
-F32 "IOT_144" B L 6525 2950 60
 F33 "IOT_146" B L 6525 2175 60
-F34 "IOT_147" B L 6525 2325 60
 F35 "IOT_148" B R 8100 2625 60
 F36 "IOT_152" B R 8100 2725 60
@@
 F41 "IOT_166" B R 8100 1925 60
 F42 "IOT_167" B R 8100 2025 60
-F44 "IOT_140" B L 6525 2525 60
 $EndSheet
 Wire Wire Line
@@
 	8100 5750 8525 5750
 $Comp
-L +5V #PWR012
+L +5V #PWR119
 U 1 1 598A074E
 P 10550 1625
-F 0 "#PWR012" H 10550 1475 50  0001 C CNN
+F 0 "#PWR119" H 10550 1475 50  0001 C CNN
 F 1 "+5V" H 10550 1765 50  0000 C CNN
 F 2 "" H 10550 1625 50  0001 C CNN
@@
 	8425 1650 8425 1575
 $Comp
-L GNDD #PWR013
+L GNDD #PWR113
 U 1 1 598A55A1
 P 8325 6275
-F 0 "#PWR013" H 8325 6025 50  0001 C CNN
+F 0 "#PWR113" H 8325 6025 50  0001 C CNN
 F 1 "GNDD" H 8325 6125 50  0000 C CNN
 F 2 "" H 8325 6275 50  0001 C CNN
@@
 Connection ~ 8325 6225
 $Comp
-L GNDA #PWR014
+L GNDA #PWR120
 U 1 1 598A69B6
 P 10575 6200
-F 0 "#PWR014" H 10575 5950 50  0001 C CNN
+F 0 "#PWR120" H 10575 5950 50  0001 C CNN
 F 1 "GNDA" H 10575 6050 50  0000 C CNN
 F 2 "" H 10575 6200 50  0001 C CNN
@@
 	6525 5800 5525 5800
 $Comp
-L +3.3V #PWR015
+L +3.3V #PWR111
 U 1 1 5980F198
 P 6175 1650
-F 0 "#PWR015" H 6175 1500 50  0001 C CNN
+F 0 "#PWR111" H 6175 1500 50  0001 C CNN
 F 1 "+3.3V" H 6175 1790 50  0000 C CNN
 F 2 "" H 6175 1650 50  0001 C CNN
@@
 $EndComp
 $Comp
-L +5V #PWR016
+L +5V #PWR112
 U 1 1 5980F81B
 P 6400 1650
-F 0 "#PWR016" H 6400 1500 50  0001 C CNN
+F 0 "#PWR112" H 6400 1500 50  0001 C CNN
 F 1 "+5V" H 6400 1790 50  0000 C CNN
 F 2 "" H 6400 1650 50  0001 C CNN
@@
 	10450 1925 10800 1925
 $Comp
-L GNDD #PWR017
+L GNDD #PWR121
 U 1 1 59938834
 P 10875 4000
-F 0 "#PWR017" H 10875 3750 50  0001 C CNN
+F 0 "#PWR121" H 10875 3750 50  0001 C CNN
 F 1 "GNDD" H 10875 3850 50  0000 C CNN
 F 2 "" H 10875 4000 50  0001 C CNN
@@
 Connection ~ 10875 3950
 $Comp
-L GNDD #PWR018
+L GNDD #PWR114
 U 1 1 59940669
 P 8350 2125
-F 0 "#PWR018" H 8350 1875 50  0001 C CNN
+F 0 "#PWR114" H 8350 1875 50  0001 C CNN
 F 1 "GNDD" H 8350 1975 50  0000 C CNN
 F 2 "" H 8350 2125 50  0001 C CNN
@@
 $EndComp
 $Comp
-L GNDD #PWR019
+L GNDD #PWR115
 U 1 1 599409AA
 P 8350 2525
-F 0 "#PWR019" H 8350 2275 50  0001 C CNN
+F 0 "#PWR115" H 8350 2275 50  0001 C CNN
 F 1 "GNDD" H 8350 2375 50  0000 C CNN
 F 2 "" H 8350 2525 50  0001 C CNN
@@
 $EndComp
 $Comp
-L GNDD #PWR020
+L GNDD #PWR116
 U 1 1 59940CEB
 P 8350 3125
-F 0 "#PWR020" H 8350 2875 50  0001 C CNN
+F 0 "#PWR116" H 8350 2875 50  0001 C CNN
 F 1 "GNDD" H 8350 2975 50  0000 C CNN
 F 2 "" H 8350 3125 50  0001 C CNN
@@
 	8350 3125 8525 3125
 $Comp
-L GNDD #PWR021
+L GNDD #PWR117
 U 1 1 5994102C
 P 8350 3525
-F 0 "#PWR021" H 8350 3275 50  0001 C CNN
+F 0 "#PWR117" H 8350 3275 50  0001 C CNN
 F 1 "GNDD" H 8350 3375 50  0000 C CNN
 F 2 "" H 8350 3525 50  0001 C CNN
@@
 Wire Wire Line
 	8350 3525 8525 3525
+$Comp
+L CONN_01X01 J101
+U 1 1 5993A8F3
+P 5750 2175
+F 0 "J101" H 5750 2275 50  0000 C CNN
+F 1 "CONN_01X01" V 5850 2175 50  0000 C CNN
+F 2 "Pin_Headers:Pin_Header_Angled_1x01_Pitch1.27mm" H 5750 2175 50  0001 C CNN
+F 3 "" H 5750 2175 50  0001 C CNN
+	1    5750 2175
+	-1   0    0    1
+$EndComp
+Text Notes 5775 2600 0    60   ~ 0
+Rectangular \npulsed signal\n
+$Comp
+L R R101
+U 1 1 5993D9BD
+P 6250 2175
+F 0 "R101" V 6330 2175 50  0000 C CNN
+F 1 "10k" V 6250 2175 50  0000 C CNN
+F 2 "Resistors_SMD:R_0603_HandSoldering" V 6180 2175 50  0001 C CNN
+F 3 "http://ar.mouser.com/ProductDetail/Vishay/CRCW060310K0FKEA/?qs=sGAEpiMZZMvdGkrng054t%252b8cnVAnHPZkqchqPaQRdrE%3d" H 6250 2175 50  0001 C CNN
+F 4 "CRCW060310K0FKEA" V 6250 2175 60  0001 C CNN "Manufacterer Part"
+	1    6250 2175
+	0    1    1    0
+$EndComp
+Wire Wire Line
+	6100 2175 5950 2175
+Wire Wire Line
+	6400 2175 6525 2175
 $EndSCHEMATC

Commit message: Modified a lot of fields in components parts. BOM generated. Added BOM plugin script.
Parts:
- removed J101: CONN_01X01, Pin_Headers:Pin_Header_Angled_1x01_Pitch1.27mm, symbol CONN_01X01
- added J101: CONN_01X02, Pin_Headers:Pin_Header_Angled_1x02_Pitch1.27mm, symbol CONN_01X02
- R101: value 10k -> 10K; MPN (none) -> RT0603DRE0710KL; Manufacterer Part CRCW060310K0FKEA -> (none)
Connections:
- wire segments 86 -> 87
