File: iCE40hxk4_dev_board.sch (KiCad schematic (older format))
At the start: 5 parts, among them J101 CONN_01X02, J102 KobiConn_161-3507_Jack_3.5mm, J103 CONN_COAXIAL, J104 CONN_COAXIAL

Commit message: Almost rev1
Parts:
- added J105, J106, J107, J108: MountingHole, library:MountingHole, symbol MountingHole
Connections:
- wire segments 93 -> 99
Changed lines of the file:
@@
 LIBS:switches
 LIBS:kobiconn_161-3507_jack_3
+LIBS:mountinghole
 LIBS:iCE40hxk4_dev_board-cache
 EELAYER 25 0
@@
 	-1   0    0    1
 $EndComp
-$Comp
-L GNDD #PWR022
-U 1 1 599C8049
-P 5000 2275
-F 0 "#PWR022" H 5000 2025 50  0001 C CNN
-F 1 "GNDD" H 5000 2125 50  0000 C CNN
-F 2 "" H 5000 2275 50  0001 C CNN
-F 3 "" H 5000 2275 50  0001 C CNN
-	1    5000 2275
-	1    0    0    -1
-$EndComp
 Text Notes 4725 2650 0    60   ~ 0
 Rectangular \npulsed signal\n
@@
 $EndComp
 $Comp
-L GNDA #PWR023
+L GNDA #PWR022
 U 1 1 59A349F5
 P 10575 1425
-F 0 "#PWR023" H 10575 1175 50  0001 C CNN
+F 0 "#PWR022" H 10575 1175 50  0001 C CNN
 F 1 "GNDA" H 10575 1275 50  0000 C CNN
 F 2 "" H 10575 1425 50  0001 C CNN
@@
 $EndComp
 $Comp
-L GNDA #PWR024
+L GNDA #PWR023
 U 1 1 59A34D3A
 P 10575 2125
-F 0 "#PWR024" H 10575 1875 50  0001 C CNN
+F 0 "#PWR023" H 10575 1875 50  0001 C CNN
 F 1 "GNDA" H 10575 1975 50  0000 C CNN
 F 2 "" H 10575 2125 50  0001 C CNN
@@
 	10125 1225 10425 1225
 $Comp
-L GNDA #PWR025
+L GNDA #PWR024
 U 1 1 59A41356
 P 9800 2875
-F 0 "#PWR025" H 9800 2625 50  0001 C CNN
+F 0 "#PWR024" H 9800 2625 50  0001 C CNN
 F 1 "GNDA" H 9800 2725 50  0000 C CNN
 F 2 "" H 9800 2875 50  0001 C CNN
@@
 Wire Wire Line
 	10425 2525 10425 2750
+Wire Wire Line
+	5000 2275 5000 2175
+Connection ~ 5000 2175
+$Comp
+L MountingHole J106
+U 1 1 59A63C8B
+P 3000 7050
+F 0 "J106" H 3000 7150 60  0000 C CNN
+F 1 "MountingHole" H 3050 6900 60  0001 C CNN
+F 2 "library:MountingHole" H 3000 7050 60  0001 C CNN
+F 3 "" H 3000 7050 60  0001 C CNN
+	1    3000 7050
+	1    0    0    -1
+$EndComp
+$Comp
+L MountingHole J107
+U 1 1 59A644BA
+P 3000 7225
+F 0 "J107" H 3000 7325 60  0000 C CNN
+F 1 "MountingHole" H 3050 7075 60  0001 C CNN
+F 2 "library:MountingHole" H 3000 7225 60  0001 C CNN
+F 3 "" H 3000 7225 60  0001 C CNN
+	1    3000 7225
+	1    0    0    -1
+$EndComp
+$Comp
+L MountingHole J108
+U 1 1 59A64829
+P 3000 7425
+F 0 "J108" H 3000 7525 60  0000 C CNN
+F 1 "MountingHole" H 3050 7275 60  0000 C CNN
+F 2 "library:MountingHole" H 3000 7425 60  0001 C CNN
+F 3 "" H 3000 7425 60  0001 C CNN
+	1    3000 7425
+	1    0    0    -1
+$EndComp
+$Comp
+L MountingHole J105
+U 1 1 59A64B8B
+P 3000 6875
+F 0 "J105" H 3000 6975 60  0000 C CNN
+F 1 "MountingHole" H 3050 6725 60  0001 C CNN
+F 2 "library:MountingHole" H 3000 6875 60  0001 C CNN
+F 3 "" H 3000 6875 60  0001 C CNN
+	1    3000 6875
+	1    0    0    -1
+$EndComp
+Wire Wire Line
+	2850 7425 2625 7425
+Wire Wire Line
+	2625 6875 2625 7500
+Wire Wire Line
+	2625 6875 2850 6875
+Wire Wire Line
+	2850 7050 2625 7050
+Connection ~ 2625 7050
+Wire Wire Line
+	2850 7225 2625 7225
+Connection ~ 2625 7225
+Connection ~ 2625 7425
+$Comp
+L GND #PWR?
+U 1 1 59A6AB48
+P 2625 7500
+F 0 "#PWR?" H 2625 7250 50  0001 C CNN
+F 1 "GND" H 2625 7350 50  0000 C CNN
+F 2 "" H 2625 7500 50  0001 C CNN
+F 3 "" H 2625 7500 50  0001 C CNN
+	1    2625 7500
+	1    0    0    -1
+$EndComp
 $EndSCHEMATC

Commit message: Updated MPN to components avalaible in mouser. Updating footprints now ...
Parts:
- J102: value KobiConn_161-3507_Jack_3.5mm -> KobiConn_161-3509-E_Jack_3.5mm; MPN KobiConn_161-3507 -> KobiConn_161-3509-E
- J103, J104: MPN 73100-0105 -> 1-1337543-0

Commit message: Updated jack symbol and footprint
Parts:
- removed J102: KobiConn_161-3509-E_Jack_3.5mm, library:KobiConn_161-3507_Jack_3.5mm, symbol KobiConn_161-3507_Jack_3.5mm
- added J102: Jack Estereo, library:KobiConn_161-3509-E_Jack_3.5mm, symbol KobiConn_161-3509-E_Jack_3.5mm
Changed lines of the file:
@@
 LIBS:voltage-regulators
 LIBS:switches
-LIBS:kobiconn_161-3507_jack_3
 LIBS:mountinghole
+LIBS:kobiconn_161-3507_3.5mm_jack
+LIBS:kobiconn_161-3509-E_3.5mm_jack
 LIBS:iCE40hxk4_dev_board-cache
 EELAYER 25 0
@@
 $EndComp
 $Comp
-L KobiConn_161-3507_Jack_3.5mm J102
-U 1 1 59A2F66A
-P 10525 3450
-F 0 "J102" V 9825 3450 60  0000 C CNN
-F 1 "KobiConn_161-3509-E_Jack_3.5mm" V 9925 3550 60  0000 C CNN
-F 2 "library:KobiConn_161-3507_Jack_3.5mm" H 10675 3450 60  0001 C CNN
-F 3 "http://ar.mouser.com/ProductDetail/Kobiconn/161-3509-E/?qs=sGAEpiMZZMv0W4pxf2HiV4Mt5ZQSVq1hR5HUmztPvpo%3d" H 10675 3450 60  0001 C CNN
-F 4 "KobiConn_161-3509-E" V 10525 3450 60  0001 C CNN "MPN"
-	1    10525 3450
-	0    -1   -1   0
-$EndComp
-$Comp
 L MountingHole J106
 U 1 1 59A63C8B
@@
 	9800 2750 10225 2750
 Wire Wire Line
-	10925 2750 10825 2750
+	10625 2750 10925 2750
 Wire Wire Line
 	10425 2525 10425 2750
@@
 Connection ~ 2625 7225
 Connection ~ 2625 7425
+$Comp
+L KobiConn_161-3509-E_Jack_3.5mm J102
+U 1 1 59A6731A
+P 10525 3450
+F 0 "J102" H 10525 4050 60  0000 C CNN
+F 1 "Jack Estereo" H 10525 3950 60  0000 C CNN
+F 2 "library:KobiConn_161-3509-E_Jack_3.5mm" H 10675 3450 60  0001 C CNN
+F 3 "http://ar.mouser.com/ProductDetail/Kobiconn/161-3509-E/?qs=sGAEpiMZZMv0W4pxf2HiV4Mt5ZQSVq1hR5HUmztPvpo%3d" H 10675 3450 60  0001 C CNN
+F 4 "KobiConn_161-3509-E" H 10525 3450 60  0001 C CNN "MPN"
+	1    10525 3450
+	0    -1   -1   0
+$EndComp
+Connection ~ 10825 2750
 $EndSCHEMATC

Commit message: Updated BNC and USB footprints
Parts:
- J103, J104: footprint library:Molex_73100-0105_BNC -> library:BNC_1-1337543-0
Changed lines of the file:
@@
 F 0 "J104" H 10585 2045 50  0000 C CNN
 F 1 "CONN_COAXIAL" V 10690 1925 50  0000 C CNN
-F 2 "library:Molex_73100-0105_BNC" H 10575 1925 50  0001 C CNN
+F 2 "library:BNC_1-1337543-0" H 10575 1925 50  0001 C CNN
 F 3 "http://ar.mouser.com/ProductDetail/TE-Connectivity-AMP/1-1337543-0/?qs=sGAEpiMZZMuLQf%252bEuFsOrkN5sFI71Kzav1a2hPGpKm8%3d" H 10575 1925 50  0001 C CNN
 F 4 "1-1337543-0" H 10575 1925 60  0001 C CNN "MPN"
@@
 F 0 "J103" H 10585 1345 50  0000 C CNN
 F 1 "CONN_COAXIAL" V 10690 1225 50  0000 C CNN
-F 2 "library:Molex_73100-0105_BNC" H 10575 1225 50  0001 C CNN
+F 2 "library:BNC_1-1337543-0" H 10575 1225 50  0001 C CNN
 F 3 "http://ar.mouser.com/ProductDetail/TE-Connectivity-AMP/1-1337543-0/?qs=sGAEpiMZZMuLQf%252bEuFsOrkN5sFI71Kzav1a2hPGpKm8%3d" H 10575 1225 50  0001 C CNN
 F 4 "1-1337543-0" H 10575 1225 60  0001 C CNN "MPN"
