File: PGA.sch (KiCad schematic (older format))
At the start: 43 parts, among them U301 CD4051BM96, U302 CD4051BM96, U303 CLC4007

Commit message: Completed part selection of analog board. Merged analog and digital boards.
Parts:
- renumbered R301 to R801, R302 to R802, R303 to R803, R304 to R804, R305 to R805, R306 to R806, R307 to R807, R308 to R808, R309 to R809, R310 to R810, R311 to R811, R312 to R812, R313 to R813, R314 to R814, R315 to R815, R316 to R816, R317 to R817, R318 to R818, R319 to R819, R320 to R820, R321 to R821, R322 to R822, R323 to R823, R324 to R824, R325 to R825, R326 to R826, R327 to R827, R328 to R828, R329 to R829, R330 to R830, R331 to R831, R332 to R832, R333 to R833, R334 to R834, R335 to R835, R336 to R836, R337 to R837, R338 to R838, R339 to R839, R340 to R840, U301 to U801, U302 to U802, U303 to U803

Commit message: Started final routing ...
Parts:
- R801, R803: footprint Resistors_SMD:R_0603 -> Resistors_SMD:R_0603_HandSoldering
- R805, R806, R807, R808, R809, R810, R811, R812, R813, R814, R815, R816, R817, R818, R819, R820, R821, R822, R823, R824, R825, R826, R827, R829, R830, R831, R832, R833, R834, R835, R836, R837, R838, R839, R840: footprint Capacitors_SMD:C_0603_HandSoldering -> Resistors_SMD:R_0603_HandSoldering
- R828: footprint Capacitors_SMD:C_0603_HandSoldering -> Resistors_SMD:R_0603

Commit message: Ended placing (?)
Parts:
- R828: footprint Resistors_SMD:R_0603 -> Resistors_SMD:R_0603_HandSoldering
Changed lines of the file:
@@
 F 0 "R828" V 7500 2625 50  0000 L CNN
 F 1 "47K" V 7550 2450 50  0000 L CNN
-F 2 "Resistors_SMD:R_0603" H 7475 2525 50  0001 C CNN
+F 2 "Resistors_SMD:R_0603_HandSoldering" H 7475 2525 50  0001 C CNN
 F 3 "http://www.mouser.com/ds/2/447/RC0603-272842.pdf" H 7475 2525 50  0001 C CNN
 F 4 "RC0603FR-0747KL" V 7475 2525 60  0001 C CNN "Manufacturer Part"

Commit message: Modified a lot of fields in components parts. BOM generated. Added BOM plugin script.
Parts:
- R801, R803: value 0 -> 0R; MPN (none) -> RC1206JR-070RL; Manufacturer Part RC1206JR-070RL -> (none)
- R802, R804: value 1G -> Let it open; Comment Let it open -> (none)
- R805, R806, R807, R808: value 470 -> 470R; MPN (none) -> RC0603FR-07470RL; Manufacturer Part RC0603JR-07470RL -> (none)
- R809, R810, R813, R814, R816, R819, R822, R825: MPN (none) -> RC0603FR-071K8L; Manufacturer Part RC0603FR-071K8L -> (none)
- R811, R812, R815, R817, R818, R820: value 220 -> 220R; MPN (none) -> RC0603JR-07220RL; Manufacturer Part RC0603JR-07220RL -> (none)
- R821, R823, R824, R826: value 100 -> 100R; MPN (none) -> RC0603FR-07100RL; Manufacturer Part RC0603FR-07100RL -> (none)
- R827, R830: MPN (none) -> RC0603FR-071KL; Manufacturer Part RC0603FR-071KL -> (none)
- R828, R831: MPN (none) -> RC0603FR-0747KL; Manufacturer Part RC0603FR-0747KL -> (none)
- R829, R832: MPN (none) -> RC0603FR-072K2L; Manufacturer Part RC0603FR-072K2L -> (none)
- R833, R834, R835, R836, R837, R838, R839, R840: value R -> Not used
- U801, U802: MPN (none) -> CD4051BM96; Manuf. Part Number CD4051BM96 -> (none)
- U803: MPN (none) -> CLC4007; Manuf. Part Number CLC4007ITP14MTR -> (none)
