File: PGA.sch (KiCad schematic (older format))
At the start: 43 parts, among them U801 CD4051BM96, U802 CD4051BM96, U803 CLC4007

Commit message: Added testpoints to schematic.
Parts:
- added J? (x2): Testpoint, library:Via-0.8mm, symbol CONN_01X01
Connections:
- wire segments 78 -> 80
Changed lines of the file:
@@
 $Descr A4 11693 8268
 encoding utf-8
-Sheet 7 11
+Sheet 5 11
 Title ""
 Date ""
@@
 Connection ~ 6725 5375
 Connection ~ 6725 5575
+$Comp
+L CONN_01X01 J?
+U 1 1 599EBDBC
+P 7900 3900
+F 0 "J?" H 7900 4000 50  0000 C CNN
+F 1 "Testpoint" V 8000 3900 50  0000 C CNN
+F 2 "library:Via-0.8mm" H 7900 3900 50  0001 C CNN
+F 3 "" H 7900 3900 50  0001 C CNN
+	1    7900 3900
+	1    0    0    -1
+$EndComp
+$Comp
+L CONN_01X01 J?
+U 1 1 599EBE1F
+P 7825 1250
+F 0 "J?" H 7825 1350 50  0000 C CNN
+F 1 "Testpoint" V 7925 1250 50  0000 C CNN
+F 2 "library:Via-0.8mm" H 7825 1250 50  0001 C CNN
+F 3 "" H 7825 1250 50  0001 C CNN
+	1    7825 1250
+	1    0    0    -1
+$EndComp
+Wire Wire Line
+	7625 1250 7625 1575
+Connection ~ 7625 1575
+Wire Wire Line
+	7700 3900 7700 4425
+Connection ~ 7700 4425
 $EndSCHEMATC

Commit message: Updated BOM and netlist
Parts:
- gave numbers to parts that had none: 2
Changed lines of the file:
@@
 Connection ~ 6725 5575
 $Comp
-L CONN_01X01 J?
+L CONN_01X01 J502
 U 1 1 599EBDBC
 P 7900 3900
-F 0 "J?" H 7900 4000 50  0000 C CNN
+F 0 "J502" H 7900 4000 50  0000 C CNN
 F 1 "Testpoint" V 8000 3900 50  0000 C CNN
 F 2 "library:Via-0.8mm" H 7900 3900 50  0001 C CNN
@@
 $EndComp
 $Comp
-L CONN_01X01 J?
+L CONN_01X01 J501
 U 1 1 599EBE1F
 P 7825 1250
-F 0 "J?" H 7825 1350 50  0000 C CNN
+F 0 "J501" H 7825 1350 50  0000 C CNN
 F 1 "Testpoint" V 7925 1250 50  0000 C CNN
 F 2 "library:Via-0.8mm" H 7825 1250 50  0001 C CNN

Commit message: DRC
Parts:
- J501, J502: footprint library:Via-0.8mm -> library:TestPoint
Changed lines of the file:
@@
 F 0 "J502" H 7900 4000 50  0000 C CNN
 F 1 "Testpoint" V 8000 3900 50  0000 C CNN
-F 2 "library:Via-0.8mm" H 7900 3900 50  0001 C CNN
+F 2 "library:TestPoint" H 7900 3900 50  0001 C CNN
 F 3 "" H 7900 3900 50  0001 C CNN
 	1    7900 3900
@@
 F 0 "J501" H 7825 1350 50  0000 C CNN
 F 1 "Testpoint" V 7925 1250 50  0000 C CNN
-F 2 "library:Via-0.8mm" H 7825 1250 50  0001 C CNN
+F 2 "library:TestPoint" H 7825 1250 50  0001 C CNN
 F 3 "" H 7825 1250 50  0001 C CNN
 	1    7825 1250

Commit message: Updated some MPN
Parts:
- R833, R834, R835, R836, R837, R838, R839, R840: DNP (none) -> 1
Changed lines of the file:
@@
 P 7725 1800
 F 0 "R833" V 7800 1875 50  0000 L CNN
-F 1 "Not used" V 7800 1725 50  0000 L CNN
+F 1 "Not used" V 7875 1725 50  0000 L CNN
 F 2 "Resistors_SMD:R_0603_HandSoldering" H 7725 1800 50  0001 C CNN
 F 3 "" H 7725 1800 50  0001 C CNN
+F 4 "1" V 7725 1800 60  0001 C CNN "DNP"
 	1    7725 1800
 	1    0    0    -1
@@
 P 7975 1825
 F 0 "R837" V 8050 1900 50  0000 L CNN
-F 1 "Not used" V 8050 1750 50  0000 L CNN
+F 1 "Not used" V 8125 1750 50  0000 L CNN
 F 2 "Resistors_SMD:R_0603_HandSoldering" H 7975 1825 50  0001 C CNN
 F 3 "" H 7975 1825 50  0001 C CNN
+F 4 "1" V 7975 1825 60  0001 C CNN "DNP"
 	1    7975 1825
 	1    0    0    -1
@@
 P 7725 2625
 F 0 "R834" V 7800 2700 50  0000 L CNN
-F 1 "Not used" V 7800 2550 50  0000 L CNN
+F 1 "Not used" V 7875 2550 50  0000 L CNN
 F 2 "Resistors_SMD:R_0603_HandSoldering" H 7725 2625 50  0001 C CNN
 F 3 "" H 7725 2625 50  0001 C CNN
+F 4 "1" V 7725 2625 60  0001 C CNN "DNP"
 	1    7725 2625
 	1    0    0    -1
@@
 P 7975 2625
 F 0 "R838" V 8050 2700 50  0000 L CNN
-F 1 "Not used" V 8050 2550 50  0000 L CNN
+F 1 "Not used" V 8125 2550 50  0000 L CNN
 F 2 "Resistors_SMD:R_0603_HandSoldering" H 7975 2625 50  0001 C CNN
 F 3 "" H 7975 2625 50  0001 C CNN
+F 4 "1" V 7975 2625 60  0001 C CNN "DNP"
 	1    7975 2625
 	1    0    0    -1
@@
 P 7725 4650
 F 0 "R835" V 7800 4725 50  0000 L CNN
-F 1 "Not used" V 7800 4575 50  0000 L CNN
+F 1 "Not used" V 7875 4625 50  0000 L CNN
 F 2 "Resistors_SMD:R_0603_HandSoldering" H 7725 4650 50  0001 C CNN
 F 3 "" H 7725 4650 50  0001 C CNN
+F 4 "1" V 7725 4650 60  0001 C CNN "DNP"
 	1    7725 4650
 	1    0    0    -1
@@
 P 7975 4675
 F 0 "R839" V 8050 4750 50  0000 L CNN
-F 1 "Not used" V 8050 4600 50  0000 L CNN
+F 1 "Not used" V 8100 4675 50  0000 L CNN
 F 2 "Resistors_SMD:R_0603_HandSoldering" H 7975 4675 50  0001 C CNN
 F 3 "" H 7975 4675 50  0001 C CNN
+F 4 "1" V 7975 4675 60  0001 C CNN "DNP"
 	1    7975 4675
 	1    0    0    -1
@@
 P 7725 5475
 F 0 "R836" V 7800 5550 50  0000 L CNN
-F 1 "Not used" V 7800 5400 50  0000 L CNN
+F 1 "Not used" V 7875 5400 50  0000 L CNN
 F 2 "Resistors_SMD:R_0603_HandSoldering" H 7725 5475 50  0001 C CNN
 F 3 "" H 7725 5475 50  0001 C CNN
+F 4 "1" V 7725 5475 60  0001 C CNN "DNP"
 	1    7725 5475
 	1    0    0    -1
@@
 P 7975 5475
 F 0 "R840" V 8050 5550 50  0000 L CNN
-F 1 "Not used" V 8050 5400 50  0000 L CNN
+F 1 "Not used" V 8125 5400 50  0000 L CNN
 F 2 "Resistors_SMD:R_0603_HandSoldering" H 7975 5475 50  0001 C CNN
 F 3 "" H 7975 5475 50  0001 C CNN
+F 4 "1" V 7975 5475 60  0001 C CNN "DNP"
 	1    7975 5475
 	1    0    0    -1
