File: PGA.sch (KiCad schematic (older format))
At the start: 45 parts, among them J501 Testpoint, J502 Testpoint, U801 CD4051BM96, U802 CD4051BM96, U803 CLC4007

Commit message: Updated MPN to components avalaible in mouser. Updating footprints now ...
Parts:
- R833, R834, R835, R836, R837, R838, R839, R840: VDC (none) -> 1

Commit message: New BOM generated with kicost
Parts:
- J501, J502, R802, R804: DNP (none) -> 1

Commit message: Renamed PN: AS4C1M16S->AS4C1M16S-7TCN; MIC5270->MIC5270-3.0YM5-TR; CLC4007->CLC4007ITP14MTR
Parts:
- U803: MPN CLC4007 -> CLC4007ITP14MTR

Commit message: Corrected PCB
Parts:
- U803: value CLC4007 -> TLV3544IPWR; MPN CLC4007ITP14MTR -> TLV3544IPWR
Changed lines of the file:
@@
 P 5225 1575
 F 0 "U803" H 5425 1750 50  0000 L CNN
-F 1 "CLC4007" H 5500 1525 50  0000 L CNN
+F 1 "TLV3544IPWR" H 5500 1525 50  0000 L CNN
 F 2 "Housings_SSOP:TSSOP-14_4.4x5mm_Pitch0.65mm" H 250 925 50  0001 C CNN
-F 3 "https://www.exar.com/content/document.ashx?id=21366" H 350 1025 50  0001 C CNN
-F 4 "CLC4007ITP14MTR" H 5425 1850 50  0001 C CNN "MPN"
+F 3 "https://www.ti.com/lit/ds/symlink/tlv3544.pdf" H 350 1025 50  0001 C CNN
+F 4 "TLV3544IPWR" H 5425 1850 50  0001 C CNN "MPN"
 	2    5225 1575
 	1    0    0    -1
@@
 P 5225 4425
 F 0 "U803" H 5425 4600 50  0000 L CNN
-F 1 "CLC4007" H 5500 4375 50  0000 L CNN
+F 1 "TLV3544IPWR" H 5500 4375 50  0000 L CNN
 F 2 "Housings_SSOP:TSSOP-14_4.4x5mm_Pitch0.65mm" H 250 3775 50  0001 C CNN
-F 3 "https://www.exar.com/content/document.ashx?id=21366" H 350 3875 50  0001 C CNN
-F 4 "CLC4007ITP14MTR" H 5425 4700 50  0001 C CNN "MPN"
+F 3 "https://www.ti.com/lit/ds/symlink/tlv3544.pdf" H 350 3875 50  0001 C CNN
+F 4 "TLV3544IPWR" H 5425 4700 50  0001 C CNN "MPN"
 	1    5225 4425
 	1    0    0    -1
@@
 F 4 "RC0603FR-071K8L" H 6950 2775 50  0001 C CNN "MPN"
 	1    6975 2550
-	1    0    0    -1
+	-1   0    0    1
 $EndComp
 $Comp
@@
 U 1 1 595D946E
 P 7225 4650
-F 0 "R824" V 7300 4725 50  0000 L CNN
-F 1 "100R" V 7275 4425 50  0000 L CNN
+F 0 "R824" V 7300 4575 50  0000 L CNN
+F 1 "100R" V 7125 4550 50  0000 L CNN
 F 2 "Resistors_SMD:R_0603_HandSoldering" H 7225 4650 50  0001 C CNN
 F 3 "http://www.mouser.com/ds/2/447/RC0603-272842.pdf" H 7225 4650 50  0001 C CNN
@@
 U 1 1 595D94F5
 P 6975 4650
-F 0 "R818" V 7025 4750 50  0000 L CNN
-F 1 "220R" V 7025 4425 50  0000 L CNN
+F 0 "R818" V 6900 4575 50  0000 L CNN
+F 1 "220R" V 7050 4575 50  0000 L CNN
 F 2 "Resistors_SMD:R_0603_HandSoldering" H 6975 4650 50  0001 C CNN
 F 3 "http://ar.mouser.com/ProductDetail/Yageo/RC0603JR-07220RL/?qs=sGAEpiMZZMtlubZbdhIBIJ0YzvSJmY5pWcxq0LcTcWE%3d" H 6975 4650 50  0001 C CNN
@@
 U 1 1 595D94FC
 P 6975 5675
-F 0 "R820" V 7005 5785 50  0000 L CNN
-F 1 "220R" V 7025 5450 50  0000 L CNN
+F 0 "R820" V 6900 5600 50  0000 L CNN
+F 1 "220R" V 7050 5600 50  0000 L CNN
 F 2 "Resistors_SMD:R_0603_HandSoldering" H 6975 5675 50  0001 C CNN
 F 3 "http://ar.mouser.com/ProductDetail/Yageo/RC0603JR-07220RL/?qs=sGAEpiMZZMtlubZbdhIBIJ0YzvSJmY5pWcxq0LcTcWE%3d" H 6975 5675 50  0001 C CNN
@@
 U 1 1 595D9503
 P 6975 5400
-F 0 "R819" V 6950 5525 50  0000 L CNN
+F 0 "R819" V 6900 5325 50  0000 L CNN
 F 1 "1K8" V 7050 5350 50  0000 L CNN
 F 2 "Resistors_SMD:R_0603_HandSoldering" H 6975 5400 50  0001 C CNN
@@
 F 4 "RC0603FR-071K8L" H 6950 5625 50  0001 C CNN "MPN"
 	1    6975 5400
-	1    0    0    -1
+	-1   0    0    1
 $EndComp
 $Comp
@@
 U 1 1 595D950A
 P 7225 5375
-F 0 "R825" V 7200 5500 50  0000 L CNN
+F 0 "R825" V 7175 5300 50  0000 L CNN
 F 1 "1K8" V 7300 5325 50  0000 L CNN
 F 2 "Resistors_SMD:R_0603_HandSoldering" H 7225 5375 50  0001 C CNN
@@
 F 4 "RC0603FR-071K8L" H 7200 5600 50  0001 C CNN "MPN"
 	1    7225 5375
-	1    0    0    -1
+	-1   0    0    1
 $EndComp
 $Comp
@@
 U 1 1 595D9511
 P 7225 5650
-F 0 "R826" V 7300 5725 50  0000 L CNN
-F 1 "100R" V 7275 5425 50  0000 L CNN
+F 0 "R826" V 7150 5550 50  0000 L CNN
+F 1 "100R" V 7300 5575 50  0000 L CNN
 F 2 "Resistors_SMD:R_0603_HandSoldering" H 7225 5650 50  0001 C CNN
 F 3 "http://www.mouser.com/ds/2/447/RC0603-272842.pdf" H 7225 5650 50  0001 C CNN
