File: Analog_Power_Supply.sch (KiCad schematic (older format))
At the start: 10 parts, among them U901 LM2776DBVR, U902 TCR2EF13, U903 MIC5270

Commit message: Added testpoints to schematic.
Parts:
- added J? (x3): Testpoint, library:Via-0.8mm, symbol CONN_01X01
Connections:
- wire segments 34 -> 36
Changed lines of the file:
@@
 $Descr A4 11693 8268
 encoding utf-8
-Sheet 8 11
+Sheet 6 11
 Title ""
 Date ""
@@
 	5900 4200 6150 4200
 Wire Wire Line
-	6075 3825 6075 4200
-Wire Wire Line
-	7425 3775 7425 4200
+	6075 3825 6075 4775
+Wire Wire Line
+	7425 3775 7425 4775
 Wire Wire Line
 	7425 3500 7425 3575
@@
 Connection ~ 6075 4200
 Connection ~ 7425 4200
+$Comp
+L CONN_01X01 J?
+U 1 1 599EBADE
+P 6275 4775
+F 0 "J?" H 6275 4875 50  0000 C CNN
+F 1 "Testpoint" V 6375 4775 50  0000 C CNN
+F 2 "library:Via-0.8mm" H 6275 4775 50  0001 C CNN
+F 3 "" H 6275 4775 50  0001 C CNN
+	1    6275 4775
+	1    0    0    -1
+$EndComp
+$Comp
+L CONN_01X01 J?
+U 1 1 599EBAFD
+P 7625 4775
+F 0 "J?" H 7625 4875 50  0000 C CNN
+F 1 "Testpoint" V 7725 4775 50  0000 C CNN
+F 2 "library:Via-0.8mm" H 7625 4775 50  0001 C CNN
+F 3 "" H 7625 4775 50  0001 C CNN
+	1    7625 4775
+	1    0    0    -1
+$EndComp
+$Comp
+L CONN_01X01 J?
+U 1 1 599EBB63
+P 7300 1625
+F 0 "J?" H 7300 1725 50  0000 C CNN
+F 1 "Testpoint" V 7400 1625 50  0000 C CNN
+F 2 "library:Via-0.8mm" H 7300 1625 50  0001 C CNN
+F 3 "" H 7300 1625 50  0001 C CNN
+	1    7300 1625
+	1    0    0    -1
+$EndComp
+Wire Wire Line
+	7100 1625 7100 2050
+Connection ~ 7100 2050
+Wire Wire Line
+	7425 4200 7400 4200
+Connection ~ 7400 4200
 $EndSCHEMATC

Commit message: Updated BOM and netlist
Parts:
- gave numbers to parts that had none: 3
Changed lines of the file:
@@
 Connection ~ 7425 4200
 $Comp
-L CONN_01X01 J?
+L CONN_01X01 J603
 U 1 1 599EBADE
 P 6275 4775
-F 0 "J?" H 6275 4875 50  0000 C CNN
+F 0 "J603" H 6275 4875 50  0000 C CNN
 F 1 "Testpoint" V 6375 4775 50  0000 C CNN
 F 2 "library:Via-0.8mm" H 6275 4775 50  0001 C CNN
@@
 $EndComp
 $Comp
-L CONN_01X01 J?
+L CONN_01X01 J605
 U 1 1 599EBAFD
 P 7625 4775
-F 0 "J?" H 7625 4875 50  0000 C CNN
+F 0 "J605" H 7625 4875 50  0000 C CNN
 F 1 "Testpoint" V 7725 4775 50  0000 C CNN
 F 2 "library:Via-0.8mm" H 7625 4775 50  0001 C CNN
@@
 $EndComp
 $Comp
-L CONN_01X01 J?
+L CONN_01X01 J604
 U 1 1 599EBB63
 P 7300 1625
-F 0 "J?" H 7300 1725 50  0000 C CNN
+F 0 "J604" H 7300 1725 50  0000 C CNN
 F 1 "Testpoint" V 7400 1625 50  0000 C CNN
 F 2 "library:Via-0.8mm" H 7300 1625 50  0001 C CNN

Commit message: DRC
Parts:
- J603, J604, J605: footprint library:Via-0.8mm -> library:TestPoint
Changed lines of the file:
@@
 F 0 "J603" H 6275 4875 50  0000 C CNN
 F 1 "Testpoint" V 6375 4775 50  0000 C CNN
-F 2 "library:Via-0.8mm" H 6275 4775 50  0001 C CNN
+F 2 "library:TestPoint" H 6275 4775 50  0001 C CNN
 F 3 "" H 6275 4775 50  0001 C CNN
 	1    6275 4775
@@
 F 0 "J605" H 7625 4875 50  0000 C CNN
 F 1 "Testpoint" V 7725 4775 50  0000 C CNN
-F 2 "library:Via-0.8mm" H 7625 4775 50  0001 C CNN
+F 2 "library:TestPoint" H 7625 4775 50  0001 C CNN
 F 3 "" H 7625 4775 50  0001 C CNN
 	1    7625 4775
@@
 F 0 "J604" H 7300 1725 50  0000 C CNN
 F 1 "Testpoint" V 7400 1625 50  0000 C CNN
-F 2 "library:Via-0.8mm" H 7300 1625 50  0001 C CNN
+F 2 "library:TestPoint" H 7300 1625 50  0001 C CNN
 F 3 "" H 7300 1625 50  0001 C CNN
 	1    7300 1625

Commit message: Updated some MPN
Parts:
- U902: value TCR2EF13 -> TCR2EF13,LM(CT; MPN TCR2EF13 -> TCR2EF13,LM(CT
Changed lines of the file:
@@
 P 6600 2200
 F 0 "U902" H 6600 1870 60  0000 C CNN
-F 1 "TCR2EF13" H 6600 1764 60  0000 C CNN
+F 1 "TCR2EF13,LM(CT" H 6600 1764 60  0000 C CNN
 F 2 "library:SC-74(5-pins)" H 4625 -1600 60  0001 C CNN
 F 3 "https://toshiba.semicon-storage.com/info/docget.jsp?did=13794&prodName=TCR2EF13" H 4225 -1700 60  0001 C CNN
-F 4 "TCR2EF13" H 6600 1970 50  0001 C CNN "MPN"
+F 4 "TCR2EF13,LM(CT" H 6600 1970 50  0001 C CNN "MPN"
 	1    6600 2200
 	1    0    0    -1
