File: RIGHT_TOP_BANKs.sch (KiCad schematic (older format))
At the start: 25 parts, among them J401 CONN_01X20, U301 iCE40-HX4K-TQ144

Commit message: Assignement of FPGA pins for analog stage control
Connections:
- net labels added: A4, A5, IOT_139, IOT_140, IOT_144, IOT_146, IOT_147, IOT_148, IOT_152, IOT_160, IOT_161, IOT_164, IOT_165, IOT_166, IOT_167, IOT_177, IOT_178
- net labels removed: ADC_16, ADC_17, DQ14, DQ15, IOR_139, IOR_140, IOR_144, IOR_146, IOR_147, IOR_148, IOR_152, IOR_160, IOR_161, IOR_164, IOR_165, IOR_166, IOR_167
Changed lines of the file:
@@
 $Descr A4 11693 8268
 encoding utf-8
-Sheet 4 11
+Sheet 11 11
 Title ""
 Date ""
@@
 	-1   0    0    -1
 $EndComp
-Text Label 6050 3600 0    60   ~ 0
-IOR_139
 Text Label 6050 3500 0    60   ~ 0
 IOR_138
 Text Label 6050 3400 0    60   ~ 0
 IOR_137
-Text Label 6050 4000 0    60   ~ 0
-IOR_146
-Text Label 6050 3900 0    60   ~ 0
-IOR_144
-Text Label 6050 3700 0    60   ~ 0
-IOR_140
 Text Notes 5150 1600 0    60   ~ 12
 FPGA BANK 1\n(RIGHT BANK)
@@
 	1    0    0    -1
 $EndComp
-Text Label 6050 4100 0    60   ~ 0
-IOR_147
-Text Label 6050 4200 0    60   ~ 0
-IOR_148
-Text Label 6050 4300 0    60   ~ 0
-IOR_152
-Text Label 6050 4400 0    60   ~ 0
-IOR_160
-Text Label 6050 4500 0    60   ~ 0
-IOR_161
-Text Label 6050 4600 0    60   ~ 0
-IOR_164
-Text Label 6050 4700 0    60   ~ 0
-IOR_165
-Text Label 6050 4800 0    60   ~ 0
-IOR_166
-Text Label 6050 4900 0    60   ~ 0
-IOR_167
 $Comp
 L C C404
@@
 IOT_174
 Text HLabel 3300 4550 0    60   BiDi ~ 12
-DQ15
+A5
 Text HLabel 3300 4650 0    60   BiDi ~ 12
-DQ14
-Wire Notes Line
-	1900 4450 2950 4450
+A4
 Text Notes 2550 4700 2    60   ~ 0
 RAM connections
-Text HLabel 3300 2750 0    60   BiDi ~ 12
+Text HLabel 3300 2950 0    60   BiDi ~ 12
 ADC_0
-Text HLabel 3300 2850 0    60   BiDi ~ 12
+Text HLabel 3300 3050 0    60   BiDi ~ 12
 ADC_1
-Text HLabel 3300 2950 0    60   BiDi ~ 12
+Text HLabel 3300 3150 0    60   BiDi ~ 12
 ADC_2
-Text HLabel 3300 3050 0    60   BiDi ~ 12
+Text HLabel 3300 3250 0    60   BiDi ~ 12
 ADC_3
-Text HLabel 3300 3150 0    60   BiDi ~ 12
+Text HLabel 3300 3350 0    60   BiDi ~ 12
 ADC_4
-Text HLabel 3300 3250 0    60   BiDi ~ 12
+Text HLabel 3300 3450 0    60   BiDi ~ 12
 ADC_5
-Text HLabel 3300 3350 0    60   BiDi ~ 12
+Text HLabel 3300 3550 0    60   BiDi ~ 12
 ADC_6
-Text HLabel 3300 3450 0    60   BiDi ~ 12
+Text HLabel 3300 3650 0    60   BiDi ~ 12
 ADC_7
-Text HLabel 3300 3550 0    60   BiDi ~ 12
+Text HLabel 3300 3750 0    60   BiDi ~ 12
 ADC_8
-Text HLabel 3300 3650 0    60   BiDi ~ 12
+Text HLabel 3300 3850 0    60   BiDi ~ 12
 ADC_9
-Text HLabel 3300 3750 0    60   BiDi ~ 12
+Text HLabel 3300 3950 0    60   BiDi ~ 12
 ADC_10
-Text HLabel 3300 3850 0    60   BiDi ~ 12
+Text HLabel 3300 4050 0    60   BiDi ~ 12
 ADC_11
-Text HLabel 3300 3950 0    60   BiDi ~ 12
+Text HLabel 3300 4150 0    60   BiDi ~ 12
 ADC_12
-Text HLabel 3300 4050 0    60   BiDi ~ 12
+Text HLabel 3300 4250 0    60   BiDi ~ 12
 ADC_13
-Text HLabel 3300 4150 0    60   BiDi ~ 12
+Text HLabel 3300 4350 0    60   BiDi ~ 12
 ADC_14
-Text HLabel 3300 4250 0    60   BiDi ~ 12
+Text HLabel 3300 4450 0    60   BiDi ~ 12
 ADC_15
-Text HLabel 3300 4350 0    60   BiDi ~ 12
-ADC_16
-Text HLabel 3300 4450 0    60   BiDi ~ 12
-ADC_17
 Text HLabel 3050 5050 0    60   Input ~ 12
 +3.3V
@@
 	1    0    0    -1
 $EndComp
-Text Label 7850 3700 2    60   ~ 0
-IOR_139
 Text Label 7850 3600 2    60   ~ 0
 IOR_138
@@
 Text Label 7850 3400 2    60   ~ 0
 IOR_136
-Text Label 7850 3800 2    60   ~ 0
-IOR_140
+Wire Notes Line
+	1800 4500 2850 4500
+Text HLabel 3300 2750 0    60   BiDi ~ 12
+IOT_177
+Text HLabel 3300 2850 0    60   BiDi ~ 12
+IOT_178
+Text HLabel 6050 3900 2    60   BiDi ~ 12
+IOT_144
+Text HLabel 6050 4000 2    60   BiDi ~ 12
+IOT_146
+Text HLabel 6050 4100 2    60   BiDi ~ 12
+IOT_147
+Text HLabel 6050 4200 2    60   BiDi ~ 12
+IOT_148
+Text HLabel 6050 4300 2    60   BiDi ~ 12
+IOT_152
+Text HLabel 6050 4400 2    60   BiDi ~ 12
+IOT_160
+Text HLabel 6050 4500 2    60   BiDi ~ 12
+IOT_161
+Text HLabel 6050 4600 2    60   BiDi ~ 12
+IOT_164
+Text HLabel 6050 4700 2    60   BiDi ~ 12
+IOT_165
+Text HLabel 6050 4800 2    60   BiDi ~ 12
+IOT_166
+Text HLabel 6050 4900 2    60   BiDi ~ 12
+IOT_167
+Text HLabel 6650 5350 2    60   Input ~ 12
++3.3V
+Text HLabel 6650 5700 2    60   Input ~ 12
+GNDD
+Text HLabel 6050 3600 2    60   BiDi ~ 12
+IOT_139
+Text HLabel 6050 3700 2    60   BiDi ~ 12
+IOT_140
+Text HLabel 7850 3700 0    60   Input ~ 12
+GNDD
+Text HLabel 7850 3800 0    60   Input ~ 12
++3.3V
 $EndSCHEMATC

Commit message: Added reset button. Delated unused fpga analog control connections. Added this connections to the expansion connector
Parts:
- removed J401: CONN_01X20, Pin_Headers:Pin_Header_Straight_1x20_Pitch1.27mm, symbol CONN_01X20
- added J1101: CONN_01X25, Pin_Headers:Pin_Header_Straight_1x25_Pitch1.27mm, symbol CONN_01X25
- added SW1101: SW_Push, Buttons_Switches_THT:SW_PUSH_6mm_h4.3mm, symbol SW_Push
Connections:
- net labels added: IOR_139, IOR_140, IOR_144, IOR_146
- net labels removed: IOT_139, IOT_140, IOT_144, IOT_146, IOT_147
- wire segments 51 -> 54
Changed lines of the file:
@@
 LIBS:voltage-references
 LIBS:voltage-regulators
+LIBS:switches
 LIBS:iCE40hxk4_dev_board-cache
 EELAYER 25 0
@@
 Wire Wire Line
 	7400 1900 7850 1900
-$Comp
-L CONN_01X20 J401
-U 1 1 59699B76
-P 8050 2850
-F 0 "J401" H 8050 3900 50  0000 C CNN
-F 1 "CONN_01X20" V 8150 2850 50  0000 C CNN
-F 2 "Pin_Headers:Pin_Header_Straight_1x20_Pitch1.27mm" H 8050 2850 50  0001 C CNN
-F 3 "" H 8050 2850 50  0001 C CNN
-	1    8050 2850
-	1    0    0    -1
-$EndComp
 Text Label 7850 3600 2    60   ~ 0
 IOR_138
@@
 Text HLabel 3300 2850 0    60   BiDi ~ 12
 IOT_178
-Text HLabel 6050 3900 2    60   BiDi ~ 12
-IOT_144
-Text HLabel 6050 4000 2    60   BiDi ~ 12
-IOT_146
-Text HLabel 6050 4100 2    60   BiDi ~ 12
-IOT_147
 Text HLabel 6050 4200 2    60   BiDi ~ 12
 IOT_148
@@
 Text HLabel 6650 5700 2    60   Input ~ 12
 GNDD
-Text HLabel 6050 3600 2    60   BiDi ~ 12
-IOT_139
-Text HLabel 6050 3700 2    60   BiDi ~ 12
-IOT_140
-Text HLabel 7850 3700 0    60   Input ~ 12
+Text HLabel 7850 4100 0    60   Input ~ 12
 GNDD
-Text HLabel 7850 3800 0    60   Input ~ 12
+Text HLabel 7850 4300 0    60   Input ~ 12
 +3.3V
+$Comp
+L SW_Push SW1101
+U 1 1 59936E4F
+P 6725 4100
+F 0 "SW1101" H 6775 4200 50  0000 L CNN
+F 1 "SW_Push" H 6725 4040 50  0000 C CNN
+F 2 "Buttons_Switches_THT:SW_PUSH_6mm_h4.3mm" H 6725 4300 50  0001 C CNN
+F 3 "" H 6725 4300 50  0001 C CNN
+	1    6725 4100
+	1    0    0    -1
+$EndComp
+Text HLabel 7025 4100 2    60   Input ~ 12
+GNDD
+Wire Wire Line
+	7025 4100 6925 4100
+$Comp
+L CONN_01X25 J1101
+U 1 1 5994C423
+P 8050 3100
+F 0 "J1101" H 8050 4400 50  0000 C CNN
+F 1 "CONN_01X25" V 8150 3100 50  0000 C CNN
+F 2 "Pin_Headers:Pin_Header_Straight_1x25_Pitch1.27mm" H 8050 3100 50  0001 C CNN
+F 3 "" H 8050 3100 50  0001 C CNN
+	1    8050 3100
+	1    0    0    -1
+$EndComp
+Text Label 7850 3800 2    60   ~ 0
+IOR_140
+Text Label 7850 3900 2    60   ~ 0
+IOR_144
+Text Label 6050 4000 0    60   ~ 0
+IOR_146
+Text Label 7850 3700 2    60   ~ 0
+IOR_139
+Wire Wire Line
+	7850 4300 7850 4200
+Text Label 6050 3600 0    60   ~ 0
+IOR_139
+Text Label 7850 4000 2    60   ~ 0
+IOR_146
+Text Label 6050 3900 0    60   ~ 0
+IOR_144
+Text Label 6050 3700 0    60   ~ 0
+IOR_140
+Wire Wire Line
+	6050 4100 6525 4100
 $EndSCHEMATC

Commit message: Added square wave output.
Connections:
- net labels added: IOT_146
- net labels removed: IOR_146
- wire segments 54 -> 55
Changed lines of the file:
@@
 Text Label 7850 3900 2    60   ~ 0
 IOR_144
-Text Label 6050 4000 0    60   ~ 0
-IOR_146
 Text Label 7850 3700 2    60   ~ 0
 IOR_139
@@
 Text Label 6050 3600 0    60   ~ 0
 IOR_139
-Text Label 7850 4000 2    60   ~ 0
-IOR_146
 Text Label 6050 3900 0    60   ~ 0
 IOR_144
@@
 Wire Wire Line
 	6050 4100 6525 4100
+Text HLabel 6050 4000 2    60   BiDi ~ 12
+IOT_146
+Wire Wire Line
+	7850 4000 7850 4100
 $EndSCHEMATC

Commit message: Modified a lot of fields in components parts. BOM generated. Added BOM plugin script.
Parts:
- C401, C402, C403, C404, C405, C407: MPN (none) -> C0603C104K3RACTU; Manufacturer Part C0603C104K3RACTU -> (none); Type (none) -> Ceramic; VDC 25V (min. 10V) -> 25V
- D401, D402, D403, D404, D405, D406, D407, D408: MPN (none) -> APTD1608LCGCK; Manufacturer Part APTD1608LCGCK -> (none)
- R401, R402, R403, R404, R405, R406, R407, R408: value 680 -> 680R; MPN (none) -> RC0603FR-07680RL; Manufacturer Part CRCW06031K50JNEA -> (none)
- U301: MPN (none) -> iCE40-HX4K-TQ144
- Xtal401: MPN (none) -> LFSPXO019966
