File: RIGHT_TOP_BANKs.sch (KiCad schematic (older format))
At the start: 26 parts, among them J1101 CONN_01X25, SW1101 SW_Push, U301 iCE40-HX4K-TQ144

Commit message: Updated MPN to components avalaible in mouser. Updating footprints now ...
Parts:
- J1101: MPN (none) -> M52-5002545
- SW1101: MPN (none) -> 1301.9309
