File: Offset.sch (KiCad schematic (older format))
At the start: 31 parts, among them U1101 MIC7300, U1102 MIC7300, U1103 MCP4716, U1104 MCP4716, U1105 MIC7300, U1106 MIC7300, U803 CLC4007

Commit message: Added testpoints to schematic.
Parts:
- added J? (x8): Testpoint, library:Via-0.8mm, symbol CONN_01X01
Connections:
- wire segments 87 -> 96
Changed lines of the file:
@@
 $Descr A4 11693 8268
 encoding utf-8
-Sheet 10 11
+Sheet 8 11
 Title ""
 Date ""
@@
 Connection ~ 3875 1700
 Connection ~ 3875 2050
+$Comp
+L CONN_01X01 J?
+U 1 1 599E2B08
+P 10100 3975
+F 0 "J?" H 10100 4075 50  0000 C CNN
+F 1 "Testpoint" V 10200 3975 50  0000 C CNN
+F 2 "library:Via-0.8mm" H 10100 3975 50  0001 C CNN
+F 3 "" H 10100 3975 50  0001 C CNN
+	1    10100 3975
+	1    0    0    -1
+$EndComp
+Wire Wire Line
+	2775 3650 2900 3650
+Connection ~ 2775 3650
+Wire Wire Line
+	5475 2875 5400 2875
+Wire Wire Line
+	5400 2875 5400 3150
+Connection ~ 5400 3150
+Wire Wire Line
+	9750 3975 9900 3975
+Connection ~ 9750 3975
+Wire Wire Line
+	6700 3675 6625 3675
+Connection ~ 6625 3675
+Wire Wire Line
+	6500 5750 6350 5750
+Connection ~ 6350 5750
+Wire Wire Line
+	9825 5900 9725 5900
+Connection ~ 9725 5900
+Wire Wire Line
+	5375 4750 5375 5225
+Connection ~ 5375 5225
+Wire Wire Line
+	2800 5625 2850 5625
+Connection ~ 2800 5625
+$Comp
+L CONN_01X01 J?
+U 1 1 599F1C55
+P 10025 5900
+F 0 "J?" H 10025 6000 50  0000 C CNN
+F 1 "Testpoint" V 10125 5900 50  0000 C CNN
+F 2 "library:Via-0.8mm" H 10025 5900 50  0001 C CNN
+F 3 "" H 10025 5900 50  0001 C CNN
+	1    10025 5900
+	1    0    0    -1
+$EndComp
+$Comp
+L CONN_01X01 J?
+U 1 1 599F1D31
+P 6700 5750
+F 0 "J?" H 6700 5850 50  0000 C CNN
+F 1 "Testpoint" V 6800 5750 50  0000 C CNN
+F 2 "library:Via-0.8mm" H 6700 5750 50  0001 C CNN
+F 3 "" H 6700 5750 50  0001 C CNN
+	1    6700 5750
+	1    0    0    -1
+$EndComp
+$Comp
+L CONN_01X01 J?
+U 1 1 599F1E16
+P 6900 3675
+F 0 "J?" H 6900 3775 50  0000 C CNN
+F 1 "Testpoint" V 7000 3675 50  0000 C CNN
+F 2 "library:Via-0.8mm" H 6900 3675 50  0001 C CNN
+F 3 "" H 6900 3675 50  0001 C CNN
+	1    6900 3675
+	1    0    0    -1
+$EndComp
+$Comp
+L CONN_01X01 J?
+U 1 1 599F1F79
+P 5675 2875
+F 0 "J?" H 5675 2975 50  0000 C CNN
+F 1 "Testpoint" V 5800 2950 50  0000 C CNN
+F 2 "library:Via-0.8mm" H 5675 2875 50  0001 C CNN
+F 3 "" H 5675 2875 50  0001 C CNN
+	1    5675 2875
+	1    0    0    -1
+$EndComp
+$Comp
+L CONN_01X01 J?
+U 1 1 599F20B1
+P 5575 4750
+F 0 "J?" H 5575 4850 50  0000 C CNN
+F 1 "Testpoint" V 5700 4825 50  0000 C CNN
+F 2 "library:Via-0.8mm" H 5575 4750 50  0001 C CNN
+F 3 "" H 5575 4750 50  0001 C CNN
+	1    5575 4750
+	1    0    0    -1
+$EndComp
+$Comp
+L CONN_01X01 J?
+U 1 1 599F21E0
+P 3100 3650
+F 0 "J?" H 3100 3750 50  0000 C CNN
+F 1 "Testpoint" V 3225 3725 50  0000 C CNN
+F 2 "library:Via-0.8mm" H 3100 3650 50  0001 C CNN
+F 3 "" H 3100 3650 50  0001 C CNN
+	1    3100 3650
+	1    0    0    -1
+$EndComp
+$Comp
+L CONN_01X01 J?
+U 1 1 599F233C
+P 3050 5625
+F 0 "J?" H 3050 5725 50  0000 C CNN
+F 1 "Testpoint" V 3175 5700 50  0000 C CNN
+F 2 "library:Via-0.8mm" H 3050 5625 50  0001 C CNN
+F 3 "" H 3050 5625 50  0001 C CNN
+	1    3050 5625
+	1    0    0    -1
+$EndComp
 $EndSCHEMATC

Commit message: Updated BOM and netlist
Parts:
- gave numbers to parts that had none: 8
Changed lines of the file:
@@
 $EndComp
 $Comp
-L GNDA #PWR038
+L GNDA #PWR801
 U 1 1 592FB96C
 P 4150 4650
-F 0 "#PWR038" H 4150 4400 50  0001 C CNN
+F 0 "#PWR801" H 4150 4400 50  0001 C CNN
 F 1 "GNDA" H 4150 4500 50  0000 C CNN
 F 2 "" H 4150 4650 50  0001 C CNN
@@
 Connection ~ 3875 2050
 $Comp
-L CONN_01X01 J?
+L CONN_01X01 J808
 U 1 1 599E2B08
 P 10100 3975
-F 0 "J?" H 10100 4075 50  0000 C CNN
+F 0 "J808" H 10100 4075 50  0000 C CNN
 F 1 "Testpoint" V 10200 3975 50  0000 C CNN
 F 2 "library:Via-0.8mm" H 10100 3975 50  0001 C CNN
@@
 Connection ~ 2800 5625
 $Comp
-L CONN_01X01 J?
+L CONN_01X01 J807
 U 1 1 599F1C55
 P 10025 5900
-F 0 "J?" H 10025 6000 50  0000 C CNN
+F 0 "J807" H 10025 6000 50  0000 C CNN
 F 1 "Testpoint" V 10125 5900 50  0000 C CNN
 F 2 "library:Via-0.8mm" H 10025 5900 50  0001 C CNN
@@
 $EndComp
 $Comp
-L CONN_01X01 J?
+L CONN_01X01 J805
 U 1 1 599F1D31
 P 6700 5750
-F 0 "J?" H 6700 5850 50  0000 C CNN
+F 0 "J805" H 6700 5850 50  0000 C CNN
 F 1 "Testpoint" V 6800 5750 50  0000 C CNN
 F 2 "library:Via-0.8mm" H 6700 5750 50  0001 C CNN
@@
 $EndComp
 $Comp
-L CONN_01X01 J?
+L CONN_01X01 J806
 U 1 1 599F1E16
 P 6900 3675
-F 0 "J?" H 6900 3775 50  0000 C CNN
+F 0 "J806" H 6900 3775 50  0000 C CNN
 F 1 "Testpoint" V 7000 3675 50  0000 C CNN
 F 2 "library:Via-0.8mm" H 6900 3675 50  0001 C CNN
@@
 $EndComp
 $Comp
-L CONN_01X01 J?
+L CONN_01X01 J804
 U 1 1 599F1F79
 P 5675 2875
-F 0 "J?" H 5675 2975 50  0000 C CNN
+F 0 "J804" H 5675 2975 50  0000 C CNN
 F 1 "Testpoint" V 5800 2950 50  0000 C CNN
 F 2 "library:Via-0.8mm" H 5675 2875 50  0001 C CNN
@@
 $EndComp
 $Comp
-L CONN_01X01 J?
+L CONN_01X01 J803
 U 1 1 599F20B1
 P 5575 4750
-F 0 "J?" H 5575 4850 50  0000 C CNN
+F 0 "J803" H 5575 4850 50  0000 C CNN
 F 1 "Testpoint" V 5700 4825 50  0000 C CNN
 F 2 "library:Via-0.8mm" H 5575 4750 50  0001 C CNN
@@
 $EndComp
 $Comp
-L CONN_01X01 J?
+L CONN_01X01 J802
 U 1 1 599F21E0
 P 3100 3650
-F 0 "J?" H 3100 3750 50  0000 C CNN
+F 0 "J802" H 3100 3750 50  0000 C CNN
 F 1 "Testpoint" V 3225 3725 50  0000 C CNN
 F 2 "library:Via-0.8mm" H 3100 3650 50  0001 C CNN
@@
 $EndComp
 $Comp
-L CONN_01X01 J?
+L CONN_01X01 J801
 U 1 1 599F233C
 P 3050 5625
-F 0 "J?" H 3050 5725 50  0000 C CNN
+F 0 "J801" H 3050 5725 50  0000 C CNN
 F 1 "Testpoint" V 3175 5700 50  0000 C CNN
 F 2 "library:Via-0.8mm" H 3050 5625 50  0001 C CNN

Commit message: Updated schematic
Parts:
- added J? (x2): Testpoint, library:Via-0.8mm, symbol CONN_01X01
- U1103: MPN MCP4716 -> MCP4716A1-E/CH
- U1104: MPN MCP4716 -> MCP4716A0-E/CH
Connections:
- wire segments 96 -> 99
Changed lines of the file:
@@
 LIBS:switches
 LIBS:iCE40hxk4_dev_board-cache
-EELAYER 26 0
+EELAYER 25 0
 EELAYER END
 $Descr A4 11693 8268
@@
 F 2 "TO_SOT_Packages_SMD:SOT-23-6" H 5075 3150 60  0001 C CNN
 F 3 "http://ww1.microchip.com/downloads/en/DeviceDoc/22272C.pdf" H 4575 2450 60  0001 C CNN
-F 4 "MCP4716" H 5325 3100 50  0001 C CNN "MPN"
+F 4 "MCP4716A0-E/CH" H 5325 3100 50  0001 C CNN "MPN"
 	1    5025 3150
 	1    0    0    -1
@@
 F 2 "TO_SOT_Packages_SMD:SOT-23-6" H 4725 5150 60  0001 C CNN
 F 3 "http://ww1.microchip.com/downloads/en/DeviceDoc/22272C.pdf" H 4225 4450 60  0001 C CNN
-F 4 "MCP4716" H 4850 5550 50  0001 C CNN "MPN"
+F 4 "MCP4716A1-E/CH" H 4850 5550 50  0001 C CNN "MPN"
 	1    4675 5150
 	1    0    0    -1
@@
 Text Label 1475 5750 2    60   ~ 0
 GND_A
+$Comp
+L CONN_01X01 J808
+U 1 1 599E2B08
+P 10100 3975
+F 0 "J808" H 10100 4075 50  0000 C CNN
+F 1 "Testpoint" V 10200 3975 50  0000 C CNN
+F 2 "library:Via-0.8mm" H 10100 3975 50  0001 C CNN
+F 3 "" H 10100 3975 50  0001 C CNN
+	1    10100 3975
+	1    0    0    -1
+$EndComp
+$Comp
+L CONN_01X01 J807
+U 1 1 599F1C55
+P 10025 5900
+F 0 "J807" H 10025 6000 50  0000 C CNN
+F 1 "Testpoint" V 10125 5900 50  0000 C CNN
+F 2 "library:Via-0.8mm" H 10025 5900 50  0001 C CNN
+F 3 "" H 10025 5900 50  0001 C CNN
+	1    10025 5900
+	1    0    0    -1
+$EndComp
+$Comp
+L CONN_01X01 J805
+U 1 1 599F1D31
+P 6700 5750
+F 0 "J805" H 6700 5850 50  0000 C CNN
+F 1 "Testpoint" V 6800 5750 50  0000 C CNN
+F 2 "library:Via-0.8mm" H 6700 5750 50  0001 C CNN
+F 3 "" H 6700 5750 50  0001 C CNN
+	1    6700 5750
+	1    0    0    -1
+$EndComp
+$Comp
+L CONN_01X01 J806
+U 1 1 599F1E16
+P 6900 3675
+F 0 "J806" H 6900 3775 50  0000 C CNN
+F 1 "Testpoint" V 7000 3675 50  0000 C CNN
+F 2 "library:Via-0.8mm" H 6900 3675 50  0001 C CNN
+F 3 "" H 6900 3675 50  0001 C CNN
+	1    6900 3675
+	1    0    0    -1
+$EndComp
+$Comp
+L CONN_01X01 J804
+U 1 1 599F1F79
+P 5675 2875
+F 0 "J804" H 5675 2975 50  0000 C CNN
+F 1 "Testpoint" V 5800 2950 50  0000 C CNN
+F 2 "library:Via-0.8mm" H 5675 2875 50  0001 C CNN
+F 3 "" H 5675 2875 50  0001 C CNN
+	1    5675 2875
+	1    0    0    -1
+$EndComp
+$Comp
+L CONN_01X01 J803
+U 1 1 599F20B1
+P 5575 4750
+F 0 "J803" H 5575 4850 50  0000 C CNN
+F 1 "Testpoint" V 5700 4825 50  0000 C CNN
+F 2 "library:Via-0.8mm" H 5575 4750 50  0001 C CNN
+F 3 "" H 5575 4750 50  0001 C CNN
+	1    5575 4750
+	1    0    0    -1
+$EndComp
+$Comp
+L CONN_01X01 J802
+U 1 1 599F21E0
+P 3100 3650
+F 0 "J802" H 3100 3750 50  0000 C CNN
+F 1 "Testpoint" V 3225 3725 50  0000 C CNN
+F 2 "library:Via-0.8mm" H 3100 3650 50  0001 C CNN
+F 3 "" H 3100 3650 50  0001 C CNN
+	1    3100 3650
+	1    0    0    -1
+$EndComp
+$Comp
+L CONN_01X01 J801
+U 1 1 599F233C
+P 3050 5625
+F 0 "J801" H 3050 5725 50  0000 C CNN
+F 1 "Testpoint" V 3175 5700 50  0000 C CNN
+F 2 "library:Via-0.8mm" H 3050 5625 50  0001 C CNN
+F 3 "" H 3050 5625 50  0001 C CNN
+	1    3050 5625
+	1    0    0    -1
+$EndComp
+$Comp
+L CONN_01X01 J?
+U 1 1 599F7542
+P 4675 1250
+F 0 "J?" H 4675 1350 50  0000 C CNN
+F 1 "Testpoint" V 4800 1325 50  0000 C CNN
+F 2 "library:Via-0.8mm" H 4675 1250 50  0001 C CNN
+F 3 "" H 4675 1250 50  0001 C CNN
+	1    4675 1250
+	1    0    0    -1
+$EndComp
+$Comp
+L CONN_01X01 J?
+U 1 1 599F7603
+P 4650 1875
+F 0 "J?" H 4650 1975 50  0000 C CNN
+F 1 "Testpoint" V 4775 1950 50  0000 C CNN
+F 2 "library:Via-0.8mm" H 4650 1875 50  0001 C CNN
+F 3 "" H 4650 1875 50  0001 C CNN
+	1    4650 1875
+	1    0    0    -1
+$EndComp
 Wire Wire Line
 	1050 725  1200 725
@@
 	4375 2675 4550 2675
 Wire Wire Line
-	4125 1750 4125 1600
+	4125 1250 4125 1750
 Wire Wire Line
 	3875 1750 3875 1700
@@
 Connection ~ 3875 1700
 Connection ~ 3875 2050
-$Comp
-L CONN_01X01 J808
-U 1 1 599E2B08
-P 10100 3975
-F 0 "J808" H 10100 4075 50  0000 C CNN
-F 1 "Testpoint" V 10200 3975 50  0000 C CNN
-F 2 "library:Via-0.8mm" H 10100 3975 50  0001 C CNN
-F 3 "" H 10100 3975 50  0001 C CNN
-	1    10100 3975
-	1    0    0    -1
-$EndComp
 Wire Wire Line
 	2775 3650 2900 3650
@@
 	2800 5625 2850 5625
 Connection ~ 2800 5625
-$Comp
-L CONN_01X01 J807
-U 1 1 599F1C55
-P 10025 5900
-F 0 "J807" H 10025 6000 50  0000 C CNN
-F 1 "Testpoint" V 10125 5900 50  0000 C CNN
-F 2 "library:Via-0.8mm" H 10025 5900 50  0001 C CNN
-F 3 "" H 10025 5900 50  0001 C CNN
-	1    10025 5900
-	1    0    0    -1
-$EndComp
-$Comp
-L CONN_01X01 J805
-U 1 1 599F1D31
-P 6700 5750
-F 0 "J805" H 6700 5850 50  0000 C CNN
-F 1 "Testpoint" V 6800 5750 50  0000 C CNN
-F 2 "library:Via-0.8mm" H 6700 5750 50  0001 C CNN
-F 3 "" H 6700 5750 50  0001 C CNN
-	1    6700 5750
-	1    0    0    -1
-$EndComp
-$Comp
-L CONN_01X01 J806
-U 1 1 599F1E16
-P 6900 3675
-F 0 "J806" H 6900 3775 50  0000 C CNN
-F 1 "Testpoint" V 7000 3675 50  0000 C CNN
-F 2 "library:Via-0.8mm" H 6900 3675 50  0001 C CNN
-F 3 "" H 6900 3675 50  0001 C CNN
-	1    6900 3675
-	1    0    0    -1
-$EndComp
-$Comp
-L CONN_01X01 J804
-U 1 1 599F1F79
-P 5675 2875
-F 0 "J804" H 5675 2975 50  0000 C CNN
-F 1 "Testpoint" V 5800 2950 50  0000 C CNN
-F 2 "library:Via-0.8mm" H 5675 2875 50  0001 C CNN
-F 3 "" H 5675 2875 50  0001 C CNN
-	1    5675 2875
-	1    0    0    -1
-$EndComp
-$Comp
-L CONN_01X01 J803
-U 1 1 599F20B1
-P 5575 4750
-F 0 "J803" H 5575 4850 50  0000 C CNN
-F 1 "Testpoint" V 5700 4825 50  0000 C CNN
-F 2 "library:Via-0.8mm" H 5575 4750 50  0001 C CNN
-F 3 "" H 5575 4750 50  0001 C CNN
-	1    5575 4750
-	1    0    0    -1
-$EndComp
-$Comp
-L CONN_01X01 J802
-U 1 1 599F21E0
-P 3100 3650
-F 0 "J802" H 3100 3750 50  0000 C CNN
-F 1 "Testpoint" V 3225 3725 50  0000 C CNN
-F 2 "library:Via-0.8mm" H 3100 3650 50  0001 C CNN
-F 3 "" H 3100 3650 50  0001 C CNN
-	1    3100 3650
-	1    0    0    -1
-$EndComp
-$Comp
-L CONN_01X01 J801
-U 1 1 599F233C
-P 3050 5625
-F 0 "J801" H 3050 5725 50  0000 C CNN
-F 1 "Testpoint" V 3175 5700 50  0000 C CNN
-F 2 "library:Via-0.8mm" H 3050 5625 50  0001 C CNN
-F 3 "" H 3050 5625 50  0001 C CNN
-	1    3050 5625
-	1    0    0    -1
-$EndComp
+Wire Wire Line
+	4475 1250 4125 1250
+Wire Wire Line
+	4450 1875 4250 1875
+Wire Wire Line
+	4250 1875 4250 1700
+Connection ~ 4250 1700
 $EndSCHEMATC

Commit message: Doing re-routing
Parts:
- gave numbers to parts that had none: 2
Changed lines of the file:
@@
 $EndComp
 $Comp
-L GNDA #PWR801
+L GNDA #PWR038
 U 1 1 592FB96C
 P 4150 4650
-F 0 "#PWR801" H 4150 4400 50  0001 C CNN
+F 0 "#PWR038" H 4150 4400 50  0001 C CNN
 F 1 "GNDA" H 4150 4500 50  0000 C CNN
 F 2 "" H 4150 4650 50  0001 C CNN
@@
 $EndComp
 $Comp
-L CONN_01X01 J?
+L CONN_01X01 J810
 U 1 1 599F7542
 P 4675 1250
-F 0 "J?" H 4675 1350 50  0000 C CNN
+F 0 "J810" H 4675 1350 50  0000 C CNN
 F 1 "Testpoint" V 4800 1325 50  0000 C CNN
 F 2 "library:Via-0.8mm" H 4675 1250 50  0001 C CNN
@@
 $EndComp
 $Comp
-L CONN_01X01 J?
+L CONN_01X01 J809
 U 1 1 599F7603
 P 4650 1875
-F 0 "J?" H 4650 1975 50  0000 C CNN
+F 0 "J809" H 4650 1975 50  0000 C CNN
 F 1 "Testpoint" V 4775 1950 50  0000 C CNN
 F 2 "library:Via-0.8mm" H 4650 1875 50  0001 C CNN

Commit message: DRC
Parts:
- J801, J802, J803, J804, J805, J806, J807, J808, J809, J810: footprint library:Via-0.8mm -> library:TestPoint
Changed lines of the file:
@@
 F 0 "J808" H 10100 4075 50  0000 C CNN
 F 1 "Testpoint" V 10200 3975 50  0000 C CNN
-F 2 "library:Via-0.8mm" H 10100 3975 50  0001 C CNN
+F 2 "library:TestPoint" H 10100 3975 50  0001 C CNN
 F 3 "" H 10100 3975 50  0001 C CNN
 	1    10100 3975
@@
 F 0 "J807" H 10025 6000 50  0000 C CNN
 F 1 "Testpoint" V 10125 5900 50  0000 C CNN
-F 2 "library:Via-0.8mm" H 10025 5900 50  0001 C CNN
+F 2 "library:TestPoint" H 10025 5900 50  0001 C CNN
 F 3 "" H 10025 5900 50  0001 C CNN
 	1    10025 5900
@@
 F 0 "J805" H 6700 5850 50  0000 C CNN
 F 1 "Testpoint" V 6800 5750 50  0000 C CNN
-F 2 "library:Via-0.8mm" H 6700 5750 50  0001 C CNN
+F 2 "library:TestPoint" H 6700 5750 50  0001 C CNN
 F 3 "" H 6700 5750 50  0001 C CNN
 	1    6700 5750
@@
 F 0 "J806" H 6900 3775 50  0000 C CNN
 F 1 "Testpoint" V 7000 3675 50  0000 C CNN
-F 2 "library:Via-0.8mm" H 6900 3675 50  0001 C CNN
+F 2 "library:TestPoint" H 6900 3675 50  0001 C CNN
 F 3 "" H 6900 3675 50  0001 C CNN
 	1    6900 3675
@@
 F 0 "J804" H 5675 2975 50  0000 C CNN
 F 1 "Testpoint" V 5800 2950 50  0000 C CNN
-F 2 "library:Via-0.8mm" H 5675 2875 50  0001 C CNN
+F 2 "library:TestPoint" H 5675 2875 50  0001 C CNN
 F 3 "" H 5675 2875 50  0001 C CNN
 	1    5675 2875
@@
 F 0 "J803" H 5575 4850 50  0000 C CNN
 F 1 "Testpoint" V 5700 4825 50  0000 C CNN
-F 2 "library:Via-0.8mm" H 5575 4750 50  0001 C CNN
+F 2 "library:TestPoint" H 5575 4750 50  0001 C CNN
 F 3 "" H 5575 4750 50  0001 C CNN
 	1    5575 4750
@@
 F 0 "J802" H 3100 3750 50  0000 C CNN
 F 1 "Testpoint" V 3225 3725 50  0000 C CNN
-F 2 "library:Via-0.8mm" H 3100 3650 50  0001 C CNN
+F 2 "library:TestPoint" H 3100 3650 50  0001 C CNN
 F 3 "" H 3100 3650 50  0001 C CNN
 	1    3100 3650
@@
 F 0 "J801" H 3050 5725 50  0000 C CNN
 F 1 "Testpoint" V 3175 5700 50  0000 C CNN
-F 2 "library:Via-0.8mm" H 3050 5625 50  0001 C CNN
+F 2 "library:TestPoint" H 3050 5625 50  0001 C CNN
 F 3 "" H 3050 5625 50  0001 C CNN
 	1    3050 5625
@@
 F 0 "J810" H 4675 1350 50  0000 C CNN
 F 1 "Testpoint" V 4800 1325 50  0000 C CNN
-F 2 "library:Via-0.8mm" H 4675 1250 50  0001 C CNN
+F 2 "library:TestPoint" H 4675 1250 50  0001 C CNN
 F 3 "" H 4675 1250 50  0001 C CNN
 	1    4675 1250
@@
 F 0 "J809" H 4650 1975 50  0000 C CNN
 F 1 "Testpoint" V 4775 1950 50  0000 C CNN
-F 2 "library:Via-0.8mm" H 4650 1875 50  0001 C CNN
+F 2 "library:TestPoint" H 4650 1875 50  0001 C CNN
 F 3 "" H 4650 1875 50  0001 C CNN
 	1    4650 1875
