File: Offset.sch (KiCad schematic (older format))
At the start: 41 parts, among them J801 Testpoint, J802 Testpoint, J803 Testpoint, J804 Testpoint, J805 Testpoint, J806 Testpoint, J807 Testpoint, J808 Testpoint, J809 Testpoint, J810 Testpoint, U1101 MIC7300, U1102 MIC7300, U1103 MCP4716, U1104 MCP4716, U1105 MIC7300, U1106 MIC7300, U803 CLC4007

Commit message: Updated some MPN
Parts:
- U1103: MPN MCP4716A1-E/CH -> MCP4716A1T-E/CH
- U1104: MPN MCP4716A0-E/CH -> MCP4716A0T-E/CH
Changed lines of the file:
@@
 F 2 "TO_SOT_Packages_SMD:SOT-23-6" H 5075 3150 60  0001 C CNN
 F 3 "http://ww1.microchip.com/downloads/en/DeviceDoc/22272C.pdf" H 4575 2450 60  0001 C CNN
-F 4 "MCP4716A0-E/CH" H 5325 3100 50  0001 C CNN "MPN"
+F 4 "MCP4716A0T-E/CH" H 5325 3100 50  0001 C CNN "MPN"
 	1    5025 3150
 	1    0    0    -1
@@
 F 2 "TO_SOT_Packages_SMD:SOT-23-6" H 4725 5150 60  0001 C CNN
 F 3 "http://ww1.microchip.com/downloads/en/DeviceDoc/22272C.pdf" H 4225 4450 60  0001 C CNN
-F 4 "MCP4716A1-E/CH" H 4850 5550 50  0001 C CNN "MPN"
+F 4 "MCP4716A1T-E/CH" H 4850 5550 50  0001 C CNN "MPN"
 	1    4675 5150
 	1    0    0    -1
 $EndComp
 $Comp
-L GNDA #PWR801
+L GNDA #PWR038
 U 1 1 592FB96C
 P 4150 4650
-F 0 "#PWR801" H 4150 4400 50  0001 C CNN
+F 0 "#PWR038" H 4150 4400 50  0001 C CNN
 F 1 "GNDA" H 4150 4500 50  0000 C CNN
 F 2 "" H 4150 4650 50  0001 C CNN

Commit message: New BOM generated with kicost
Parts:
- J801, J802, J803, J804, J805, J806, J807, J808, J809, J810, R1101, R1102: DNP (none) -> 1

Commit message: Renamed PN: AS4C1M16S->AS4C1M16S-7TCN; MIC5270->MIC5270-3.0YM5-TR; CLC4007->CLC4007ITP14MTR
Parts:
- U803: MPN CLC4007 -> CLC4007ITP14MTR
