File: Offset.sch (KiCad schematic (older format))
At the start: 41 parts, among them J801 Testpoint, J802 Testpoint, J803 Testpoint, J804 Testpoint, J805 Testpoint, J806 Testpoint, J807 Testpoint, J808 Testpoint, J809 Testpoint, J810 Testpoint, U1101 MIC7300, U1102 MIC7300, U1103 MCP4716, U1104 MCP4716, U1105 MIC7300, U1106 MIC7300, U803 CLC4007

Commit message: New version of mainboard. Corrected errors and modified analog part.
Parts:
- U803: value CLC4007 -> TLV3544IPWR; MPN CLC4007ITP14MTR -> TLV3544IPWR
Changed lines of the file:
@@
 P 9325 3450
 F 0 "U803" H 9500 3825 50  0000 L CNN
-F 1 "CLC4007" H 9450 3750 50  0000 L CNN
+F 1 "TLV3544IPWR" H 9450 3750 50  0000 L CNN
 F 2 "Housings_SSOP:TSSOP-14_4.4x5mm_Pitch0.65mm" H 4350 2800 50  0001 C CNN
-F 3 "https://www.exar.com/content/document.ashx?id=21366" H 4450 2900 50  0001 C CNN
-F 4 "CLC4007ITP14MTR" H 9500 3925 50  0001 C CNN "MPN"
+F 3 "https://www.ti.com/lit/ds/symlink/tlv3544.pdf" H 4450 2900 50  0001 C CNN
+F 4 "TLV3544IPWR" H 9500 3925 50  0001 C CNN "MPN"
 	3    9325 3450
 	1    0    0    -1
@@
 P 9300 5425
 F 0 "U803" H 9475 5800 50  0000 L CNN
-F 1 "CLC4007" H 9425 5725 50  0000 L CNN
+F 1 "TLV3544IPWR" H 9425 5725 50  0000 L CNN
 F 2 "Housings_SSOP:TSSOP-14_4.4x5mm_Pitch0.65mm" H 4325 4775 50  0001 C CNN
-F 3 "https://www.exar.com/content/document.ashx?id=21366" H 4425 4875 50  0001 C CNN
-F 4 "CLC4007ITP14MTR" H 9475 5900 50  0001 C CNN "MPN"
+F 3 "https://www.ti.com/lit/ds/symlink/tlv3544.pdf" H 4425 4875 50  0001 C CNN
+F 4 "TLV3544IPWR" H 9475 5900 50  0001 C CNN "MPN"
 	4    9300 5425
 	1    0    0    -1
@@
 $EndComp
 $Comp
-L GNDA #PWR037
+L GNDA #PWR038
 U 1 1 592FB96C
 P 4150 4650
-F 0 "#PWR037" H 4150 4400 50  0001 C CNN
+F 0 "#PWR038" H 4150 4400 50  0001 C CNN
 F 1 "GNDA" H 4150 4500 50  0000 C CNN
 F 2 "" H 4150 4650 50  0001 C CNN

Commit message: changed ref of adc (2.5V-->2V), and Rf of last amp stage (62K-->51K)
Parts:
- R1121, R1122: value 62K -> 51K
Changed lines of the file:
@@
 U 1 1 58FE9F45
 P 9375 6100
-F 0 "R1121" V 9275 6050 50  0000 L CNN
-F 1 "62K" V 9425 6000 50  0000 L CNN
+F 0 "R1121" V 9275 5975 50  0000 L CNN
+F 1 "51K" V 9450 6025 50  0000 L CNN
 F 2 "Resistors_SMD:R_0603_HandSoldering" H 9375 6100 50  0001 C CNN
 F 3 "http://www.mouser.com/ds/2/447/RC0603-272842.pdf" H 9375 6100 50  0001 C CNN
@@
 U 1 1 58FE9F4B
 P 8775 6100
-F 0 "R1119" V 8675 6050 50  0000 L CNN
-F 1 "6K8" V 8825 6000 50  0000 L CNN
+F 0 "R1119" V 8675 6000 50  0000 L CNN
+F 1 "6K8" V 8850 6025 50  0000 L CNN
 F 2 "Resistors_SMD:R_0603_HandSoldering" H 8775 6100 50  0001 C CNN
 F 3 "http://www.mouser.com/ds/2/447/RC0603-272842.pdf" H 8775 6100 50  0001 C CNN
@@
 U 1 1 59674700
 P 9400 4125
-F 0 "R1122" V 9300 4075 50  0000 L CNN
-F 1 "62K" V 9450 4025 50  0000 L CNN
+F 0 "R1122" V 9300 4025 50  0000 L CNN
+F 1 "51K" V 9475 4050 50  0000 L CNN
 F 2 "Resistors_SMD:R_0603_HandSoldering" H 9400 4125 50  0001 C CNN
 F 3 "http://www.mouser.com/ds/2/447/RC0603-272842.pdf" H 9400 4125 50  0001 C CNN
@@
 U 1 1 59674838
 P 8800 4125
-F 0 "R1120" V 8700 4075 50  0000 L CNN
-F 1 "6K8" V 8850 4025 50  0000 L CNN
+F 0 "R1120" V 8700 4025 50  0000 L CNN
+F 1 "6K8" V 8875 4050 50  0000 L CNN
 F 2 "Resistors_SMD:R_0603_HandSoldering" H 8800 4125 50  0001 C CNN
 F 3 "http://www.mouser.com/ds/2/447/RC0603-272842.pdf" H 8800 4125 50  0001 C CNN

Commit message: Changed resistance values in last offset stage
Parts:
- R1111, R1112: value 330R -> 1K2
- R1114, R1117: value 1K2 -> 4K7//4K7
- R1115, R1118: value 1K -> 1K5
- R1119, R1120: value 6K8 -> 1K8
- R1121, R1122: value 51K -> 12K
Changed lines of the file:
@@
 P 8500 2925
 F 0 "R1112" V 8425 2800 50  0000 L CNN
-F 1 "330R" V 8575 2900 50  0000 L CNN
+F 1 "1K2" V 8575 2900 50  0000 L CNN
 F 2 "Resistors_SMD:R_0603_HandSoldering" H 8500 2925 50  0001 C CNN
 F 3 "http://www.mouser.com/ds/2/447/RC0603-272842.pdf" H 8500 2925 50  0001 C CNN
@@
 P 8750 5125
 F 0 "R1114" V 8800 4900 50  0000 L CNN
-F 1 "1K2" V 8825 5075 50  0000 L CNN
+F 1 "4K7//4K7" V 8650 4825 50  0000 L CNN
 F 2 "Resistors_SMD:R_0603_HandSoldering" H 8750 5125 50  0001 C CNN
 F 3 "http://www.mouser.com/ds/2/447/RC0603-272842.pdf" H 8750 5125 50  0001 C CNN
@@
 P 9375 6100
 F 0 "R1121" V 9275 5975 50  0000 L CNN
-F 1 "51K" V 9450 6025 50  0000 L CNN
+F 1 "12K" V 9450 6025 50  0000 L CNN
 F 2 "Resistors_SMD:R_0603_HandSoldering" H 9375 6100 50  0001 C CNN
 F 3 "http://www.mouser.com/ds/2/447/RC0603-272842.pdf" H 9375 6100 50  0001 C CNN
@@
 P 8775 6100
 F 0 "R1119" V 8675 6000 50  0000 L CNN
-F 1 "6K8" V 8850 6025 50  0000 L CNN
+F 1 "1K8" V 8850 6025 50  0000 L CNN
 F 2 "Resistors_SMD:R_0603_HandSoldering" H 8775 6100 50  0001 C CNN
 F 3 "http://www.mouser.com/ds/2/447/RC0603-272842.pdf" H 8775 6100 50  0001 C CNN
@@
 P 8775 3350
 F 0 "R1118" V 8850 3425 50  0000 L CNN
-F 1 "1K" V 8825 3150 50  0000 L CNN
+F 1 "1K5" V 8825 3150 50  0000 L CNN
 F 2 "Resistors_SMD:R_0603_HandSoldering" H 8775 3350 50  0001 C CNN
 F 3 "http://www.mouser.com/ds/2/447/RC0603-272842.pdf" H 8775 3350 50  0001 C CNN
@@
 P 8750 5325
 F 0 "R1115" V 8825 5400 50  0000 L CNN
-F 1 "1K" V 8800 5125 50  0000 L CNN
+F 1 "1K5" V 8800 5125 50  0000 L CNN
 F 2 "Resistors_SMD:R_0603_HandSoldering" H 8750 5325 50  0001 C CNN
 F 3 "http://www.mouser.com/ds/2/447/RC0603-272842.pdf" H 8750 5325 50  0001 C CNN
@@
 P 8475 4900
 F 0 "R1111" V 8400 4775 50  0000 L CNN
-F 1 "330R" V 8550 4875 50  0000 L CNN
+F 1 "1K2" V 8550 4875 50  0000 L CNN
 F 2 "Resistors_SMD:R_0603_HandSoldering" H 8475 4900 50  0001 C CNN
 F 3 "http://www.mouser.com/ds/2/447/RC0603-272842.pdf" H 8475 4900 50  0001 C CNN
@@
 P 9400 4125
 F 0 "R1122" V 9300 4025 50  0000 L CNN
-F 1 "51K" V 9475 4050 50  0000 L CNN
+F 1 "12K" V 9475 4050 50  0000 L CNN
 F 2 "Resistors_SMD:R_0603_HandSoldering" H 9400 4125 50  0001 C CNN
 F 3 "http://www.mouser.com/ds/2/447/RC0603-272842.pdf" H 9400 4125 50  0001 C CNN
@@
 P 8800 4125
 F 0 "R1120" V 8700 4025 50  0000 L CNN
-F 1 "6K8" V 8875 4050 50  0000 L CNN
+F 1 "1K8" V 8875 4050 50  0000 L CNN
 F 2 "Resistors_SMD:R_0603_HandSoldering" H 8800 4125 50  0001 C CNN
 F 3 "http://www.mouser.com/ds/2/447/RC0603-272842.pdf" H 8800 4125 50  0001 C CNN
@@
 P 8775 3150
 F 0 "R1117" V 8825 2925 50  0000 L CNN
-F 1 "1K2" V 8850 3100 50  0000 L CNN
+F 1 "4K7//4K7" V 8675 2800 50  0000 L CNN
 F 2 "Resistors_SMD:R_0603_HandSoldering" H 8775 3150 50  0001 C CNN
 F 3 "http://www.mouser.com/ds/2/447/RC0603-272842.pdf" H 8775 3150 50  0001 C CNN
