File: USB+OSCILLATOR+REGULATOR.sch (KiCad schematic (older format))
At the start: 79 parts, among them J1001 Testpoint, J1002 Testpoint, J1003 Testpoint, J1004 Testpoint, J201 CONN_01X02, J202 USB_OTG, U201 MIC2005A-2YM5, U203 93LC56BT-I/O, U204 MIC5355/6-xYMME, U205 FT2232H

Commit message: replaced external dc connector: usb instead of pines. Sí, pines
Parts:
- removed J201: CONN_01X02, Pin_Headers:Pin_Header_Angled_1x02_Pitch1.27mm, symbol CONN_01X02
- added J?: USB_EXT, Connect:USB_Micro-B, symbol USB_OTG
Connections:
- wire segments 164 -> 163
- no-connect marks 14 -> 17
Changed lines of the file:
@@
 LIBS:switches
 LIBS:iCE40hxk4_dev_board-cache
-EELAYER 25 0
+EELAYER 26 0
 EELAYER END
 $Descr A4 11693 8268
@@
 $EndComp
 $Comp
-L CONN_01X02 J201
-U 1 1 58E0AC97
-P 1000 1050
-F 0 "J201" H 1000 1200 50  0000 C CNN
-F 1 "CONN_01X02" V 1100 1050 50  0000 C CNN
-F 2 "Pin_Headers:Pin_Header_Angled_1x02_Pitch1.27mm" H 1000 1050 50  0001 C CNN
-F 3 "" H 1000 1050 50  0001 C CNN
-	1    1000 1050
-	-1   0    0    1
-$EndComp
-$Comp
 L D_Schottky D201
 U 1 1 58E0BC42
@@
 L PWR_FLAG #FLG1001
 U 1 1 58F8188C
-P 900 1550
-F 0 "#FLG1001" H 900 1625 50  0001 C CNN
-F 1 "PWR_FLAG" H 900 1700 50  0000 C CNN
-F 2 "" H 900 1550 50  0001 C CNN
-F 3 "" H 900 1550 50  0001 C CNN
-	1    900  1550
-	1    0    0    -1
+P 800 1800
+F 0 "#FLG1001" H 800 1875 50  0001 C CNN
+F 1 "PWR_FLAG" H 800 1950 50  0000 C CNN
+F 2 "" H 800 1800 50  0001 C CNN
+F 3 "" H 800 1800 50  0001 C CNN
+	1    800  1800
+	0    -1   -1   0
 $EndComp
 $Comp
@@
 Text HLabel 5550 1600 0    60   Output ~ 12
 GNDD
-Text HLabel 1350 1450 2    60   Output ~ 12
+Text HLabel 1200 1800 2    60   Output ~ 12
 GND
 Text HLabel 6400 2900 0    60   Output ~ 12
@@
 	2350 2450 2400 2450
 Wire Wire Line
-	1200 1100 1250 1100
-Wire Wire Line
-	1200 1000 1500 1000
+	1100 1000 1500 1000
 Wire Wire Line
 	1400 1300 3750 1300
@@
 	8650 950  8750 950
 Wire Wire Line
-	1350 1450 1250 1450
-Wire Wire Line
-	1250 1100 1250 1550
-Wire Wire Line
 	6400 2900 6500 2900
 Wire Wire Line
@@
 Wire Wire Line
 	3800 4950 4100 4950
-Wire Wire Line
-	1250 1550 900  1550
 Wire Wire Line
 	3650 3700 3750 3700
@@
 Connection ~ 3950 4650
 Connection ~ 3950 4950
-Connection ~ 1250 1450
 Connection ~ 3750 4000
 Connection ~ 5700 2650
@@
 	5300 1800 5275 1800
 Connection ~ 5300 1900
+$Comp
+L USB_OTG J?
+U 1 1 599EBDA6
+P 800 1200
+F 0 "J?" H 600 1650 50  0000 L CNN
+F 1 "USB_EXT" H 600 1550 50  0000 L CNN
+F 2 "Connect:USB_Micro-B" H 950 1150 50  0001 C CNN
+F 3 "" H 950 1150 50  0001 C CNN
+	1    800  1200
+	1    0    0    -1
+$EndComp
+Wire Wire Line
+	850  1600 850  1800
+Wire Wire Line
+	800  1800 1200 1800
+Connection ~ 850  1800
+Wire Wire Line
+	700  1600 850  1600
+Connection ~ 800  1600
+NoConn ~ 1100 1200
+NoConn ~ 1100 1300
+NoConn ~ 1100 1400
 $EndSCHEMATC

Commit message: Updated schematic
Parts:
- removed D205: GREEN, LEDs:LED_0603, symbol LED_ALT
- removed D206: YELLOW, LEDs:LED_0603, symbol LED_ALT
- removed D207: RED, LEDs:LED_0603, symbol LED_ALT
- removed R232, R233, R234: 680R, Resistors_SMD:R_0603_HandSoldering, symbol R
Connections:
- wire segments 163 -> 154
- no-connect marks 17 -> 20
Changed lines of the file:
@@
 LIBS:switches
 LIBS:iCE40hxk4_dev_board-cache
-EELAYER 26 0
+EELAYER 25 0
 EELAYER END
 $Descr A4 11693 8268
@@
 $EndComp
 $Comp
-L LED_ALT D205
-U 1 1 58F97BFA
-P 9250 3150
-F 0 "D205" H 9250 3250 50  0000 C CNN
-F 1 "GREEN" H 9250 3100 50  0000 C CNN
-F 2 "LEDs:LED_0603" H 9250 3150 50  0001 C CNN
-F 3 "www.kingbrightusa.com/images/catalog/SPEC/APTD1608LCGCK.pdf" H 9250 3150 50  0001 C CNN
-F 4 "2mA" H 9250 3150 60  0001 C CNN "If"
-F 5 "APTD1608LCGCK" H 9250 3350 50  0001 C CNN "MPN"
-F 6 "1.9V" H 9250 3150 60  0001 C CNN "Vf"
-	1    9250 3150
-	1    0    0    -1
-$EndComp
-$Comp
 L FT2232H U205
 U 1 1 58DACB1C
@@
 F 4 "FT2232H" H 6750 6350 50  0001 C CNN "MPN"
 	1    7800 4150
-	1    0    0    -1
-$EndComp
-$Comp
-L R R232
-U 1 1 58F9B086
-P 10300 3150
-F 0 "R232" V 10250 3300 50  0000 C CNN
-F 1 "680R" V 10300 3150 50  0000 C CNN
-F 2 "Resistors_SMD:R_0603_HandSoldering" V 10230 3150 50  0001 C CNN
-F 3 "http://www.mouser.com/ds/2/447/RC0603-272842.pdf" H 10300 3150 50  0001 C CNN
-F 4 "RC0603FR-07680RL" H 10250 3400 50  0001 C CNN "MPN"
-	1    10300 3150
-	0    1    1    0
-$EndComp
-$Comp
-L R R233
-U 1 1 58F9B3F0
-P 10300 3250
-F 0 "R233" V 10250 3400 50  0000 C CNN
-F 1 "680R" V 10300 3250 50  0000 C CNN
-F 2 "Resistors_SMD:R_0603_HandSoldering" V 10230 3250 50  0001 C CNN
-F 3 "http://www.mouser.com/ds/2/447/RC0603-272842.pdf" H 10300 3250 50  0001 C CNN
-F 4 "RC0603FR-07680RL" H 10250 3500 50  0001 C CNN "MPN"
-	1    10300 3250
-	0    1    1    0
-$EndComp
-$Comp
-L R R234
-U 1 1 58F9B988
-P 10300 3350
-F 0 "R234" V 10250 3500 50  0000 C CNN
-F 1 "680R" V 10300 3350 50  0000 C CNN
-F 2 "Resistors_SMD:R_0603_HandSoldering" V 10230 3350 50  0001 C CNN
-F 3 "http://www.mouser.com/ds/2/447/RC0603-272842.pdf" H 10300 3350 50  0001 C CNN
-F 4 "RC0603FR-07680RL" H 10250 3600 50  0001 C CNN "MPN"
-	1    10300 3350
-	0    1    1    0
-$EndComp
-$Comp
-L LED_ALT D206
-U 1 1 58F9D81C
-P 9550 3250
-F 0 "D206" H 9550 3350 50  0000 C CNN
-F 1 "YELLOW" H 9550 3200 50  0000 C CNN
-F 2 "LEDs:LED_0603" H 9550 3250 50  0001 C CNN
-F 3 "http://www.kingbrightusa.com/images/catalog/SPEC/APTD1608LSYCK.pdf" H 9550 3250 50  0001 C CNN
-F 4 "2mA" H 9550 3250 60  0001 C CNN "If"
-F 5 "APTD1608LSYCK" H 9550 3450 50  0001 C CNN "MPN"
-F 6 "1.75V" H 9550 3250 60  0001 C CNN "Vf"
-	1    9550 3250
-	1    0    0    -1
-$EndComp
-$Comp
-L LED_ALT D207
-U 1 1 58F9E03E
-P 9900 3350
-F 0 "D207" H 9900 3450 50  0000 C CNN
-F 1 "RED" H 9900 3300 50  0000 C CNN
-F 2 "LEDs:LED_0603" H 9900 3350 50  0001 C CNN
-F 3 "http://www.kingbrightusa.com/images/catalog/SPEC/APTD1608LSURCK.pdf" H 9900 3350 50  0001 C CNN
-F 4 "2mA" H 9900 3350 60  0001 C CNN "If"
-F 5 "APTD1608LSURCK" H 9900 3550 50  0001 C CNN "MPN"
-F 6 "1.75V" H 9900 3350 60  0001 C CNN "Vf"
-	1    9900 3350
 	1    0    0    -1
 $EndComp
@@
 Text Notes 1200 750  0    79   ~ 16
 EXTERNAL SOURCE
-Text Label 2250 1000 0    79   ~ 0
+Text Label 2075 1000 0    79   ~ 0
 Vext_filtered
 Text Label 1850 1700 2    79   ~ 0
@@
 Text HLabel 5200 3900 0    60   Output ~ 12
 +3.3V
-Text HLabel 10750 3250 2    60   Output ~ 12
-+3.3V
 Text Notes 3700 3000 0    51   ~ 0
 Fault is active low.
@@
 Wire Wire Line
 	3300 1000 3450 1000
-Wire Wire Line
-	9000 3150 9100 3150
-Wire Wire Line
-	9000 3250 9400 3250
-Wire Wire Line
-	9000 3350 9750 3350
-Wire Wire Line
-	10150 3350 10050 3350
-Wire Wire Line
-	10150 3250 9700 3250
-Wire Wire Line
-	10150 3150 9400 3150
-Wire Wire Line
-	10450 3150 10600 3150
-Wire Wire Line
-	10600 3150 10600 3350
-Wire Wire Line
-	10600 3350 10450 3350
-Wire Wire Line
-	10450 3250 10750 3250
 Wire Wire Line
 	5550 5800 6150 5800
@@
 Connection ~ 5700 2650
 Connection ~ 3450 1300
-Connection ~ 10600 3250
 Connection ~ 3850 1950
 $Comp
@@
 	1    0    0    -1
 $EndComp
-Wire Wire Line
-	3425 775  3425 1000
 Connection ~ 3425 1000
 Wire Wire Line
@@
 NoConn ~ 1100 1300
 NoConn ~ 1100 1400
+Wire Wire Line
+	3425 775  2950 775
+Wire Wire Line
+	2950 775  2950 1000
+Connection ~ 2950 1000
+NoConn ~ 9000 3150
+NoConn ~ 9000 3250
+NoConn ~ 9000 3350
 $EndSCHEMATC

Commit message: Doing re-routing
Parts:
- J1005: renamed from J?; footprint Connect:USB_Micro-B -> Connectors:USB_Micro-B
Changed lines of the file:
@@
 $EndComp
 $Comp
-L PWR_FLAG #FLG1003
+L PWR_FLAG #FLG039
 U 1 1 58E1521D
 P 1600 3600
-F 0 "#FLG1003" H 1600 3675 50  0001 C CNN
+F 0 "#FLG039" H 1600 3675 50  0001 C CNN
 F 1 "PWR_FLAG" H 1600 3750 50  0000 C CNN
 F 2 "" H 1600 3600 50  0001 C CNN
@@
 $EndComp
 $Comp
-L PWR_FLAG #FLG1002
+L PWR_FLAG #FLG040
 U 1 1 58E1552A
 P 1250 950
-F 0 "#FLG1002" H 1250 1025 50  0001 C CNN
+F 0 "#FLG040" H 1250 1025 50  0001 C CNN
 F 1 "PWR_FLAG" H 1250 1100 50  0000 C CNN
 F 2 "" H 1250 950 50  0001 C CNN
@@
 $EndComp
 $Comp
-L PWR_FLAG #FLG1006
+L PWR_FLAG #FLG041
 U 1 1 58F4F305
 P 6900 1200
-F 0 "#FLG1006" H 6900 1275 50  0001 C CNN
+F 0 "#FLG041" H 6900 1275 50  0001 C CNN
 F 1 "PWR_FLAG" H 6850 1450 50  0000 C CNN
 F 2 "" H 6900 1200 50  0001 C CNN
@@
 $EndComp
 $Comp
-L PWR_FLAG #FLG1004
+L PWR_FLAG #FLG042
 U 1 1 58F4F46B
 P 2600 3600
-F 0 "#FLG1004" H 2600 3675 50  0001 C CNN
+F 0 "#FLG042" H 2600 3675 50  0001 C CNN
 F 1 "PWR_FLAG" H 2600 3750 50  0000 C CNN
 F 2 "" H 2600 3600 50  0001 C CNN
@@
 $EndComp
 $Comp
-L PWR_FLAG #FLG1001
+L PWR_FLAG #FLG043
 U 1 1 58F8188C
 P 800 1800
-F 0 "#FLG1001" H 800 1875 50  0001 C CNN
+F 0 "#FLG043" H 800 1875 50  0001 C CNN
 F 1 "PWR_FLAG" H 800 1950 50  0000 C CNN
 F 2 "" H 800 1800 50  0001 C CNN
@@
 $EndComp
 $Comp
-L PWR_FLAG #FLG1005
+L PWR_FLAG #FLG044
 U 1 1 59694747
 P 4150 2200
-F 0 "#FLG1005" H 4150 2275 50  0001 C CNN
+F 0 "#FLG044" H 4150 2275 50  0001 C CNN
 F 1 "PWR_FLAG" H 4150 2350 50  0000 C CNN
 F 2 "" H 4150 2200 50  0001 C CNN
@@
 Connection ~ 5300 1900
 $Comp
-L USB_OTG J?
+L USB_OTG J1005
 U 1 1 599EBDA6
 P 800 1200
-F 0 "J?" H 600 1650 50  0000 L CNN
+F 0 "J1005" H 600 1650 50  0000 L CNN
 F 1 "USB_EXT" H 600 1550 50  0000 L CNN
-F 2 "Connect:USB_Micro-B" H 950 1150 50  0001 C CNN
+F 2 "Connectors:USB_Micro-B" H 950 1150 50  0001 C CNN
 F 3 "" H 950 1150 50  0001 C CNN
 	1    800  1200

Commit message: DRC
Parts:
- J1001, J1002, J1003, J1004: footprint library:Via-0.8mm -> library:TestPoint
Changed lines of the file:
@@
 F 0 "J1001" H 3625 875 50  0000 C CNN
 F 1 "Testpoint" V 3725 775 50  0000 C CNN
-F 2 "library:Via-0.8mm" H 3625 775 50  0001 C CNN
+F 2 "library:TestPoint" H 3625 775 50  0001 C CNN
 F 3 "" H 3625 775 50  0001 C CNN
 	1    3625 775
@@
 F 0 "J1002" H 3925 3600 50  0000 C CNN
 F 1 "Testpoint" V 4025 3500 50  0000 C CNN
-F 2 "library:Via-0.8mm" H 3925 3500 50  0001 C CNN
+F 2 "library:TestPoint" H 3925 3500 50  0001 C CNN
 F 3 "" H 3925 3500 50  0001 C CNN
 	1    3925 3500
@@
 F 0 "J1003" H 5075 1900 50  0000 C CNN
 F 1 "Testpoint" V 5175 1800 50  0000 C CNN
-F 2 "library:Via-0.8mm" H 5075 1800 50  0001 C CNN
+F 2 "library:TestPoint" H 5075 1800 50  0001 C CNN
 F 3 "" H 5075 1800 50  0001 C CNN
 	1    5075 1800
@@
 F 0 "J1004" H 6175 2600 50  0000 C CNN
 F 1 "Testpoint" V 6275 2500 50  0000 C CNN
-F 2 "library:Via-0.8mm" H 6175 2500 50  0001 C CNN
+F 2 "library:TestPoint" H 6175 2500 50  0001 C CNN
 F 3 "" H 6175 2500 50  0001 C CNN
 	1    6175 2500

Commit message: Updated some MPN
Parts:
- J1005, J202: MPN (none) -> 47642-0001
- U203: value 93LC56BT-I/O -> 93LC56BT-I/OT; MPN 93LC56BT-I/O -> 93LC56BT-I/OT
- U204: value MIC5355/6-xYMME -> MIC5355-S4YMME; MPN MIC5355/6-xYMME -> MIC5355-S4YMME
Changed lines of the file:
@@
 P 4500 4750
 F 0 "U203" H 4200 5000 50  0000 L CNN
-F 1 "93LC56BT-I/O" H 4550 5000 50  0000 L CNN
+F 1 "93LC56BT-I/OT" H 4550 5000 50  0000 L CNN
 F 2 "TO_SOT_Packages_SMD:SOT-23-6_Handsoldering" H 4150 4700 50  0001 C CNN
 F 3 "http://www.mouser.com/ds/2/268/21794b-74044.pdf" H 4150 4700 50  0001 C CNN
-F 4 "93LC56BT-I/O" H 4200 5100 50  0001 C CNN "MPN"
+F 4 "93LC56BT-I/OT" H 4200 5100 50  0001 C CNN "MPN"
 	1    4500 4750
 	1    0    0    -1
@@
 P 4800 2350
 F 0 "U204" H 4800 2675 50  0000 C CNN
-F 1 "MIC5355/6-xYMME" H 4800 2600 50  0000 C CNN
+F 1 "MIC5355-S4YMME" H 4800 2600 50  0000 C CNN
 F 2 "TO_SOT_Packages_SMD:SOT-23-8_Handsoldering" H 4850 2100 50  0001 L CNN
-F 3 "" H 4800 2350 50  0001 C CNN
-F 4 "MIC5355/6-xYMME" H 4800 2775 50  0001 C CNN "MPN"
+F 3 "http://www.mouser.com/ds/2/268/mic5355_6-779175.pdf" H 4800 2350 50  0001 C CNN
+F 4 "MIC5355-S4YMME " H 4800 2775 50  0001 C CNN "MPN"
 	1    4800 2350
 	1    0    0    -1
@@
 $EndComp
 $Comp
-L PWR_FLAG #FLG1003
+L PWR_FLAG #FLG039
 U 1 1 58E1521D
 P 1600 3600
-F 0 "#FLG1003" H 1600 3675 50  0001 C CNN
+F 0 "#FLG039" H 1600 3675 50  0001 C CNN
 F 1 "PWR_FLAG" H 1600 3750 50  0000 C CNN
 F 2 "" H 1600 3600 50  0001 C CNN
@@
 $EndComp
 $Comp
-L PWR_FLAG #FLG1002
+L PWR_FLAG #FLG040
 U 1 1 58E1552A
 P 1250 950
-F 0 "#FLG1002" H 1250 1025 50  0001 C CNN
+F 0 "#FLG040" H 1250 1025 50  0001 C CNN
 F 1 "PWR_FLAG" H 1250 1100 50  0000 C CNN
 F 2 "" H 1250 950 50  0001 C CNN
@@
 $EndComp
 $Comp
-L PWR_FLAG #FLG1006
+L PWR_FLAG #FLG041
 U 1 1 58F4F305
 P 6900 1200
-F 0 "#FLG1006" H 6900 1275 50  0001 C CNN
+F 0 "#FLG041" H 6900 1275 50  0001 C CNN
 F 1 "PWR_FLAG" H 6850 1450 50  0000 C CNN
 F 2 "" H 6900 1200 50  0001 C CNN
@@
 $EndComp
 $Comp
-L PWR_FLAG #FLG1004
+L PWR_FLAG #FLG042
 U 1 1 58F4F46B
 P 2600 3600
-F 0 "#FLG1004" H 2600 3675 50  0001 C CNN
+F 0 "#FLG042" H 2600 3675 50  0001 C CNN
 F 1 "PWR_FLAG" H 2600 3750 50  0000 C CNN
 F 2 "" H 2600 3600 50  0001 C CNN
@@
 $EndComp
 $Comp
-L PWR_FLAG #FLG1001
+L PWR_FLAG #FLG043
 U 1 1 58F8188C
 P 800 1800
-F 0 "#FLG1001" H 800 1875 50  0001 C CNN
+F 0 "#FLG043" H 800 1875 50  0001 C CNN
 F 1 "PWR_FLAG" H 800 1950 50  0000 C CNN
 F 2 "" H 800 1800 50  0001 C CNN
@@
 F 2 "Connectors:USB_Micro-B" H 1350 3850 50  0001 C CNN
 F 3 "" H 1350 3850 50  0001 C CNN
+F 4 "47642-0001" H 1200 3900 60  0001 C CNN "MPN"
 	1    1200 3900
 	1    0    0    -1
@@
 $EndComp
 $Comp
-L PWR_FLAG #FLG1005
+L PWR_FLAG #FLG044
 U 1 1 59694747
 P 4150 2200
-F 0 "#FLG1005" H 4150 2275 50  0001 C CNN
+F 0 "#FLG044" H 4150 2275 50  0001 C CNN
 F 1 "PWR_FLAG" H 4150 2350 50  0000 C CNN
 F 2 "" H 4150 2200 50  0001 C CNN
@@
 F 2 "Connectors:USB_Micro-B" H 950 1150 50  0001 C CNN
 F 3 "" H 950 1150 50  0001 C CNN
+F 4 "47642-0001" H 800 1200 60  0001 C CNN "MPN"
 	1    800  1200
 	1    0    0    -1
