File: USB+OSCILLATOR+REGULATOR.sch (KiCad schematic (older format))
At the start: 73 parts, among them J1001 Testpoint, J1002 Testpoint, J1003 Testpoint, J1004 Testpoint, J1005 USB_EXT, J202 USB_OTG, U201 MIC2005A-2YM5, U203 93LC56BT-I/OT, U204 MIC5355-S4YMME, U205 FT2232H

Commit message: Updated MPN to components avalaible in mouser. Updating footprints now ...
Parts:
- C205, C207, C213, C215: Datashet http://www.mouser.com/ds/2/40/TAJ_AUTO-783622-1093304.pdf -> (none); MPN TAJA475K016UNJ -> TMCMA1A475MTRF; VDC 16V -> 10V
- C214: MPN GRM21BR71C475KE51L -> GRM21BR71A475KE51L; VDC 16V -> 10V

Commit message: Updated BNC and USB footprints
Parts:
- J1005, J202: footprint Connectors:USB_Micro-B -> library:USB_Micro-B_47642-0001
Changed lines of the file:
@@
 F 0 "J202" H 1000 4350 50  0000 L CNN
 F 1 "USB_OTG" H 1000 4250 50  0000 L CNN
-F 2 "Connectors:USB_Micro-B" H 1350 3850 50  0001 C CNN
-F 3 "" H 1350 3850 50  0001 C CNN
+F 2 "library:USB_Micro-B_47642-0001" H 1350 3850 50  0001 C CNN
+F 3 "http://www.mouser.com/ds/2/276/0476420001_IO_CONNECTORS-229216.pdf" H 1350 3850 50  0001 C CNN
 F 4 "47642-0001" H 1200 3900 60  0001 C CNN "MPN"
 	1    1200 3900
@@
 F 0 "J1005" H 600 1650 50  0000 L CNN
 F 1 "USB_EXT" H 600 1550 50  0000 L CNN
-F 2 "Connectors:USB_Micro-B" H 950 1150 50  0001 C CNN
-F 3 "" H 950 1150 50  0001 C CNN
+F 2 "library:USB_Micro-B_47642-0001" H 950 1150 50  0001 C CNN
+F 3 "http://www.mouser.com/ds/2/276/0476420001_IO_CONNECTORS-229216.pdf" H 950 1150 50  0001 C CNN
 F 4 "47642-0001" H 800 1200 60  0001 C CNN "MPN"
 	1    800  1200

Commit message: Changed incorrect footprint
Parts:
- U204: footprint TO_SOT_Packages_SMD:SOT-23-8_Handsoldering -> Housings_SSOP:MSOP-8_3x3mm_Pitch0.65mm
Changed lines of the file:
@@
 F 0 "U204" H 4800 2675 50  0000 C CNN
 F 1 "MIC5355-S4YMME" H 4800 2600 50  0000 C CNN
-F 2 "TO_SOT_Packages_SMD:SOT-23-8_Handsoldering" H 4850 2100 50  0001 L CNN
+F 2 "Housings_SSOP:MSOP-8_3x3mm_Pitch0.65mm" H 4850 2100 50  0001 L CNN
 F 3 "http://www.mouser.com/ds/2/268/mic5355_6-779175.pdf" H 4800 2350 50  0001 C CNN
 F 4 "MIC5355-S4YMME " H 4800 2775 50  0001 C CNN "MPN"

Commit message: Changed MPN FT2232H to FT2232HL
Parts:
- U205: MPN FT2232H -> FT2232HL
Changed lines of the file:
@@
 F 2 "Housings_QFP:LQFP-64_10x10mm_Pitch0.5mm" H 7800 4150 50  0001 C CNN
 F 3 "" H 7800 4150 50  0001 C CNN
-F 4 "FT2232H" H 6750 6350 50  0001 C CNN "MPN"
+F 4 "FT2232HL" H 6750 6350 50  0001 C CNN "MPN"
 	1    7800 4150
 	1    0    0    -1

Commit message: New BOM generated with kicost
Parts:
- J1001, J1002, J1003, J1004: DNP (none) -> 1
